File: Hardware/BPS-Leader.kicad_sch (KiCad schematic)
At the start: 42 parts, among them J11 Conn_02x06_Counter_Clockwise, J15 Conn_01x05, J16 Conn_01x05, J21 SFH11-PBPC-D05-ST-BK, J3 Conn_01x02, J5 Conn_02x06_Counter_Clockwise, J8 CarCANConnector, Q11 IRLML0030, U12 SHT4x

Commit message: condensed custom lirbraries
Parts:
- F2, F3: footprint FUSE 3568:3568 -> CustomKiCad-Library:3568
- LOGO3: footprint Custom-KiCadLibraries:Beach -> CustomKiCad-Library:Beach
- LOGO4: footprint Custom-KiCadLibraries:Gear -> CustomKiCad-Library:Gear
Changed lines of the file:
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@@
 			)
 		)
-		(property "Footprint" "Custom-KiCadLibraries:Gear"
+		(property "Footprint" "CustomKiCad-Library:Gear"
 			(at 360.68 221.615 0)
 			(effects
@@
 			)
 		)
-		(property "Footprint" "FUSE 3568:3568"
+		(property "Footprint" "CustomKiCad-Library:3568"
 			(at 74.93 108.458 90)
 			(effects
@@
 			)
 		)
-		(property "Footprint" "FUSE 3568:3568"
+		(property "Footprint" "CustomKiCad-Library:3568"
 			(at 139.7 98.298 90)
 			(effects
@@
 			)
 		)
-		(property "Footprint" "Custom-KiCadLibraries:Beach"
+		(property "Footprint" "CustomKiCad-Library:Beach"
 			(at 360.68 230.505 0)
 			(effects
@@
 			)
 		)
-		(property "Datasheet" "https://www.mouser.com/datasheet/3/1278/1/HT_DS_Datasheet_SHT4x_5.pdf"
+		(property "Datasheet" "https://sensirion.com/media/documents/33FD6951/624C4357/Datasheet_SHT4x.pdf"
 			(at 256.2478 190.9428 0)
 			(effects
