File: Hardware/ArrPreContactor.kicad_sch (KiCad schematic)
At the start: 15 parts, among them Q10 IRLML0030, Q14 IRLML0030

Commit message: circuit blocks designed, schematic updated
Parts:
- removed TP18: TestPoint, TestPoint:TestPoint_Pad_1.0x1.0mm, symbol Connector:TestPoint
Changed lines of the file:
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@@
+	(wire
+		(pts
+			(xy 92.71 99.06) (xy 102.87 99.06)
+		)
+		(stroke
+			(width 0)
+			(type default)
+		)
+	)
 	(wire
 		(pts
@@
 	(wire
 		(pts
-			(xy 226.06 92.71) (xy 241.3 92.71)
-		)
-		(stroke
-			(width 0)
-			(type default)
-		)
-	)
-	(wire
-		(pts
 			(xy 88.9 85.09) (xy 92.71 85.09)
 		)
@@
 	(wire
 		(pts
-			(xy 92.71 99.06) (xy 116.84 99.06)
-		)
-		(stroke
-			(width 0)
-			(type default)
-		)
-	)
-	(wire
-		(pts
 			(xy 191.77 101.6) (xy 191.77 102.87)
 		)
@@
 			(width 0)
 			(type default)
-		)
-	)
-	(label "ARRAY_PRE_CONTROL-"
-		(at 116.84 99.06 180)
-		(effects
-			(font
-				(size 1.27 1.27)
-			)
-			(justify right bottom)
 		)
 	)
@@
 		)
 	)
+	(hierarchical_label "ARRAY_PRE_CONTROL-"
+		(shape input)
+		(at 102.87 99.06 0)
+		(effects
+			(font
+				(size 1.27 1.27)
+			)
+			(justify left)
+		)
+	)
 	(hierarchical_label "ARRAY_PRE_SENSE-"
 		(shape input)
 		(at 241.3 96.52 0)
-		(effects
-			(font
-				(size 1.27 1.27)
-			)
-			(justify left)
-		)
-	)
-	(hierarchical_label "ARRAY_PRE_CONTROL-"
-		(shape input)
-		(at 241.3 92.71 0)
 		(effects
 			(font
@@
 					(unit 1)
 				)
-			)
-		)
-	)
-	(symbol
-		(lib_id "Connector:TestPoint")
-		(at 226.06 92.71 90)
-		(mirror x)
-		(unit 1)
-		(exclude_from_sim no)
-		(in_bom no)
-		(on_board yes)
-		(dnp no)
-		(property "Reference" "TP18"
-			(at 225.044 89.662 90)
-			(effects
-				(font
-					(size 1.27 1.27)
-				)
-				(justify left)
-			)
-		)
-		(property "Value" "TestPoint"
-			(at 227.838 87.122 90)
-			(effects
-				(font
-					(size 1.27 1.27)
-				)
-				(justify left)
-			)
-		)
-		(property "Footprint" "TestPoint:TestPoint_Pad_1.0x1.0mm"
-			(at 226.06 97.79 0)
-			(effects
-				(font
-					(size 1.27 1.27)
-				)
-				(hide yes)
-			)
-		)
-		(property "Datasheet" "~"
-			(at 226.06 97.79 0)
-			(effects
-				(font
-					(size 1.27 1.27)
-				)
-				(hide yes)
-			)
-		)
-		(property "Description" "test point"
-			(at 226.06 92.71 0)
-			(effects
-				(font
-					(size 1.27 1.27)
-				)
-				(hide yes)
-			)
-		)
-		(property "Manufactuerer" ""
-			(at 226.06 92.71 90)
-			(effects
-				(font
-					(size 1.27 1.27)
-				)
-				(hide yes)
-			)
-		)
-		(pin "1"
-		)
-		(instances
-			(project "BPS-Leader"
-				(path "/fb37da34-e420-4994-8cc1-079e8c0fa48e/3dd44f8f-72d2-4c34-a907-2c0b2702aa52"
-					(reference "TP18")
-					(unit 1)
-				)

Commit message: RevB layout completed
Parts:
- TP16: value TestPoint -> ArrPreCtrl
- TP17: value TestPoint -> ArrPreSns
Changed lines of the file:
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@@
 			)
 		)
-		(property "Value" "TestPoint"
+		(property "Value" "ArrPreSns"
 			(at 187.706 97.028 0)
 			(effects
@@
 			)
 		)
-		(property "Value" "TestPoint"
+		(property "Value" "ArrPreCtrl"
 			(at 72.39 105.664 90)
 			(effects

Commit message: JLC Production Files
Parts:
- ArrayPre1: LCSC (none) -> C84263
- C23: LCSC (none) -> C15849
- C39: LCSC (none) -> C14663
- D9: LCSC (none) -> C6326606
- Q10, Q14: LCSC (none) -> C67272
- R77, R79, R86, R87: LCSC (none) -> C25804
- R78: LCSC (none) -> C2907165
- R80: LCSC (none) -> C21190
Changed lines of the file:
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@@
+			)
+		)
+		(property "LCSC" "C25804"
+			(at 224.282 101.854 0)
+			(effects
+				(font
+					(size 1.27 1.27)
+				)
+				(hide yes)
 			)
 		)
@@
 			)
 		)
+		(property "LCSC" "C25804"
+			(at 194.31 107.9499 0)
+			(effects
+				(font
+					(size 1.27 1.27)
+				)
+				(hide yes)
+			)
+		)
 		(pin "2"
 		)
@@
 			)
 		)
+		(property "LCSC" "C67272"
+			(at 199.644 98.806 0)
+			(effects
+				(font
+					(size 1.27 1.27)
+				)
+				(hide yes)
+			)
+		)
 		(pin "1"
 		)
@@
 			)
 		)
+		(property "LCSC" "C2907165"
+			(at 85.09 79.375 0)
+			(effects
+				(font
+					(size 1.27 1.27)
+				)
+				(hide yes)
+			)
+		)
 		(pin "2"
 		)
@@
 			)
 		)
+		(property "LCSC" "C6326606"
+			(at 95.25 88.9 0)
+			(effects
+				(font
+					(size 1.27 1.27)
+				)
+				(hide yes)
+			)
+		)
 		(pin "1"
 		)
@@
 			)
 		)
+		(property "LCSC" "C67272"
+			(at 97.028 108.966 0)
+			(effects
+				(font
+					(size 1.27 1.27)
+				)
+				(hide yes)
+			)
+		)
 		(pin "1"
 		)
@@
 			)
 		)
+		(property "LCSC" "C25804"
+			(at 82.55 111.7599 0)
+			(effects
+				(font
+					(size 1.27 1.27)
+				)
+				(hide yes)
+			)
+		)
 		(pin "2"
 		)
@@
 			)
 		)
+		(property "LCSC" "C15849"
+			(at 179.705 107.9499 0)
+			(effects
+				(font
+					(size 1.27 1.27)
+				)
+				(hide yes)
+			)
+		)
 		(pin "2"
 		)
@@
 			)
 		)
+		(property "LCSC" "C14663"
+			(at 210.82 104.1401 0)
+			(effects
+				(font
+					(size 1.27 1.27)
+				)
+				(hide yes)
+			)
+		)
 		(pin "1"
 		)
@@
 			)
 		)
+		(property "LCSC" "C21190"
+			(at 216.916 94.488 0)
+			(effects
+				(font
+					(size 1.27 1.27)
+				)
+				(hide yes)
+			)
+		)
 		(pin "2"
 		)
@@
 			)
 		)
+		(property "LCSC" "C25804"
+			(at 232.156 94.488 0)
+			(effects
+				(font
+					(size 1.27 1.27)
+				)
+				(hide yes)
+			)
+		)
 		(pin "2"
 		)
@@
 			(effects
 				(font
+					(size 1.27 1.27)
+				)
+				(hide yes)
+			)
+		)
+		(property "LCSC" "C84263"
+			(at 81.28 91.7574 0)
+			(effects
+				(font

Commit message: condensed custom lirbraries
Parts:
- D9: footprint VSSAF522-M3/H:SODFL5226X100N -> CustomKiCad-Library:SODFL5226X100N
Changed lines of the file:
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@@
 			)
 		)
-		(property "Footprint" "VSSAF522-M3/H:SODFL5226X100N"
+		(property "Footprint" "CustomKiCad-Library:SODFL5226X100N"
 			(at 88.265 91.44 0)
 			(effects

Commit message: RevC layout
Parts:
- D33: renamed from ArrayPre1; value LED -> ArrayPre
Changed lines of the file:
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@@
 		(dnp no)
 		(fields_autoplaced yes)
-		(property "Reference" "ArrayPre1"
+		(property "Reference" "D33"
 			(at 81.28 91.7574 90)
 			(effects
@@
 			)
 		)
-		(property "Value" "LED"
+		(property "Value" "ArrayPre"
 			(at 81.28 94.2974 90)
 			(effects
@@
 			(project "BPS-Leader"
 				(path "/fb37da34-e420-4994-8cc1-079e8c0fa48e/3dd44f8f-72d2-4c34-a907-2c0b2702aa52"
-					(reference "ArrayPre1")
+					(reference "D33")
 					(unit 1)
 				)

Commit message: JLCPCB ouput files
Parts:
- R80: P/N CRCW060310K0FKEI -> CRCW06031K00FKEI
