File: Hardware/Arr_Contactor.kicad_sch (KiCad schematic)
At the start: 15 parts, among them Q6 IRLML0030, Q9 IRLML0030

Commit message: circuit blocks designed, schematic updated
Parts:
- removed TP15: TestPoint, TestPoint:TestPoint_Pad_1.0x1.0mm, symbol Connector:TestPoint
Changed lines of the file:
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@@
+	(wire
+		(pts
+			(xy 92.71 102.87) (xy 101.6 102.87)
+		)
+		(stroke
+			(width 0)
+			(type default)
+		)
+	)
 	(wire
 		(pts
@@
 	(wire
 		(pts
-			(xy 226.06 96.52) (xy 241.3 96.52)
-		)
-		(stroke
-			(width 0)
-			(type default)
-		)
-	)
-	(wire
-		(pts
 			(xy 191.77 105.41) (xy 191.77 106.68)
 		)
@@
 	(wire
 		(pts
-			(xy 92.71 102.87) (xy 111.76 102.87)
-		)
-		(stroke
-			(width 0)
-			(type default)
-		)
-	)
-	(wire
-		(pts
 			(xy 207.01 100.33) (xy 213.36 100.33)
 		)
@@
 			(width 0)
 			(type default)
-		)
-	)
-	(label "ARRAY_CONTROL-"
-		(at 111.76 102.87 180)
-		(effects
-			(font
-				(size 1.27 1.27)
-			)
-			(justify right bottom)
 		)
 	)
@@
 	(hierarchical_label "ARRAY_CONTROL-"
 		(shape input)
-		(at 241.3 96.52 0)
+		(at 101.6 102.87 0)
 		(effects
 			(font
@@
 					(unit 1)
 				)
-			)
-		)
-	)
-	(symbol
-		(lib_id "Connector:TestPoint")
-		(at 226.06 96.52 90)
-		(mirror x)
-		(unit 1)
-		(exclude_from_sim no)
-		(in_bom no)
-		(on_board yes)
-		(dnp no)
-		(property "Reference" "TP15"
-			(at 225.044 93.472 90)
-			(effects
-				(font
-					(size 1.27 1.27)
-				)
-				(justify left)
-			)
-		)
-		(property "Value" "TestPoint"
-			(at 227.838 90.932 90)
-			(effects
-				(font
-					(size 1.27 1.27)
-				)
-				(justify left)
-			)
-		)
-		(property "Footprint" "TestPoint:TestPoint_Pad_1.0x1.0mm"
-			(at 226.06 101.6 0)
-			(effects
-				(font
-					(size 1.27 1.27)
-				)
-				(hide yes)
-			)
-		)
-		(property "Datasheet" "~"
-			(at 226.06 101.6 0)
-			(effects
-				(font
-					(size 1.27 1.27)
-				)
-				(hide yes)
-			)
-		)
-		(property "Description" "test point"
-			(at 226.06 96.52 0)
-			(effects
-				(font
-					(size 1.27 1.27)
-				)
-				(hide yes)
-			)
-		)
-		(property "Manufactuerer" ""
-			(at 226.06 96.52 90)
-			(effects
-				(font
-					(size 1.27 1.27)
-				)
-				(hide yes)
-			)
-		)
-		(pin "1"
-		)
-		(instances
-			(project "BPS-Leader"
-				(path "/fb37da34-e420-4994-8cc1-079e8c0fa48e/013fafe9-9f8f-4070-b42f-299f0280561e"
-					(reference "TP15")
-					(unit 1)
-				)

Commit message: RevB layout completed
Parts:
- TP13: value TestPoint -> ArrCtrl
- TP14: value TestPoint -> ArrSns
Changed lines of the file:
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@@
 			)
 		)
-		(property "Value" "TestPoint"
+		(property "Value" "ArrSns"
 			(at 187.706 100.838 0)
 			(effects
@@
 			)
 		)
-		(property "Value" "TestPoint"
+		(property "Value" "ArrCtrl"
 			(at 72.39 109.474 90)
 			(effects

Commit message: JLC Production Files
Parts:
- Array1: LCSC (none) -> C84263
- C19: LCSC (none) -> C15849
- C22: LCSC (none) -> C14663
- D8: LCSC (none) -> C6326606
- Q6, Q9: LCSC (none) -> C67272
- R38, R40, R44, R45: LCSC (none) -> C25804
- R39: LCSC (none) -> C2907165
- R41: LCSC (none) -> C21190
Changed lines of the file:
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@@
+			)
+		)
+		(property "LCSC" "C14663"
+			(at 210.82 107.9501 0)
+			(effects
+				(font
+					(size 1.27 1.27)
+				)
+				(hide yes)
 			)
 		)
@@
 			)
 		)
+		(property "LCSC" "C21190"
+			(at 216.916 98.298 0)
+			(effects
+				(font
+					(size 1.27 1.27)
+				)
+				(hide yes)
+			)
+		)
 		(pin "2"
 		)
@@
 		(property "Description" "5.3A Id, 30V Vds, 27mOhm Rds, N-Channel HEXFET Power MOSFET, SOT-23"
 			(at 90.17 110.49 0)
+			(effects
+				(font
+					(size 1.27 1.27)
+				)
+				(hide yes)
+			)
+		)
+		(property "LCSC" "C67272"
+			(at 97.028 112.776 0)
 			(effects
 				(font
@@
 			)
 		)
+		(property "LCSC" "C84263"
+			(at 81.28 95.5674 0)
+			(effects
+				(font
+					(size 1.27 1.27)
+				)
+				(hide yes)
+			)
+		)
 		(pin "1"
 		)
@@
 			)
 		)
+		(property "LCSC" "C2907165"
+			(at 85.09 83.185 0)
+			(effects
+				(font
+					(size 1.27 1.27)
+				)
+				(hide yes)
+			)
+		)
 		(pin "2"
 		)
@@
 			)
 		)
+		(property "LCSC" "C25804"
+			(at 82.55 115.5699 0)
+			(effects
+				(font
+					(size 1.27 1.27)
+				)
+				(hide yes)
+			)
+		)
 		(pin "2"
 		)
@@
 			)
 		)
+		(property "LCSC" "C15849"
+			(at 179.705 111.7599 0)
+			(effects
+				(font
+					(size 1.27 1.27)
+				)
+				(hide yes)
+			)
+		)
 		(pin "2"
 		)
@@
 			)
 		)
+		(property "LCSC" "C25804"
+			(at 194.31 111.7599 0)
+			(effects
+				(font
+					(size 1.27 1.27)
+				)
+				(hide yes)
+			)
+		)
 		(pin "2"
 		)
@@
 			)
 		)
+		(property "LCSC" "C25804"
+			(at 232.156 98.298 0)
+			(effects
+				(font
+					(size 1.27 1.27)
+				)
+				(hide yes)
+			)
+		)
 		(pin "2"
 		)
@@
 			)
 		)
+		(property "LCSC" "C25804"
+			(at 224.282 105.664 0)
+			(effects
+				(font
+					(size 1.27 1.27)
+				)
+				(hide yes)
+			)
+		)
 		(pin "2"
 		)
@@
 		(property "P/N" "VSSAF522-M3/H"
 			(at 92.71 95.25 90)
+			(effects
+				(font
+					(size 1.27 1.27)
+				)
+				(hide yes)
+			)
+		)
+		(property "LCSC" "C6326606"
+			(at 95.25 92.71 0)
 			(effects
 				(font
@@
 			(effects
 				(font
+					(size 1.27 1.27)
+				)
+				(hide yes)
+			)
+		)
+		(property "LCSC" "C67272"
+			(at 199.644 102.616 0)
+			(effects
+				(font

Commit message: condensed custom lirbraries
Parts:
- D8: footprint VSSAF522-M3/H:SODFL5226X100N -> Package_TO_SOT_THT:TO-247-2_Vertical
Changed lines of the file:
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@@
 			)
 		)
-		(property "Footprint" "VSSAF522-M3/H:SODFL5226X100N"
+		(property "Footprint" "Package_TO_SOT_THT:TO-247-2_Vertical"
 			(at 88.265 95.25 0)
 			(effects
@@
 			)
 		)
-		(property "Datasheet" "https://www.mouser.com/ProductDetail/Vishay-General-Semiconductor/VSSAF522-M3-H?qs=UkDUCjYnTB00gpgD%2Fb%2Fw%252BA%3D%3D"
+		(property "Datasheet" "https://www.wolfspeed.com/media/downloads/103/C3D25170H.pdf"
 			(at 92.71 95.25 0)
 			(effects
@@
 			)
 		)
-		(property "Description" ""
+		(property "Description" "1700V, 25A, SiC Schottky Diode, TO-247"
 			(at 92.71 95.25 0)
 			(effects

Commit message: RevC layout
Parts:
- D34: renamed from Array1; value LED -> Array
- D8: footprint Package_TO_SOT_THT:TO-247-2_Vertical -> CustomKiCad-Library:SODFL5226X100N
Changed lines of the file:
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@@
 		(dnp no)
 		(fields_autoplaced yes)
-		(property "Reference" "Array1"
+		(property "Reference" "D34"
 			(at 81.28 95.5674 90)
 			(effects
@@
 			)
 		)
-		(property "Value" "LED"
+		(property "Value" "Array"
 			(at 81.28 98.1074 90)
 			(effects
@@
 			(project "BPS-Leader"
 				(path "/fb37da34-e420-4994-8cc1-079e8c0fa48e/013fafe9-9f8f-4070-b42f-299f0280561e"
-					(reference "Array1")
+					(reference "D34")
 					(unit 1)
 				)
@@
 			)
 		)
-		(property "Footprint" "Package_TO_SOT_THT:TO-247-2_Vertical"
+		(property "Footprint" "CustomKiCad-Library:SODFL5226X100N"
 			(at 88.265 95.25 0)
 			(effects

Commit message: JLCPCB ouput files
Parts:
- R41: P/N CRCW060310K0FKEI -> CRCW06031K00FKEI
