File: Hardware/HV+Contact.kicad_sch (KiCad schematic)
At the start: 16 parts, among them J6 ContactorConnector, Q1 IRLML0030, Q3 IRLML0030

Commit message: circuit blocks designed, schematic updated
Parts:
- removed TP8: TestPoint, TestPoint:TestPoint_Pad_1.0x1.0mm, symbol Connector:TestPoint
Changed lines of the file:
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@@
-	)
-	(symbol
-		(lib_id "Connector:TestPoint")
-		(at 234.95 101.6 90)
-		(mirror x)
-		(unit 1)
-		(exclude_from_sim no)
-		(in_bom no)
-		(on_board yes)
-		(dnp no)
-		(property "Reference" "TP8"
-			(at 233.934 98.552 90)
-			(effects
-				(font
-					(size 1.27 1.27)
-				)
-				(justify left)
-			)
-		)
-		(property "Value" "TestPoint"
-			(at 236.728 96.012 90)
-			(effects
-				(font
-					(size 1.27 1.27)
-				)
-				(justify left)
-			)
-		)
-		(property "Footprint" "TestPoint:TestPoint_Pad_1.0x1.0mm"
-			(at 234.95 106.68 0)
-			(effects
-				(font
-					(size 1.27 1.27)
-				)
-				(hide yes)
-			)
-		)
-		(property "Datasheet" "~"
-			(at 234.95 106.68 0)
-			(effects
-				(font
-					(size 1.27 1.27)
-				)
-				(hide yes)
-			)
-		)
-		(property "Description" "test point"
-			(at 234.95 101.6 0)
-			(effects
-				(font
-					(size 1.27 1.27)
-				)
-				(hide yes)
-			)
-		)
-		(property "Manufactuerer" ""
-			(at 234.95 101.6 90)
-			(effects
-				(font
-					(size 1.27 1.27)
-				)
-				(hide yes)
-			)
-		)
-		(pin "1"
-		)
-		(instances
-			(project "BPS-Leader"
-				(path "/fb37da34-e420-4994-8cc1-079e8c0fa48e/74963854-952a-4575-ade4-c65bd9c86e44"
-					(reference "TP8")
-					(unit 1)
-				)
-			)
-		)
 	)
 	(symbol

Commit message: intial layout design
Changed lines of the file:
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@@
 		(dnp no)
 		(property "Reference" "TP7"
-			(at 188.468 105.664 0)
+			(at 194.564 103.886 0)
 			(effects
 				(font

Commit message: RevB layout completed
Parts:
- TP4: value TestPoint -> HV+Ctrl
- TP7: value TestPoint -> HV+Sns
Changed lines of the file:
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@@
 			)
 		)
-		(property "Value" "TestPoint"
+		(property "Value" "HV+Ctrl"
 			(at 85.09 114.554 90)
 			(effects
@@
 			)
 		)
-		(property "Value" "TestPoint"
+		(property "Value" "HV+Sns"
 			(at 197.866 105.918 0)
 			(effects

Commit message: JLC Production Files
Parts:
- C14: LCSC (none) -> C15849
- C15: LCSC (none) -> C14663
- D32: renamed from HV+1; value LED -> HV+; LCSC (none) -> C84263
- D5: LCSC (none) -> C6326606
- Q1, Q3: LCSC (none) -> C67272
- R12, R19, R21, R29: LCSC (none) -> C25804
- R15: LCSC (none) -> C2907165
- R20: LCSC (none) -> C21190
Changed lines of the file:
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@@
 		(dnp no)
 		(fields_autoplaced yes)
-		(property "Reference" "HV+1"
+		(property "Reference" "D32"
 			(at 93.98 100.6474 90)
 			(effects
@@
 			)
 		)
-		(property "Value" "LED"
+		(property "Value" "HV+"
 			(at 93.98 103.1874 90)
 			(effects
@@
 			)
 		)
+		(property "LCSC" "C84263"
+			(at 93.98 100.6474 0)
+			(effects
+				(font
+					(size 1.27 1.27)
+				)
+				(hide yes)
+			)
+		)
 		(pin "1"
 		)
@@
 			(project "BPS-Leader"
 				(path "/fb37da34-e420-4994-8cc1-079e8c0fa48e/74963854-952a-4575-ade4-c65bd9c86e44"
-					(reference "HV+1")
+					(reference "D32")
 					(unit 1)
 				)
@@
 			)
 		)
+		(property "LCSC" "C25804"
+			(at 95.25 120.6499 0)
+			(effects
+				(font
+					(size 1.27 1.27)
+				)
+				(hide yes)
+			)
+		)
 		(pin "2"
 		)
@@
 			)
 		)
+		(property "LCSC" "C25804"
+			(at 234.442 110.744 0)
+			(effects
+				(font
+					(size 1.27 1.27)
+				)
+				(hide yes)
+			)
+		)
 		(pin "2"
 		)
@@
 			)
 		)
+		(property "LCSC" "C67272"
+			(at 109.728 117.856 0)
+			(effects
+				(font
+					(size 1.27 1.27)
+				)
+				(hide yes)
+			)
+		)
 		(pin "1"
 		)
@@
 			)
 		)
+		(property "LCSC" "C25804"
+			(at 242.316 103.378 0)
+			(effects
+				(font
+					(size 1.27 1.27)
+				)
+				(hide yes)
+			)
+		)
 		(pin "2"
 		)
@@
 			)
 		)
+		(property "LCSC" "C15849"
+			(at 189.865 116.8399 0)
+			(effects
+				(font
+					(size 1.27 1.27)
+				)
+				(hide yes)
+			)
+		)
 		(pin "2"
 		)
@@
 			)
 		)
+		(property "LCSC" "C2907165"
+			(at 97.79 88.265 0)
+			(effects
+				(font
+					(size 1.27 1.27)
+				)
+				(hide yes)
+			)
+		)
 		(pin "2"
 		)
@@
 			)
 		)
+		(property "LCSC" "C25804"
+			(at 204.47 116.8399 0)
+			(effects
+				(font
+					(size 1.27 1.27)
+				)
+				(hide yes)
+			)
+		)
 		(pin "2"
 		)
@@
 			)
 		)
+		(property "LCSC" "C14663"
+			(at 220.98 113.0301 0)
+			(effects
+				(font
+					(size 1.27 1.27)
+				)
+				(hide yes)
+			)
+		)
 		(pin "1"
 		)
@@
 			)
 		)
+		(property "LCSC" "C67272"
+			(at 209.804 107.696 0)
+			(effects
+				(font
+					(size 1.27 1.27)
+				)
+				(hide yes)
+			)
+		)
 		(pin "1"
 		)
@@
 			)
 		)
+		(property "LCSC" "C21190"
+			(at 227.076 103.378 0)
+			(effects
+				(font
+					(size 1.27 1.27)
+				)
+				(hide yes)
+			)
+		)
 		(pin "2"
 		)
@@
 			(effects
 				(font
+					(size 1.27 1.27)
+				)
+				(hide yes)
+			)
+		)
+		(property "LCSC" "C6326606"
+			(at 107.95 97.79 0)
+			(effects
+				(font

Commit message: condensed custom lirbraries
Parts:
- D5: footprint VSSAF522-M3/H:SODFL5226X100N -> CustomKiCad-Library:SODFL5226X100N
Changed lines of the file:
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@@
 			)
 		)
-		(property "Footprint" "VSSAF522-M3/H:SODFL5226X100N"
+		(property "Footprint" "CustomKiCad-Library:SODFL5226X100N"
 			(at 100.965 100.33 0)
 			(effects

Commit message: RevC layout
Connections:
- net +24V: now also D5.1 (K), R15.2; no longer J6.1 (Con+(24V))
- net ESTOP_OUT: now also J6.1 (Con+(24V)); no longer D5.1 (K), R15.2
Changed lines of the file:
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@@
 	(wire
 		(pts
-			(xy 246.38 97.79) (xy 250.19 97.79)
+			(xy 247.65 97.79) (xy 250.19 97.79)
 		)
 		(stroke
@@
 		(pts
 			(xy 217.17 116.84) (xy 217.17 115.57)
-		)
-		(stroke
-			(width 0)
-			(type default)
-		)
-	)
-	(wire
-		(pts
-			(xy 246.38 92.71) (xy 246.38 97.79)
 		)
 		(stroke
@@
 	(hierarchical_label "ESTOP_OUT"
 		(shape input)
-		(at 105.41 86.36 90)
+		(at 247.65 97.79 180)
 		(effects
 			(font
 				(size 1.27 1.27)
 			)
-			(justify left)
+			(justify right)
 		)
 	)
@@
 	)
 	(symbol
+		(lib_id "power:+24V")
+		(at 105.41 86.36 0)
+		(unit 1)
+		(exclude_from_sim no)
+		(in_bom yes)
+		(on_board yes)
+		(dnp no)
+		(fields_autoplaced yes)
+		(property "Reference" "#PWR057"
+			(at 105.41 90.17 0)
+			(effects
+				(font
+					(size 1.27 1.27)
+				)
+				(hide yes)
+			)
+		)
+		(property "Value" "+24V"
+			(at 105.41 81.28 0)
+			(effects
+				(font
+					(size 1.27 1.27)
+				)
+			)
+		)
+		(property "Footprint" ""
+			(at 105.41 86.36 0)
+			(effects
+				(font
+					(size 1.27 1.27)
+				)
+				(hide yes)
+			)
+		)
+		(property "Datasheet" ""
+			(at 105.41 86.36 0)
+			(effects
+				(font
+					(size 1.27 1.27)
+				)
+				(hide yes)
+			)
+		)
+		(property "Description" "Power symbol creates a global label with name \"+24V\""
+			(at 105.41 86.36 0)
+			(effects
+				(font
+					(size 1.27 1.27)
+				)
+				(hide yes)
+			)
+		)
+		(pin "1"
+		)
+		(instances
+			(project "BPS-Leader"
+				(path "/fb37da34-e420-4994-8cc1-079e8c0fa48e/74963854-952a-4575-ade4-c65bd9c86e44"
+					(reference "#PWR057")
+					(unit 1)
+				)
+			)
+		)
+	)
+	(symbol
 		(lib_id "Device:R_US")
 		(at 242.57 105.41 90)
@@
 					(unit 1)
 				)
-			)
-		)
-	)
-	(symbol
-		(lib_id "power:+24V")
-		(at 246.38 92.71 0)
-		(unit 1)
-		(exclude_from_sim no)
-		(in_bom yes)
-		(on_board yes)
-		(dnp no)
-		(fields_autoplaced yes)
-		(property "Reference" "#PWR057"
-			(at 246.38 96.52 0)
-			(effects
-				(font
-					(size 1.27 1.27)
-				)
-				(hide yes)
-			)
-		)
-		(property "Value" "+24V"
-			(at 246.38 87.63 0)
-			(effects
-				(font
-					(size 1.27 1.27)
-				)
-			)
-		)
-		(property "Footprint" ""
-			(at 246.38 92.71 0)
-			(effects
-				(font
-					(size 1.27 1.27)
-				)
-				(hide yes)
-			)
-		)
-		(property "Datasheet" ""
-			(at 246.38 92.71 0)
-			(effects
-				(font
-					(size 1.27 1.27)
-				)
-				(hide yes)
-			)
-		)
-		(property "Description" "Power symbol creates a global label with name \"+24V\""
-			(at 246.38 92.71 0)
-			(effects
-				(font
-					(size 1.27 1.27)
-				)
-				(hide yes)
-			)
-		)
-		(pin "1"
-		)
-		(instances
-			(project "BPS-Leader"
-				(path "/fb37da34-e420-4994-8cc1-079e8c0fa48e/74963854-952a-4575-ade4-c65bd9c86e44"
-					(reference "#PWR057")
-					(unit 1)
-				)

Commit message: JLCPCB ouput files
Parts:
- R20: P/N CRCW060310K0FKEI -> CRCW06031K00FKEI
