File: Hardware/HV-Contact.kicad_sch (KiCad schematic)
At the start: 16 parts, among them J9 ContactorConnector, Q4 IRLML0030, Q5 IRLML0030

Commit message: circuit blocks designed, schematic updated
Parts:
- removed TP12: TestPoint, TestPoint:TestPoint_Pad_1.0x1.0mm, symbol Connector:TestPoint
Changed lines of the file:
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@@
-		)
-	)
-	(symbol
-		(lib_id "Connector:TestPoint")
-		(at 228.6 90.17 90)
-		(mirror x)
-		(unit 1)
-		(exclude_from_sim no)
-		(in_bom no)
-		(on_board yes)
-		(dnp no)
-		(property "Reference" "TP12"
-			(at 227.584 87.122 90)
-			(effects
-				(font
-					(size 1.27 1.27)
-				)
-				(justify left)
-			)
-		)
-		(property "Value" "TestPoint"
-			(at 230.378 84.582 90)
-			(effects
-				(font
-					(size 1.27 1.27)
-				)
-				(justify left)
-			)
-		)
-		(property "Footprint" "TestPoint:TestPoint_Pad_1.0x1.0mm"
-			(at 228.6 95.25 0)
-			(effects
-				(font
-					(size 1.27 1.27)
-				)
-				(hide yes)
-			)
-		)
-		(property "Datasheet" "~"
-			(at 228.6 95.25 0)
-			(effects
-				(font
-					(size 1.27 1.27)
-				)
-				(hide yes)
-			)
-		)
-		(property "Description" "test point"
-			(at 228.6 90.17 0)
-			(effects
-				(font
-					(size 1.27 1.27)
-				)
-				(hide yes)
-			)
-		)
-		(property "Manufactuerer" ""
-			(at 228.6 90.17 90)
-			(effects
-				(font
-					(size 1.27 1.27)
-				)
-				(hide yes)
-			)
-		)
-		(pin "1"
-		)
-		(instances
-			(project "BPS-Leader"
-				(path "/fb37da34-e420-4994-8cc1-079e8c0fa48e/282b6fe6-adb7-4bd1-bb3c-4f7b240441d9"
-					(reference "TP12")
-					(unit 1)
-				)
-			)
 		)
 	)

Commit message: RevB layout completed
Parts:
- TP11: value TestPoint -> HV-Sns
- TP9: value TestPoint -> HV-Ctrl
Changed lines of the file:
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@@
 			)
 		)
-		(property "Value" "TestPoint"
+		(property "Value" "HV-Sns"
 			(at 191.516 94.488 0)
 			(effects
@@
 			)
 		)
-		(property "Value" "TestPoint"
+		(property "Value" "HV-Ctrl"
 			(at 76.2 103.124 90)
 			(effects

Commit message: JLC Production Files
Parts:
- C16: LCSC (none) -> C15849
- C17: LCSC (none) -> C14663
- D31: renamed from HV-1; value LED -> HV-; LCSC (none) -> C84263
- D6: LCSC (none) -> C6326606
- Q4, Q5: LCSC (none) -> C67272
- R30, R33, R36, R37: LCSC (none) -> C25804
- R32: LCSC (none) -> C2907165
- R34: LCSC (none) -> C21190
Changed lines of the file:
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@@
+			)
+		)
+		(property "LCSC" "C2907165"
+			(at 88.9 76.835 0)
+			(effects
+				(font
+					(size 1.27 1.27)
+				)
+				(hide yes)
 			)
 		)
@@
 			)
 		)
+		(property "LCSC" "C15849"
+			(at 183.515 105.4099 0)
+			(effects
+				(font
+					(size 1.27 1.27)
+				)
+				(hide yes)
+			)
+		)
 		(pin "2"
 		)
@@
 		(dnp no)
 		(fields_autoplaced yes)
-		(property "Reference" "HV-1"
+		(property "Reference" "D31"
 			(at 85.09 89.2174 90)
 			(effects
@@
 			)
 		)
-		(property "Value" "LED"
+		(property "Value" "HV-"
 			(at 85.09 91.7574 90)
 			(effects
@@
 			)
 		)
+		(property "LCSC" "C84263"
+			(at 85.09 89.2174 0)
+			(effects
+				(font
+					(size 1.27 1.27)
+				)
+				(hide yes)
+			)
+		)
 		(pin "1"
 		)
@@
 			(project "BPS-Leader"
 				(path "/fb37da34-e420-4994-8cc1-079e8c0fa48e/282b6fe6-adb7-4bd1-bb3c-4f7b240441d9"
-					(reference "HV-1")
+					(reference "D31")
 					(unit 1)
 				)
@@
 			)
 		)
+		(property "LCSC" "C25804"
+			(at 198.12 105.4099 0)
+			(effects
+				(font
+					(size 1.27 1.27)
+				)
+				(hide yes)
+			)
+		)
 		(pin "2"
 		)
@@
 			)
 		)
+		(property "LCSC" "C25804"
+			(at 235.966 91.948 0)
+			(effects
+				(font
+					(size 1.27 1.27)
+				)
+				(hide yes)
+			)
+		)
 		(pin "2"
 		)
@@
 		(property "Description" "5.3A Id, 30V Vds, 27mOhm Rds, N-Channel HEXFET Power MOSFET, SOT-23"
 			(at 93.98 104.14 0)
+			(effects
+				(font
+					(size 1.27 1.27)
+				)
+				(hide yes)
+			)
+		)
+		(property "LCSC" "C67272"
+			(at 100.838 106.426 0)
 			(effects
 				(font
@@
 			)
 		)
+		(property "LCSC" "C25804"
+			(at 228.092 99.314 0)
+			(effects
+				(font
+					(size 1.27 1.27)
+				)
+				(hide yes)
+			)
+		)
 		(pin "2"
 		)
@@
 			)
 		)
+		(property "LCSC" "C14663"
+			(at 214.63 101.6001 0)
+			(effects
+				(font
+					(size 1.27 1.27)
+				)
+				(hide yes)
+			)
+		)
 		(pin "1"
 		)
@@
 			)
 		)
+		(property "LCSC" "C25804"
+			(at 86.36 109.2199 0)
+			(effects
+				(font
+					(size 1.27 1.27)
+				)
+				(hide yes)
+			)
+		)
 		(pin "2"
 		)
@@
 		(property "P/N" "VSSAF522-M3/H"
 			(at 96.52 88.9 90)
+			(effects
+				(font
+					(size 1.27 1.27)
+				)
+				(hide yes)
+			)
+		)
+		(property "LCSC" "C6326606"
+			(at 99.06 86.36 0)
 			(effects
 				(font
@@
 			)
 		)
+		(property "LCSC" "C67272"
+			(at 203.454 96.266 0)
+			(effects
+				(font
+					(size 1.27 1.27)
+				)
+				(hide yes)
+			)
+		)
 		(pin "1"
 		)
@@
 			(effects
 				(font
+					(size 1.27 1.27)
+				)
+				(hide yes)
+			)
+		)
+		(property "LCSC" "C21190"
+			(at 220.726 91.948 0)
+			(effects
+				(font

Commit message: condensed custom lirbraries
Parts:
- D6: footprint VSSAF522-M3/H:SODFL5226X100N -> CustomKiCad-Library:SODFL5226X100N
Changed lines of the file:
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@@
 			)
 		)
-		(property "Footprint" "VSSAF522-M3/H:SODFL5226X100N"
+		(property "Footprint" "CustomKiCad-Library:SODFL5226X100N"
 			(at 92.075 88.9 0)
 			(effects

Commit message: JLCPCB ouput files
Parts:
- R34: P/N CRCW060310K0FKEI -> CRCW06031K00FKEI
