File: Hardware/POWER.kicad_sch (KiCad schematic)
At the start: 16 parts, among them IC1 LM74502HDDFR, Q12 NVMFWS1D7N04XMT1G, Q13 NVMFWS1D7N04XMT1G

Commit message: JLCPCB ouput files
Parts:
- R28: P/N CRCW060310K0FKEI -> CRCW060310K0FKEI
- R83: P/N CRCW060310K0FKEI -> CRCW06034K30FKEA
