File: hardware/Array_Precharge_Contactor.kicad_sch (KiCad schematic)
At the start: 15 parts

Commit message: 🗿
Parts:
- removed C?: 1u, Capacitor_SMD:C_0603_1608Metric_Pad1.08x0.95mm_HandSolder, symbol Device:C
- removed C?: 0.1u, Capacitor_SMD:C_0603_1608Metric_Pad1.08x0.95mm_HandSolder, symbol Device:C
- removed D?: Contact, LED_SMD:LED_0603_1608Metric, symbol Device:LED
- removed D?: VSSAF522-M3/H, CustomKiCad-Library:SODFL5226X100N, symbol Diode:C3D25170H
- removed J?: ContactorConnector, UTSVT_Connectors:Molex_Nano-Fit_105309-xx04_1x04_P2.50mm_Vertical, symbol UTSVT_Connectors:ContactorConnector
- removed Q? (x2): IRLML0030, Package_TO_SOT_SMD:SOT-23, symbol Transistor_FET:IRLML0030
- removed R? (x4): 10k, symbol Device:R
- removed R?: 1k, symbol Device:R
- removed R?: 4.3k, symbol Device:R
- removed TP?: ctrl, TestPoint:TestPoint_Pad_1.0x1.0mm, symbol Connector:TestPoint
- removed TP?: Sense, TestPoint:TestPoint_Pad_1.0x1.0mm, symbol Connector:TestPoint
- added C?: 0.1u, Capacitor_SMD:C_0603_1608Metric_Pad1.08x0.95mm_HandSolder, symbol Device:C
- added C?: 1u, Capacitor_SMD:C_0603_1608Metric_Pad1.08x0.95mm_HandSolder, symbol Device:C
- added D?: Contact, LED_SMD:LED_0603_1608Metric, symbol Device:LED
- added D?: VSSAF522-M3/H, CustomKiCad-Library:SODFL5226X100N, symbol Diode:C3D25170H
- added J?: ContactorConnector, UTSVT_Connectors:Molex_Nano-Fit_105309-xx04_1x04_P2.50mm_Vertical, symbol UTSVT_Connectors:ContactorConnector
- added Q? (x2): IRLML0030, Package_TO_SOT_SMD:SOT-23, symbol Transistor_FET:IRLML0030
- added R? (x4): 10k, symbol Device:R
- added R?: 1k, symbol Device:R
- added R?: 4.3k, symbol Device:R
- added TP?: Sense, TestPoint:TestPoint_Pad_1.0x1.0mm, symbol Connector:TestPoint
- added TP?: ctrl, TestPoint:TestPoint_Pad_1.0x1.0mm, symbol Connector:TestPoint
Connections:
- net +24V: now also J?.1 (Con+(24V)), J?.4 (Sense+(24V))
- net 3.3V: now also Q?.3 (D)
- net CONTACTOR+: now also D?.1 (K), R?.2
- net CONTROL: now also Q?.1 (G), R?.2, TP?.1
- net GND: now also C?.1, C?.1, Q?.2 (S), R?.1, R?.1, R?.1
- net HV_CONTROL: now also D?.1 (K), D?.2 (A), J?.2 (Con-), Q?.3 (D)
- net SENSE: now also C?.2, Q?.2 (S), R?.2, TP?.1
- new net: C?.2, Q?.1 (G), R?.2
- new net: R?.1, R?.1, R?.2
- new net: J?.3 (Sense-), R?.2
- new net: D?.2 (A), R?.1
