File: hardware/Power_PD_Boost.kicad_sch (KiCad schematic)
At the start: 28 parts, among them IC1 TPS55340PWP

Commit message: 🗿
Parts:
- R32: renamed from R6; symbol Device:R_US -> Device:R
- R33: renamed from R7; symbol Device:R_US -> Device:R
- R36: renamed from R4; symbol Device:R_US -> Device:R
- R37: renamed from R5; symbol Device:R_US -> Device:R
- R38: renamed from R3; symbol Device:R_US -> Device:R
- R39: renamed from R1; symbol Device:R_US -> Device:R
- R40: renamed from R2; symbol Device:R_US -> Device:R
- renumbered C1 to C27, C2 to C28, C3 to C29, C6 to C30, C5 to C33, C4 to C34, C7 to C35, C8 to C36, C9 to C37, C10 to C38, C11 to C39, D2 to D10, IC1 to IC3, L1 to L2, TP7 to TP3, TP8 to TP4, TP4 to TP7
