File: hardware/PS-BPSLeader.kicad_sch (KiCad schematic)
At the start: 7 parts, among them J3 CAN_NANO_01x05, J4 CAN_NANO_01x05, J6 USB_C_Receptacle_USB2.0_16P, J7 CAN_DEBUG_NANO_01x04, J8 CarCANConnector, J9 Conn_02x06_Counter_Clockwise

Commit message: why is everything weird
Other:
- sheet ESTOP ports: added ESTOP_1+, ESTOP_1-/2+, ESTOP_1_SENSE, ESTOP_2-, ESTOP_2_SENSE, ESTOP_3_SENSE, ESTOP_OUT; removed none
- sheet Peripherals ports: added BPS_CAN_H, BPS_CAN_L, CAR_CAN_H, CAR_CAN_L, ESTOP_1_SENSE, ESTOP_2_SENSE, ESTOP_3_SENSE, MCU_3V3, MCU_USB_D+, MCU_USB_D-; removed none
