File: hardware/PS-BPSLeader.kicad_sch (KiCad schematic)
At the start: 7 parts, among them J3 CAN_NANO_01x05, J4 CAN_NANO_01x05, J6 USB_C_Receptacle_USB2.0_16P, J7 CAN_DEBUG_NANO_01x04, J8 CarCANConnector, J9 Conn_02x06_Counter_Clockwise

Commit message: interview tabling
Other:
- note added: "Export Deutsch"
- note removed: "Export MX150"
