File: hardware/ESP32_Power_Mux.kicad_sch (KiCad schematic)
At the start: 6 parts, among them U1 TPS2117DRLR

Commit message: finished schematic except for 12v buck boost
Parts:
- renumbered C1 to C50, C2 to C51, C3 to C52, C4 to C53, R1 to R84, U1 to U11
Changed lines of the file:
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@@
 		(in_pos_files yes)
 		(dnp no)
-		(property "Reference" "C4"
+		(property "Reference" "C53"
 			(at 91.8972 57.2516 0)
 			(show_name no)
@@
 			(project "PS-BPSLeader"
 				(path "/d4a4ed4f-0983-4aef-b212-0e3284ab3963/5da56964-fa04-4fec-bdfe-c6acfeda5c9a/c396b043-4a62-4d2b-b629-091a6c3457ae"
-					(reference "C4")
+					(reference "C53")
 					(unit 1)
 				)
@@
 		(in_pos_files yes)
 		(dnp no)
-		(property "Reference" "R1"
+		(property "Reference" "R84"
 			(at 78.994 67.564 0)
 			(show_name no)
@@
 			(project "PS-BPSLeader"
 				(path "/d4a4ed4f-0983-4aef-b212-0e3284ab3963/5da56964-fa04-4fec-bdfe-c6acfeda5c9a/c396b043-4a62-4d2b-b629-091a6c3457ae"
-					(reference "R1")
+					(reference "R84")
 					(unit 1)
 				)
@@
 		(in_pos_files yes)
 		(dnp no)
-		(property "Reference" "C1"
+		(property "Reference" "C50"
 			(at 24.5872 44.5516 0)
 			(show_name no)
@@
 			(project "PS-BPSLeader"
 				(path "/d4a4ed4f-0983-4aef-b212-0e3284ab3963/5da56964-fa04-4fec-bdfe-c6acfeda5c9a/c396b043-4a62-4d2b-b629-091a6c3457ae"
-					(reference "C1")
+					(reference "C50")
 					(unit 1)
 				)
@@
 		(dnp no)
 		(fields_autoplaced yes)
-		(property "Reference" "U1"
+		(property "Reference" "U11"
 			(at 60.96 44.45 0)
 			(show_name no)
@@
 			(project "PS-BPSLeader"
 				(path "/d4a4ed4f-0983-4aef-b212-0e3284ab3963/5da56964-fa04-4fec-bdfe-c6acfeda5c9a/c396b043-4a62-4d2b-b629-091a6c3457ae"
-					(reference "U1")
+					(reference "U11")
 					(unit 1)
 				)
@@
 		(in_pos_files yes)
 		(dnp no)
-		(property "Reference" "C3"
+		(property "Reference" "C52"
 			(at 42.3672 67.4116 0)
 			(show_name no)
@@
 			(project "PS-BPSLeader"
 				(path "/d4a4ed4f-0983-4aef-b212-0e3284ab3963/5da56964-fa04-4fec-bdfe-c6acfeda5c9a/c396b043-4a62-4d2b-b629-091a6c3457ae"
-					(reference "C3")
+					(reference "C52")
 					(unit 1)
 				)
@@
 		(in_pos_files yes)
 		(dnp no)
-		(property "Reference" "C2"
+		(property "Reference" "C51"
 			(at 38.5572 44.5516 0)
 			(show_name no)
@@
 			(project "PS-BPSLeader"
 				(path "/d4a4ed4f-0983-4aef-b212-0e3284ab3963/5da56964-fa04-4fec-bdfe-c6acfeda5c9a/c396b043-4a62-4d2b-b629-091a6c3457ae"
-					(reference "C2")
-					(unit 1)
-				)
+					(reference "C51")
+					(unit 1)
+				)

Commit message: added 12V buck boost
Parts:
- renumbered C50 to C51, C51 to C52, C52 to C53, C53 to C54, R84 to R88
Changed lines of the file:
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@@
 		(in_pos_files yes)
 		(dnp no)
-		(property "Reference" "C53"
+		(property "Reference" "C54"
 			(at 91.8972 57.2516 0)
 			(show_name no)
@@
 			(project "PS-BPSLeader"
 				(path "/d4a4ed4f-0983-4aef-b212-0e3284ab3963/5da56964-fa04-4fec-bdfe-c6acfeda5c9a/c396b043-4a62-4d2b-b629-091a6c3457ae"
-					(reference "C53")
+					(reference "C54")
 					(unit 1)
 				)
@@
 		(in_pos_files yes)
 		(dnp no)
-		(property "Reference" "R84"
+		(property "Reference" "R88"
 			(at 78.994 67.564 0)
 			(show_name no)
@@
 			(project "PS-BPSLeader"
 				(path "/d4a4ed4f-0983-4aef-b212-0e3284ab3963/5da56964-fa04-4fec-bdfe-c6acfeda5c9a/c396b043-4a62-4d2b-b629-091a6c3457ae"
-					(reference "R84")
+					(reference "R88")
 					(unit 1)
 				)
@@
 		(in_pos_files yes)
 		(dnp no)
-		(property "Reference" "C50"
+		(property "Reference" "C51"
 			(at 24.5872 44.5516 0)
 			(show_name no)
@@
 			(project "PS-BPSLeader"
 				(path "/d4a4ed4f-0983-4aef-b212-0e3284ab3963/5da56964-fa04-4fec-bdfe-c6acfeda5c9a/c396b043-4a62-4d2b-b629-091a6c3457ae"
-					(reference "C50")
+					(reference "C51")
 					(unit 1)
 				)
@@
 		(in_pos_files yes)
 		(dnp no)
-		(property "Reference" "C52"
+		(property "Reference" "C53"
 			(at 42.3672 67.4116 0)
 			(show_name no)
@@
 			(project "PS-BPSLeader"
 				(path "/d4a4ed4f-0983-4aef-b212-0e3284ab3963/5da56964-fa04-4fec-bdfe-c6acfeda5c9a/c396b043-4a62-4d2b-b629-091a6c3457ae"
-					(reference "C52")
+					(reference "C53")
 					(unit 1)
 				)
@@
 		(in_pos_files yes)
 		(dnp no)
-		(property "Reference" "C51"
+		(property "Reference" "C52"
 			(at 38.5572 44.5516 0)
 			(show_name no)
@@
 			(project "PS-BPSLeader"
 				(path "/d4a4ed4f-0983-4aef-b212-0e3284ab3963/5da56964-fa04-4fec-bdfe-c6acfeda5c9a/c396b043-4a62-4d2b-b629-091a6c3457ae"
-					(reference "C51")
-					(unit 1)
-				)
+					(reference "C52")
+					(unit 1)
+				)
