File: hardware/PS-BPSLeader.kicad_pcb (KiCad board)
At the start: 2 copper layers, 0 parts

Commit message: finished schematic except for 12v buck boost
Parts:
- added C1: 26p, Capacitor_SMD:C_0603_1608Metric_Pad1.08x0.95mm_HandSolder, F.Cu at (111.8, 109.4)
- added C10: 0.1u, Capacitor_SMD:C_0603_1608Metric_Pad1.08x0.95mm_HandSolder, F.Cu at (112.4, 95.1)
- added C11: 1u, Capacitor_SMD:C_0603_1608Metric_Pad1.08x0.95mm_HandSolder, F.Cu at (112.4, 97.6)
- added C12: 0.1u, Capacitor_SMD:C_0603_1608Metric_Pad1.08x0.95mm_HandSolder, F.Cu at (112.4, 100.1)
- added C13: 0.1u, Capacitor_SMD:C_0603_1608Metric_Pad1.08x0.95mm_HandSolder, F.Cu at (112.4, 102.6)
- added C14: 0.1u, Capacitor_SMD:C_0603_1608Metric_Pad1.08x0.95mm_HandSolder, F.Cu at (112.4, 105.1)
- added C15: 10u, Capacitor_SMD:C_0805_2012Metric_Pad1.18x1.45mm_HandSolder, F.Cu at (149.5, 72.0)
- added C16: 0.1u, Capacitor_SMD:C_0603_1608Metric_Pad1.08x0.95mm_HandSolder, F.Cu at (140.3, 65.2)
- added C17: 0.1u, Capacitor_SMD:C_0603_1608Metric_Pad1.08x0.95mm_HandSolder, F.Cu at (140.3, 67.7)
- added C18: 0.1u, Capacitor_SMD:C_0603_1608Metric_Pad1.08x0.95mm_HandSolder, F.Cu at (140.3, 70.2)
- added C19: 10u, Capacitor_SMD:C_0805_2012Metric_Pad1.18x1.45mm_HandSolder, F.Cu at (167.3, 73.0)
- added C2: 26p, Capacitor_SMD:C_0603_1608Metric_Pad1.08x0.95mm_HandSolder, F.Cu at (111.8, 112.9)
- added C20: 0.1u, Capacitor_SMD:C_0603_1608Metric_Pad1.08x0.95mm_HandSolder, F.Cu at (158.1, 66.2)
- added C21: 0.1u, Capacitor_SMD:C_0603_1608Metric_Pad1.08x0.95mm_HandSolder, F.Cu at (158.1, 68.7)
- added C22: 0.1u, Capacitor_SMD:C_0603_1608Metric_Pad1.08x0.95mm_HandSolder, F.Cu at (158.1, 71.2)
- added C23: 10uF, Capacitor_SMD:C_0805_2012Metric_Pad1.18x1.45mm_HandSolder, F.Cu at (158.5, 137.7)
- added C24: 10uF, Capacitor_SMD:C_0805_2012Metric_Pad1.18x1.45mm_HandSolder, F.Cu at (158.5, 140.7)
- added C25: 0.1uF, Capacitor_SMD:C_0603_1608Metric_Pad1.08x0.95mm_HandSolder, F.Cu at (131.5, 152.7)
- added C26: 0.1uF, Capacitor_SMD:C_0603_1608Metric_Pad1.08x0.95mm_HandSolder, F.Cu at (131.5, 155.2)
- added C27: 4.7u, Capacitor_SMD:C_0805_2012Metric_Pad1.18x1.45mm_HandSolder, F.Cu at (55.4, 140.3)
- added C28: 1u, Capacitor_SMD:C_0603_1608Metric_Pad1.08x0.95mm_HandSolder, F.Cu at (50.1, 120.7)
- added C29: 4.7u, Capacitor_SMD:C_0805_2012Metric_Pad1.18x1.45mm_HandSolder, F.Cu at (55.4, 143.3)
- added C3: 10u, Capacitor_SMD:C_0805_2012Metric_Pad1.18x1.45mm_HandSolder, F.Cu at (135.9, 121.8)
- added C30: 0.1n, Capacitor_SMD:C_0603_1608Metric_Pad1.08x0.95mm_HandSolder, F.Cu at (50.1, 123.2)
- added C31: 1u, Capacitor_SMD:C_0603_1608Metric_Pad1.08x0.95mm_HandSolder, F.Cu at (50.1, 125.7)
- added C32: 0.1u, Capacitor_SMD:C_0603_1608Metric_Pad1.08x0.95mm_HandSolder, F.Cu at (50.1, 128.3)
- added C33: 1u, Capacitor_SMD:C_0603_1608Metric_Pad1.08x0.95mm_HandSolder, B.Cu at (128.7, 87.6)
- added C34: 4.7u, Capacitor_SMD:C_0805_2012Metric_Pad1.18x1.45mm_HandSolder, F.Cu at (55.2, 90.2)
- added C35: 1u, Capacitor_SMD:C_0603_1608Metric_Pad1.08x0.95mm_HandSolder, F.Cu at (49.9, 70.6)
- added C36: 4.7u, Capacitor_SMD:C_0805_2012Metric_Pad1.18x1.45mm_HandSolder, F.Cu at (55.2, 93.2)
- added C37: 0.1n, Capacitor_SMD:C_0603_1608Metric_Pad1.08x0.95mm_HandSolder, F.Cu at (49.9, 73.1)
- added C38: 1u, Capacitor_SMD:C_0603_1608Metric_Pad1.08x0.95mm_HandSolder, F.Cu at (49.9, 75.6)
- added C39: 0.1u, Capacitor_SMD:C_0603_1608Metric_Pad1.08x0.95mm_HandSolder, F.Cu at (49.9, 78.2)
- added C4: 0.1u, Capacitor_SMD:C_0603_1608Metric_Pad1.08x0.95mm_HandSolder, F.Cu at (144.6, 101.2)
- added C40: 4.7u, Capacitor_SMD:C_0805_2012Metric_Pad1.18x1.45mm_HandSolder, F.Cu at (55.3, 115.4)
- added C41: 1u, Capacitor_SMD:C_0603_1608Metric_Pad1.08x0.95mm_HandSolder, F.Cu at (50.0, 95.9)
- added C42: 4.7u, Capacitor_SMD:C_0603_1608Metric_Pad1.08x0.95mm_HandSolder, F.Cu at (50.0, 98.4)
- added C43: 0.1n, Capacitor_SMD:C_0603_1608Metric_Pad1.08x0.95mm_HandSolder, F.Cu at (50.0, 100.9)
- added C44: 1u, Capacitor_SMD:C_0603_1608Metric_Pad1.08x0.95mm_HandSolder, F.Cu at (50.0, 103.4)
- added C45: 0.1u, Capacitor_SMD:C_0603_1608Metric_Pad1.08x0.95mm_HandSolder, F.Cu at (50.0, 105.9)
- added C46: 1u, Capacitor_SMD:C_0603_1608Metric_Pad1.08x0.95mm_HandSolder, F.Cu at (43.5, 63.4)
- added C47: 1u, Capacitor_SMD:C_0603_1608Metric_Pad1.08x0.95mm_HandSolder, F.Cu at (46.0, 63.4)
- added C48: 10u, Capacitor_SMD:C_0805_2012Metric_Pad1.18x1.45mm_HandSolder, F.Cu at (143.2, 133.1)
- added C49: 10u, Capacitor_SMD:C_0805_2012Metric_Pad1.18x1.45mm_HandSolder, F.Cu at (143.2, 136.1)
- added C5: 0.1u, Capacitor_SMD:C_0603_1608Metric_Pad1.08x0.95mm_HandSolder, F.Cu at (144.6, 103.7)
- added C50: 0.1uF, Capacitor_SMD:C_0603_1608Metric_Pad1.08x0.95mm_HandSolder, F.Cu at (171.8, 127.2)
- added C51: 0.1uF, Capacitor_SMD:C_0603_1608Metric_Pad1.08x0.95mm_HandSolder, F.Cu at (169.3, 127.2)
- added C52: 0.1uF, Capacitor_SMD:C_0603_1608Metric_Pad1.08x0.95mm_HandSolder, F.Cu at (166.8, 127.2)
- added C53: 0.1uF, Capacitor_SMD:C_0603_1608Metric_Pad1.08x0.95mm_HandSolder, F.Cu at (164.2, 127.2)
- added C54: 4.7u, Capacitor_SMD:C_0805_2012Metric_Pad1.18x1.45mm_HandSolder, B.Cu at (127.6, 108.4)
- added C55: 100n, Capacitor_SMD:C_0805_2012Metric_Pad1.18x1.45mm_HandSolder, B.Cu at (127.6, 105.4)
- added C56: 100n, Capacitor_SMD:C_0603_1608Metric_Pad1.08x0.95mm_HandSolder, B.Cu at (123.0, 108.7)
- added C57: 47u, Capacitor_SMD:C_1210_3225Metric_Pad1.33x2.70mm_HandSolder, B.Cu at (133.0, 107.8)
- added C58: 10uF, Capacitor_SMD:C_0805_2012Metric_Pad1.18x1.45mm_HandSolder, B.Cu at (146.2, 91.9)
- added C59: 1uF, Capacitor_SMD:C_0603_1608Metric_Pad1.08x0.95mm_HandSolder, B.Cu at (139.7, 112.2)
- added C6: 0.1u, Capacitor_SMD:C_0603_1608Metric_Pad1.08x0.95mm_HandSolder, F.Cu at (144.6, 106.2)
- added C60: 1uF, Capacitor_SMD:C_0603_1608Metric_Pad1.08x0.95mm_HandSolder, B.Cu at (139.7, 109.7)
- added C61: 1uF, Capacitor_SMD:C_0603_1608Metric_Pad1.08x0.95mm_HandSolder, B.Cu at (139.7, 107.2)
- added C62: 1uF, Capacitor_SMD:C_0603_1608Metric_Pad1.08x0.95mm_HandSolder, B.Cu at (139.7, 104.7)
- added C63: 1uF, Capacitor_SMD:C_0603_1608Metric_Pad1.08x0.95mm_HandSolder, B.Cu at (139.7, 102.2)
- added C64: 1uF, Capacitor_SMD:C_0603_1608Metric_Pad1.08x0.95mm_HandSolder, B.Cu at (139.7, 99.7)
- added C65: 0.1uF, Capacitor_SMD:C_0603_1608Metric_Pad1.08x0.95mm_HandSolder, B.Cu at (139.7, 97.1)
- added C66: 0.1uF, Capacitor_SMD:C_0603_1608Metric_Pad1.08x0.95mm_HandSolder, B.Cu at (139.7, 94.6)
- added C67: 0.1u, Capacitor_SMD:C_0603_1608Metric_Pad1.08x0.95mm_HandSolder, F.Cu at (92.7, 119.5)
- added C68: 0.22u, Capacitor_SMD:C_0603_1608Metric_Pad1.08x0.95mm_HandSolder, F.Cu at (83.8, 124.2)
- added C69: 0.22u, Capacitor_SMD:C_0603_1608Metric_Pad1.08x0.95mm_HandSolder, F.Cu at (83.8, 126.7)
- added C7: 0.1u, Capacitor_SMD:C_0603_1608Metric_Pad1.08x0.95mm_HandSolder, F.Cu at (104.5, 125.7)
- added C70: 0.1u, Capacitor_SMD:C_0603_1608Metric_Pad1.08x0.95mm_HandSolder, F.Cu at (83.8, 129.2)
- added C71: 100pF, Capacitor_SMD:C_0603_1608Metric_Pad1.08x0.95mm_HandSolder, F.Cu at (84.4, 151.3)
- added C72: 100pF, Capacitor_SMD:C_0603_1608Metric_Pad1.08x0.95mm_HandSolder, F.Cu at (84.4, 148.0)
- added C73: 100pF, Capacitor_SMD:C_0603_1608Metric_Pad1.08x0.95mm_HandSolder, F.Cu at (101.9, 150.3)
- added C74: 100pF, Capacitor_SMD:C_0603_1608Metric_Pad1.08x0.95mm_HandSolder, F.Cu at (101.9, 146.9)
- added C75: 100pF, Capacitor_SMD:C_0603_1608Metric_Pad1.08x0.95mm_HandSolder, F.Cu at (101.9, 143.6)
- added C76: 100pF, Capacitor_SMD:C_0603_1608Metric_Pad1.08x0.95mm_HandSolder, F.Cu at (84.4, 144.6)
- added C77: 0.1u, Capacitor_SMD:C_0603_1608Metric_Pad1.08x0.95mm_HandSolder, B.Cu at (105.6, 71.3)
- added C78: 1u, Capacitor_SMD:C_0603_1608Metric_Pad1.08x0.95mm_HandSolder, B.Cu at (105.6, 68.7)
- added C79: 220n, Capacitor_SMD:C_0603_1608Metric_Pad1.08x0.95mm_HandSolder, B.Cu at (105.6, 66.2)
- added C8: 0.1u, Capacitor_SMD:C_0603_1608Metric_Pad1.08x0.95mm_HandSolder, F.Cu at (144.6, 111.2)
- added C80: 10n, Capacitor_SMD:C_0603_1608Metric_Pad1.08x0.95mm_HandSolder, B.Cu at (105.6, 63.7)
- added C81: 10u, Capacitor_SMD:C_0805_2012Metric_Pad1.18x1.45mm_HandSolder, B.Cu at (101.8, 80.1)
- added C82: 0.1u, Capacitor_SMD:C_0603_1608Metric_Pad1.08x0.95mm_HandSolder, B.Cu at (110.0, 71.3)
- added C83: 0.1u, Capacitor_SMD:C_0603_1608Metric_Pad1.08x0.95mm_HandSolder, B.Cu at (110.0, 68.7)
- added C84: 0.1uF, Capacitor_SMD:C_0603_1608Metric_Pad1.08x0.95mm_HandSolder, B.Cu at (148.5, 123.9)
- added C85: 0.1uF, Capacitor_SMD:C_0603_1608Metric_Pad1.08x0.95mm_HandSolder, B.Cu at (146.0, 123.9)
- added C86: 0.1uF, Capacitor_SMD:C_0603_1608Metric_Pad1.08x0.95mm_HandSolder, B.Cu at (143.5, 123.9)
- added C87: 0.1uF, Capacitor_SMD:C_0603_1608Metric_Pad1.08x0.95mm_HandSolder, B.Cu at (141.0, 123.9)
- added C88: 10u, Capacitor_SMD:C_0805_2012Metric_Pad1.18x1.45mm_HandSolder, B.Cu at (132.1, 134.6)
- added C89: 10u, Capacitor_SMD:C_0805_2012Metric_Pad1.18x1.45mm_HandSolder, B.Cu at (132.1, 131.5)
- added C9: 1u, Capacitor_SMD:C_0603_1608Metric_Pad1.08x0.95mm_HandSolder, F.Cu at (144.6, 113.8)
- added C90: 1u, Capacitor_SMD:C_0603_1608Metric_Pad1.08x0.95mm_HandSolder, B.Cu at (133.8, 98.1)
- added C91: 10u, Capacitor_SMD:C_0805_2012Metric_Pad1.18x1.45mm_HandSolder, F.Cu at (132.5, 72.2)
- added C92: 0.1u, Capacitor_SMD:C_0603_1608Metric_Pad1.08x0.95mm_HandSolder, F.Cu at (123.3, 65.3)
- added C93: 0.1u, Capacitor_SMD:C_0603_1608Metric_Pad1.08x0.95mm_HandSolder, F.Cu at (123.3, 67.9)
- added C94: 0.1u, Capacitor_SMD:C_0603_1608Metric_Pad1.08x0.95mm_HandSolder, F.Cu at (123.3, 70.4)
- added CR1: D5V0P4UR6SO-7, LHRS_ICs:D5V0P4UR6SO-7, F.Cu at (115.3, 143.0)
- added D1: TPD2EUSB30DRTR, LHRS_ICs:TPD2EUSB30DRTR, F.Cu at (160.3, 101.2)
- added D10: ESP_LED1, LED_SMD:LED_0603_1608Metric_Pad1.05x0.95mm_HandSolder, F.Cu at (153.9, 140.1)
- added D11: ESP_LED2, LED_SMD:LED_0603_1608Metric_Pad1.05x0.95mm_HandSolder, F.Cu at (153.9, 142.7)
- added D12: VSSAF522-M3/H, LHRS_Passives:SODFL5226X100N, F.Cu at (43.1, 137.4)
- added D13: Contact, LED_SMD:LED_0603_1608Metric_Pad1.05x0.95mm_HandSolder, F.Cu at (60.0, 140.1)
- added D14: VSSAF522-M3/H, LHRS_Passives:SODFL5226X100N, F.Cu at (43.1, 141.5)
- added D15: VSSAF522-M3/H, LHRS_Passives:SODFL5226X100N, F.Cu at (42.9, 87.3)
- added D16: Contact, LED_SMD:LED_0603_1608Metric_Pad1.05x0.95mm_HandSolder, F.Cu at (59.8, 90.0)
- added D17: VSSAF522-M3/H, LHRS_Passives:SODFL5226X100N, F.Cu at (42.9, 91.4)
- added D18: VSSAF522-M3/H, LHRS_Passives:SODFL5226X100N, F.Cu at (43.0, 112.6)
- added D19: Contact, LED_SMD:LED_0603_1608Metric_Pad1.05x0.95mm_HandSolder, F.Cu at (59.9, 115.2)
- added D2: TVS, Diode_SMD:D_SOD-323, F.Cu at (114.2, 130.0)
- added D20: VSSAF522-M3/H, LHRS_Passives:SODFL5226X100N, F.Cu at (43.0, 116.7)
- added D21: VSSAF522-M3/H, LHRS_Passives:SODFL5226X100N, F.Cu at (57.3, 57.7)
- added D22: VSSAF522-M3/H, LHRS_Passives:SODFL5226X100N, F.Cu at (61.3, 57.7)
- added D23: SBA130CH-AU_R1_000A1, Diode_SMD:D_SOD-323_HandSoldering, F.Cu at (148.2, 133.1)
- added D24: SMBJ24A-E3_52, Diode_SMD:D_SMB, B.Cu at (159.4, 94.7)
- added D25: SMBJ10A-E3_52, Diode_SMD:D_SMB, B.Cu at (159.4, 89.1)
- added D26: SMBJ10A-E3_52, Diode_SMD:D_SMB, B.Cu at (159.4, 83.6)
- added D27: FAULT, LED_SMD:LED_0603_1608Metric_Pad1.05x0.95mm_HandSolder, B.Cu at (146.0, 89.1)
- added D28: SMBJ15CA, Diode_SMD:D_SMB, B.Cu at (107.7, 59.7)
- added D29: SMAF4758A, LHRS_Passives:SODFL5026X125N, B.Cu at (107.1, 54.8)
- added D3: RGB_LED, LHRS_Special:RGB_LED, F.Cu at (114.1, 117.7)
- added D30: SBA130CH-AU_R1_000A1, Diode_SMD:D_SOD-323_HandSoldering, B.Cu at (137.1, 134.6)
- added D31: CDSOT23-T24CAN, LHRS_Passives:CDSOT23-T24CAN, F.Cu at (132.5, 75.9)
- added D4: LED, LED_SMD:LED_0603_1608Metric_Pad1.05x0.95mm_HandSolder, F.Cu at (118.7, 127.2)
- added D5: CDSOT23-T24CAN, LHRS_Passives:CDSOT23-T24CAN, F.Cu at (149.5, 75.8)
- added D6: CDSOT23-T24CAN, LHRS_Passives:CDSOT23-T24CAN, F.Cu at (167.3, 76.8)
- added D7: 1N5819HW-7-F, Diode_SMD:D_SOD-123, F.Cu at (154.6, 151.9)
- added D8: SP0503BAHT, Package_TO_SOT_SMD:SOT-143, F.Cu at (159.9, 159.9)
- added D9: ESP_PWR, LED_SMD:LED_0603_1608Metric_Pad1.05x0.95mm_HandSolder, F.Cu at (153.9, 137.5)
- added ESTOP1: LED, LED_SMD:LED_0603_1608Metric_Pad1.05x0.95mm_HandSolder, F.Cu at (85.9, 54.5)
- added ESTOP2: LED, LED_SMD:LED_0603_1608Metric_Pad1.05x0.95mm_HandSolder, F.Cu at (88.5, 54.5)
- added ESTOP3: LED, LED_SMD:LED_0603_1608Metric_Pad1.05x0.95mm_HandSolder, F.Cu at (91.1, 54.5)
- added E_JP1: Jumper_2_Open, Connector_PinHeader_2.54mm:PinHeader_1x02_P2.54mm_Vertical, F.Cu at (69.7, 69.8)
- added E_JP2: Jumper_2_Open, Connector_PinHeader_2.54mm:PinHeader_1x02_P2.54mm_Vertical, F.Cu at (69.7, 65.2)
- added E_JP3: Jumper_2_Open, Connector_PinHeader_2.54mm:PinHeader_1x02_P2.54mm_Vertical, F.Cu at (69.7, 60.6)
- added F1: 5A, LHRS_Power:Fuse-3557-2, F.Cu at (97.8, 60.7)
- added F2: 5A, LHRS_Power:Fuse-3557-2, F.Cu at (159.8, 84.8)
- added FAN1: Conn_01x04, Connector_Molex:Molex_Nano-Fit_105309-xx04_1x04_P2.50mm_Vertical, F.Cu at (45.0, 55.6)
- added FAN2: Conn_01x04, Connector_Molex:Molex_Nano-Fit_105309-xx04_1x04_P2.50mm_Vertical, F.Cu at (45.0, 47.2)
- added FB1: FerriteBead, Inductor_SMD:L_0805_2012Metric_Pad1.05x1.20mm_HandSolder, F.Cu at (130.2, 121.7)
- added FB2: FerriteBead, Inductor_SMD:L_0805_2012Metric_Pad1.05x1.20mm_HandSolder, F.Cu at (133.0, 121.7)
- added IC1: TCAN3413DR, LHRS_Passives:TCAN3413DR, F.Cu at (146.8, 67.2)
- added IC2: TCAN3413DR, LHRS_Passives:TCAN3413DR, F.Cu at (164.6, 68.2)
- added IC3: CYPD3177-24LQXQ, LHRS_ICs:CYPD3177-24LQXQ, B.Cu at (140.7, 90.2)
- added IC4: BQ79600PWRQ1, LHRS_ICs:SOP65P640X120-16N, F.Cu at (90.8, 124.0)
- added IC5: LM74502DDFR, LHRS_Power:LM74502DDFR, B.Cu at (113.4, 54.7)
- added IC6: TCAN3413DR, LHRS_Passives:TCAN3413DR, F.Cu at (129.7, 67.4)
- added J1: USB_C_Receptacle_USB2.0_16P, LHRS_Connectors:USB_C_Receptacle_GCT_USB4105-xx-A_16P_TopMnt_Horizontal, F.Cu at (169.1, 101.7)
- added J10: Low SIde Conn, LHRS_Connectors:Molex_Nano-Fit_105309-xx02_1x02_P2.50mm_Vertical, F.Cu at (80.4, 166.6)
- added J11: SWD_Header, LHRS_Connectors:SWD_Conn, F.Cu at (125.9, 83.1)
- added J12: SWD, Connector_PinHeader_2.54mm:PinHeader_1x04_P2.54mm_Vertical, F.Cu at (122.2, 90.9)
- added J13: USB_C_Receptacle_USB2.0_16P, LHRS_Connectors:USB_C_Receptacle_GCT_USB4105-xx-A_16P_TopMnt_Horizontal, F.Cu at (160.0, 172.3)
- added J14: Conn_01x02, LHRS_Connectors:Molex_Nano-Fit_105309-xx02_1x02_P2.50mm_Vertical, F.Cu at (79.1, 45.0)
- added J15: Contactor Connector, LHRS_Connectors:Molex_Nano-Fit_105309-xx04_1x04_P2.50mm_Vertical, F.Cu at (44.9, 126.8)
- added J16: Contactor Connector, LHRS_Connectors:Molex_Nano-Fit_105309-xx04_1x04_P2.50mm_Vertical, F.Cu at (44.7, 76.7)
- added J17: Contactor Connector, LHRS_Connectors:Molex_Nano-Fit_105309-xx04_1x04_P2.50mm_Vertical, F.Cu at (44.8, 102.0)
- added J18: Micro_SD_Card_Det, Connector_Card:microSD_HC_Hirose_DM3AT-SF-PEJM5, F.Cu at (116.7, 157.9)
- added J2: CAN_DEBUG_NANO_01x04, LHRS_Connectors:Molex_Nano-Fit_105309-xx04_1x04_P2.50mm_Vertical, F.Cu at (161.2, 59.7)
- added J3: CAN_NANO_01x05, LHRS_Connectors:Molex_Nano-Fit_105309-xx05_1x05_P2.50mm_Vertical, F.Cu at (157.4, 45.1)
- added J4: Conn_02x06_Counter_Clockwise, Connector_Molex:Molex_Nano-Fit_105310-xx12_2x06_P2.50mm_Vertical, F.Cu at (100.0, 46.8)
- added J5: CAN_NANO_01x03, LHRS_Connectors:Molex_Nano-Fit_105309-xx03_1x03_P2.50mm_Vertical, F.Cu at (141.6, 44.4)
- added J6: CAN_NANO_01x03, LHRS_Connectors:Molex_Nano-Fit_105309-xx03_1x03_P2.50mm_Vertical, F.Cu at (143.1, 57.0)
- added J7: CAN_DEBUG_NANO_01x04, LHRS_Connectors:Molex_Nano-Fit_105309-xx04_1x04_P2.50mm_Vertical, F.Cu at (127.5, 58.4)
- added J8: CAN_NANO_01x03, LHRS_Connectors:Molex_Nano-Fit_105309-xx03_1x03_P2.50mm_Vertical, F.Cu at (125.6, 44.2)
- added J9: High Side Conn, LHRS_Connectors:Molex_Nano-Fit_105309-xx02_1x02_P2.50mm_Vertical, F.Cu at (92.0, 165.4)
- added JP1: TRM, Connector_PinHeader_2.54mm:PinHeader_1x02_P2.54mm_Vertical, F.Cu at (144.8, 72.8)
- added JP2: TRM, Connector_PinHeader_2.54mm:PinHeader_1x02_P2.54mm_Vertical, F.Cu at (162.6, 73.8)
- added JP3: TRM, Connector_PinHeader_2.54mm:PinHeader_1x02_P2.54mm_Vertical, F.Cu at (127.8, 72.9)
- added L1: 8.2u, LHRS_Passives:SRN8040-150M, B.Cu at (127.2, 115.6)
- added Q1: SQ2315CES-T1_GE3, Package_TO_SOT_SMD:TSOT-23-6_HandSoldering, F.Cu at (76.9, 68.6)
- added Q10: SI7997DP-T1-GE3, LHRS_ICs:SI7997DP-T1-GE3, B.Cu at (157.0, 109.5)
- added Q11: SI7997DP-T1-GE3, LHRS_ICs:SI7997DP-T1-GE3, B.Cu at (157.0, 101.5)
- added Q12: IRLML0030, Package_TO_SOT_SMD:SOT-23, B.Cu at (140.0, 84.8)
- added Q13: PSMN012-100YS, Package_TO_SOT_SMD:LFPAK56, B.Cu at (113.2, 78.5)
- added Q14: PSMN012-100YS, Package_TO_SOT_SMD:LFPAK56, B.Cu at (106.6, 78.5)
- added Q2: SQ2315CES-T1_GE3, Package_TO_SOT_SMD:TSOT-23-6_HandSoldering, F.Cu at (81.5, 68.6)
- added Q3: SQ2315CES-T1_GE3, Package_TO_SOT_SMD:TSOT-23-6_HandSoldering, F.Cu at (86.1, 68.6)
- added Q4: IRLML0030, Package_TO_SOT_SMD:SOT-23, F.Cu at (63.5, 121.7)
- added Q5: IRLML0030, Package_TO_SOT_SMD:SOT-23, F.Cu at (63.5, 126.1)
- added Q6: IRLML0030, Package_TO_SOT_SMD:SOT-23, F.Cu at (63.2, 71.6)
- added Q7: IRLML0030, Package_TO_SOT_SMD:SOT-23, F.Cu at (63.2, 76.0)
- added Q8: IRLML0030, Package_TO_SOT_SMD:SOT-23, F.Cu at (63.3, 96.8)
- added Q9: IRLML0030, Package_TO_SOT_SMD:SOT-23, F.Cu at (63.3, 101.3)
- added R1: 0, Resistor_SMD:R_0603_1608Metric_Pad0.98x0.95mm_HandSolder, F.Cu at (153.9, 51.7)
- added R10: 1k, Resistor_SMD:R_0603_1608Metric_Pad0.98x0.95mm_HandSolder, F.Cu at (116.7, 95.1)
- added R100: 4.7k, Resistor_SMD:R_0603_1608Metric_Pad0.98x0.95mm_HandSolder, B.Cu at (148.4, 104.7)
- added R101: 2.2k, Resistor_SMD:R_0603_1608Metric_Pad0.98x0.95mm_HandSolder, B.Cu at (148.4, 102.2)
- added R102: 2.2k, Resistor_SMD:R_0603_1608Metric_Pad0.98x0.95mm_HandSolder, B.Cu at (148.4, 99.7)
- added R103: 1k, Resistor_SMD:R_0603_1608Metric_Pad0.98x0.95mm_HandSolder, B.Cu at (148.4, 97.1)
- added R104: 10k, Resistor_SMD:R_0603_1608Metric_Pad0.98x0.95mm_HandSolder, F.Cu at (92.7, 129.5)
- added R105: 10k, Resistor_SMD:R_0603_1608Metric_Pad0.98x0.95mm_HandSolder, F.Cu at (97.0, 119.5)
- added R106: 100k, Resistor_SMD:R_0603_1608Metric_Pad0.98x0.95mm_HandSolder, F.Cu at (97.0, 122.0)
- added R107: 100k, Resistor_SMD:R_0603_1608Metric_Pad0.98x0.95mm_HandSolder, F.Cu at (97.0, 124.5)
- added R108: 10, Resistor_SMD:R_0603_1608Metric_Pad0.98x0.95mm_HandSolder, F.Cu at (88.2, 129.2)
- added R109: 1k, Resistor_SMD:R_0603_1608Metric_Pad0.98x0.95mm_HandSolder, F.Cu at (83.8, 138.4)
- added R11: 1k, Resistor_SMD:R_0603_1608Metric_Pad0.98x0.95mm_HandSolder, F.Cu at (116.7, 97.6)
- added R110: 1k, Resistor_SMD:R_0603_1608Metric_Pad0.98x0.95mm_HandSolder, F.Cu at (101.6, 139.7)
- added R111: 51, Resistor_SMD:R_0603_1608Metric_Pad0.98x0.95mm_HandSolder, F.Cu at (79.1, 141.5)
- added R112: 51, Resistor_SMD:R_0603_1608Metric_Pad0.98x0.95mm_HandSolder, F.Cu at (79.1, 139.0)
- added R113: 51, Resistor_SMD:R_0603_1608Metric_Pad0.98x0.95mm_HandSolder, F.Cu at (97.3, 139.7)
- added R114: 51, Resistor_SMD:R_0603_1608Metric_Pad0.98x0.95mm_HandSolder, F.Cu at (97.3, 137.2)
- added R115: 10k, Resistor_SMD:R_0603_1608Metric_Pad0.98x0.95mm_HandSolder, B.Cu at (110.0, 66.2)
- added R116: 33, Resistor_SMD:R_0603_1608Metric_Pad0.98x0.95mm_HandSolder, B.Cu at (110.0, 63.7)
- added R117: 100k, Resistor_SMD:R_0603_1608Metric_Pad0.98x0.95mm_HandSolder, B.Cu at (114.3, 71.3)
- added R118: 7.32k, Resistor_SMD:R_0603_1608Metric_Pad0.98x0.95mm_HandSolder, B.Cu at (114.3, 68.7)
- added R119: 100k, Resistor_SMD:R_0603_1608Metric_Pad0.98x0.95mm_HandSolder, B.Cu at (114.3, 66.2)
- added R12: 1k, Resistor_SMD:R_0603_1608Metric_Pad0.98x0.95mm_HandSolder, F.Cu at (116.7, 100.1)
- added R120: 15.8k, Resistor_SMD:R_0603_1608Metric_Pad0.98x0.95mm_HandSolder, B.Cu at (114.3, 63.7)
- added R121: 10k, Resistor_SMD:R_0603_1608Metric_Pad0.98x0.95mm_HandSolder, B.Cu at (138.5, 123.9)
- added R122: 57.6k, Resistor_SMD:R_0603_1608Metric_Pad0.98x0.95mm_HandSolder, B.Cu at (131.3, 98.1)
- added R123: 5k, Resistor_SMD:R_0603_1608Metric_Pad0.98x0.95mm_HandSolder, B.Cu at (128.8, 98.1)
- added R124: 57.6k, Resistor_SMD:R_0603_1608Metric_Pad0.98x0.95mm_HandSolder, B.Cu at (126.3, 98.1)
- added R125: 5k, Resistor_SMD:R_0603_1608Metric_Pad0.98x0.95mm_HandSolder, B.Cu at (123.8, 98.1)
- added R126: 26.1k, Resistor_SMD:R_0603_1608Metric_Pad0.98x0.95mm_HandSolder, B.Cu at (121.3, 98.1)
- added R127: 5k, Resistor_SMD:R_0603_1608Metric_Pad0.98x0.95mm_HandSolder, B.Cu at (118.8, 98.1)
- added R128: 57.6k, Resistor_SMD:R_0603_1608Metric_Pad0.98x0.95mm_HandSolder, B.Cu at (116.3, 98.1)
- added R129: 5k, Resistor_SMD:R_0603_1608Metric_Pad0.98x0.95mm_HandSolder, B.Cu at (113.8, 98.1)
- added R13: 10k, Resistor_SMD:R_0603_1608Metric_Pad0.98x0.95mm_HandSolder, F.Cu at (114.0, 123.3)
- added R130: 22.1k, Resistor_SMD:R_0603_1608Metric_Pad0.98x0.95mm_HandSolder, B.Cu at (111.2, 98.1)
- added R131: 60, Resistor_SMD:R_0603_1608Metric_Pad0.98x0.95mm_HandSolder, F.Cu at (123.3, 72.9)
- added R132: 60, Resistor_SMD:R_0603_1608Metric_Pad0.98x0.95mm_HandSolder, F.Cu at (123.3, 75.4)
- added R14: 1k, Resistor_SMD:R_0603_1608Metric_Pad0.98x0.95mm_HandSolder, F.Cu at (114.0, 125.8)
- added R15: 60, Resistor_SMD:R_0603_1608Metric_Pad0.98x0.95mm_HandSolder, F.Cu at (140.3, 72.7)
- added R16: 60, Resistor_SMD:R_0603_1608Metric_Pad0.98x0.95mm_HandSolder, F.Cu at (140.3, 75.2)
- added R17: 60, Resistor_SMD:R_0603_1608Metric_Pad0.98x0.95mm_HandSolder, F.Cu at (158.1, 73.7)
- added R18: 60, Resistor_SMD:R_0603_1608Metric_Pad0.98x0.95mm_HandSolder, F.Cu at (158.1, 76.2)
- added R19: 5.1k, Resistor_SMD:R_0603_1608Metric_Pad0.98x0.95mm_HandSolder, F.Cu at (131.5, 157.7)
- added R2: 0, Resistor_SMD:R_0603_1608Metric_Pad0.98x0.95mm_HandSolder, F.Cu at (153.9, 54.3)
- added R20: 5.1k, Resistor_SMD:R_0603_1608Metric_Pad0.98x0.95mm_HandSolder, F.Cu at (131.5, 160.2)
- added R21: 10k, Resistor_SMD:R_0603_1608Metric_Pad0.98x0.95mm_HandSolder, F.Cu at (131.5, 162.7)
- added R22: 10k, Resistor_SMD:R_0603_1608Metric_Pad0.98x0.95mm_HandSolder, F.Cu at (131.5, 165.2)
- added R23: 10k, Resistor_SMD:R_0603_1608Metric_Pad0.98x0.95mm_HandSolder, F.Cu at (131.5, 167.7)
- added R24: 1k, Resistor_SMD:R_0603_1608Metric_Pad0.98x0.95mm_HandSolder, F.Cu at (131.5, 170.2)
- added R25: 1k, Resistor_SMD:R_0603_1608Metric_Pad0.98x0.95mm_HandSolder, F.Cu at (131.5, 172.8)
- added R26: 1k, Resistor_SMD:R_0603_1608Metric_Pad0.98x0.95mm_HandSolder, F.Cu at (131.5, 175.3)
- added R27: 10k, Resistor_SMD:R_0603_1608Metric_Pad0.98x0.95mm_HandSolder, F.Cu at (75.8, 62.9)
- added R28: 10k, Resistor_SMD:R_0603_1608Metric_Pad0.98x0.95mm_HandSolder, F.Cu at (78.4, 62.9)
- added R29: 10k, Resistor_SMD:R_0603_1608Metric_Pad0.98x0.95mm_HandSolder, F.Cu at (80.9, 62.9)
- added R3: 16k, Resistor_SMD:R_0603_1608Metric_Pad0.98x0.95mm_HandSolder, B.Cu at (141.2, 119.2)
- added R30: 470, Resistor_SMD:R_0603_1608Metric_Pad0.98x0.95mm_HandSolder, F.Cu at (83.4, 62.9)
- added R31: 470, Resistor_SMD:R_0603_1608Metric_Pad0.98x0.95mm_HandSolder, F.Cu at (75.8, 58.6)
- added R32: 470, Resistor_SMD:R_0603_1608Metric_Pad0.98x0.95mm_HandSolder, F.Cu at (78.4, 58.6)
- added R33: 10k, Resistor_SMD:R_0603_1608Metric_Pad0.98x0.95mm_HandSolder, F.Cu at (80.9, 58.6)
- added R34: 10k, Resistor_SMD:R_0603_1608Metric_Pad0.98x0.95mm_HandSolder, F.Cu at (83.4, 58.6)
- added R35: 10k, Resistor_SMD:R_0603_1608Metric_Pad0.98x0.95mm_HandSolder, F.Cu at (75.8, 54.2)
- added R36: 33k, Resistor_SMD:R_0603_1608Metric_Pad0.98x0.95mm_HandSolder, F.Cu at (78.4, 54.2)
- added R37: 33k, Resistor_SMD:R_0603_1608Metric_Pad0.98x0.95mm_HandSolder, F.Cu at (80.9, 54.2)
- added R38: 33k, Resistor_SMD:R_0603_1608Metric_Pad0.98x0.95mm_HandSolder, F.Cu at (83.4, 54.2)
- added R39: 66.67k, Resistor_SMD:R_0603_1608Metric_Pad0.98x0.95mm_HandSolder, F.Cu at (50.1, 130.8)
- added R4: 4.7k, Resistor_SMD:R_0603_1608Metric_Pad0.98x0.95mm_HandSolder, B.Cu at (144.9, 118.8)
- added R40: 0, Resistor_SMD:R_0603_1608Metric_Pad0.98x0.95mm_HandSolder, F.Cu at (54.5, 120.7)
- added R41: 1k, Resistor_SMD:R_0603_1608Metric_Pad0.98x0.95mm_HandSolder, F.Cu at (54.5, 123.2)
- added R42: 120k, Resistor_SMD:R_0603_1608Metric_Pad0.98x0.95mm_HandSolder, F.Cu at (54.5, 125.7)
- added R43: 10k, Resistor_SMD:R_0603_1608Metric_Pad0.98x0.95mm_HandSolder, F.Cu at (54.5, 128.3)
- added R44: 4.3k, Resistor_SMD:R_0603_1608Metric_Pad0.98x0.95mm_HandSolder, F.Cu at (54.5, 130.8)
- added R45: 1, Resistor_SMD:R_0603_1608Metric_Pad0.98x0.95mm_HandSolder, F.Cu at (58.8, 120.7)
- added R46: 1k, Resistor_SMD:R_0603_1608Metric_Pad0.98x0.95mm_HandSolder, F.Cu at (58.8, 123.2)
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
Commit message: added 12V buck boost
Parts:
- added C1: 7.5n, Capacitor_SMD:C_0603_1608Metric_Pad1.08x0.95mm_HandSolder, F.Cu at (31.4, 15.3)
- added C100: 0.1u, Capacitor_SMD:C_0603_1608Metric_Pad1.08x0.95mm_HandSolder, F.Cu at (25.1, 17.8)
- added C101: 22u, Capacitor_SMD:C_1206_3216Metric, F.Cu at (20.1, 19.0)
- added C102: 22u, Capacitor_SMD:C_1206_3216Metric, F.Cu at (20.1, 22.4)
- added C103: 22u, Capacitor_SMD:C_1206_3216Metric, F.Cu at (20.1, 25.7)
- added C104: 45p, Capacitor_SMD:C_0603_1608Metric_Pad1.08x0.95mm_HandSolder, F.Cu at (25.1, 20.3)
- added C105: 22u, Capacitor_SMD:C_1206_3216Metric, F.Cu at (20.1, 29.1)
- added C106: 90n, Capacitor_SMD:C_0603_1608Metric_Pad1.08x0.95mm_HandSolder, F.Cu at (25.1, 22.8)
- added C107: 0.1u, Capacitor_SMD:C_0603_1608Metric_Pad1.08x0.95mm_HandSolder, F.Cu at (25.1, 25.3)
- added C16: 10u, Capacitor_SMD:C_0805_2012Metric_Pad1.18x1.45mm_HandSolder, F.Cu at (-27.6, 129.3)
- added C17: 0.1u, Capacitor_SMD:C_0603_1608Metric_Pad1.08x0.95mm_HandSolder, F.Cu at (-36.7, 129.1)
- added C18: 0.1u, Capacitor_SMD:C_0603_1608Metric_Pad1.08x0.95mm_HandSolder, F.Cu at (-36.7, 131.6)
- added C19: 0.1u, Capacitor_SMD:C_0603_1608Metric_Pad1.08x0.95mm_HandSolder, F.Cu at (37.8, 15.3)
- added C20: 10u, Capacitor_SMD:C_0805_2012Metric_Pad1.18x1.45mm_HandSolder, F.Cu at (-4.89, 133.1)
- added C21: 0.1u, Capacitor_SMD:C_0603_1608Metric_Pad1.08x0.95mm_HandSolder, F.Cu at (-14.1, 121.6)
- added C22: 0.1u, Capacitor_SMD:C_0603_1608Metric_Pad1.08x0.95mm_HandSolder, F.Cu at (-14.1, 124.1)
- added C23: 0.1u, Capacitor_SMD:C_0603_1608Metric_Pad1.08x0.95mm_HandSolder, F.Cu at (37.8, 19.8)
- added C28: 4.7u, Capacitor_SMD:C_0805_2012Metric_Pad1.18x1.45mm_HandSolder, F.Cu at (-51.4, 119.4)
- added C29: 1u, Capacitor_SMD:C_0603_1608Metric_Pad1.08x0.95mm_HandSolder, F.Cu at (-56.7, 99.8)
- added C30: 4.7u, Capacitor_SMD:C_0805_2012Metric_Pad1.18x1.45mm_HandSolder, F.Cu at (-51.4, 122.4)
- added C31: 0.1n, Capacitor_SMD:C_0603_1608Metric_Pad1.08x0.95mm_HandSolder, F.Cu at (-56.7, 102.3)
- added C32: 1u, Capacitor_SMD:C_0603_1608Metric_Pad1.08x0.95mm_HandSolder, F.Cu at (-56.7, 104.9)
- added C33: 0.1u, Capacitor_SMD:C_0603_1608Metric_Pad1.08x0.95mm_HandSolder, F.Cu at (-56.7, 107.4)
- added C35: 4.7u, Capacitor_SMD:C_0805_2012Metric_Pad1.18x1.45mm_HandSolder, F.Cu at (-23.1, 92.1)
- added C36: 1u, Capacitor_SMD:C_0603_1608Metric_Pad1.08x0.95mm_HandSolder, F.Cu at (-28.3, 72.5)
- added C37: 4.7u, Capacitor_SMD:C_0805_2012Metric_Pad1.18x1.45mm_HandSolder, F.Cu at (-23.1, 95.1)
- added C38: 0.1n, Capacitor_SMD:C_0603_1608Metric_Pad1.08x0.95mm_HandSolder, F.Cu at (-28.3, 75.0)
- added C39: 1u, Capacitor_SMD:C_0603_1608Metric_Pad1.08x0.95mm_HandSolder, F.Cu at (-28.3, 77.5)
- added C40: 0.1u, Capacitor_SMD:C_0603_1608Metric_Pad1.08x0.95mm_HandSolder, F.Cu at (-28.3, 80.0)
- added C41: 4.7u, Capacitor_SMD:C_0805_2012Metric_Pad1.18x1.45mm_HandSolder, F.Cu at (-51.4, 92.1)
- added C42: 1u, Capacitor_SMD:C_0603_1608Metric_Pad1.08x0.95mm_HandSolder, F.Cu at (-56.7, 72.5)
- added C43: 4.7u, Capacitor_SMD:C_0805_2012Metric_Pad1.18x1.45mm_HandSolder, F.Cu at (-51.4, 95.1)
- added C44: 0.1n, Capacitor_SMD:C_0603_1608Metric_Pad1.08x0.95mm_HandSolder, F.Cu at (-56.7, 75.0)
- added C45: 1u, Capacitor_SMD:C_0603_1608Metric_Pad1.08x0.95mm_HandSolder, F.Cu at (-56.7, 77.5)
- added C46: 0.1u, Capacitor_SMD:C_0603_1608Metric_Pad1.08x0.95mm_HandSolder, F.Cu at (-56.7, 80.0)
- added C55: 4.7u, Capacitor_SMD:C_0805_2012Metric_Pad1.18x1.45mm_HandSolder, F.Cu at (-21.4, 117.4)
- added C56: 100n, Capacitor_SMD:C_0603_1608Metric_Pad1.08x0.95mm_HandSolder, F.Cu at (-27.7, 117.2)
- added C57: 100n, Capacitor_SMD:C_0603_1608Metric_Pad1.08x0.95mm_HandSolder, F.Cu at (-31.8, 113.0)
- added C58: 47u, Capacitor_SMD:C_1210_3225Metric_Pad1.33x2.70mm_HandSolder, F.Cu at (-26.8, 113.9)
- added C95: 0.1u, Capacitor_SMD:C_0603_1608Metric_Pad1.08x0.95mm_HandSolder, F.Cu at (37.8, 24.3)
- added C96: 0.1u, Capacitor_SMD:C_0603_1608Metric_Pad1.08x0.95mm_HandSolder, F.Cu at (25.1, 15.3)
- added C97: 22u, Capacitor_SMD:C_1206_3216Metric, F.Cu at (20.1, 15.7)
- added C98: 4.7u, Capacitor_SMD:C_0805_2012Metric_Pad1.18x1.45mm_HandSolder, F.Cu at (19.7, 36.5)
- added C99: 0.1u, Capacitor_SMD:C_0603_1608Metric_Pad1.08x0.95mm_HandSolder, F.Cu at (-3.52, 115.1)
- added D12: VSSAF522-M3/H, LHRS_Passives:SODFL5226X100N, F.Cu at (-63.7, 116.6)
- added D13: Contact, LED_SMD:LED_0603_1608Metric_Pad1.05x0.95mm_HandSolder, F.Cu at (-46.8, 119.2)
- added D14: VSSAF522-M3/H, LHRS_Passives:SODFL5226X100N, F.Cu at (-63.7, 120.6)
- added D15: VSSAF522-M3/H, LHRS_Passives:SODFL5226X100N, F.Cu at (-35.3, 89.2)
- added D17: VSSAF522-M3/H, LHRS_Passives:SODFL5226X100N, F.Cu at (-35.3, 93.3)
- added D18: VSSAF522-M3/H, LHRS_Passives:SODFL5226X100N, F.Cu at (-63.7, 89.2)
- added D19: Contact, LED_SMD:LED_0603_1608Metric_Pad1.05x0.95mm_HandSolder, F.Cu at (-46.8, 91.9)
- added D2: LED, LED_SMD:LED_0603_1608Metric, F.Cu at (-8.51, 85.8)
- added D20: VSSAF522-M3/H, LHRS_Passives:SODFL5226X100N, F.Cu at (-63.7, 93.3)
- added D3: LED, LED_SMD:LED_0603_1608Metric, F.Cu at (-8.51, 88.4)
- added IC1: TCAN3413DR, LHRS_Passives:TCAN3413DR, F.Cu at (-34.6, 124.5)
- added IC2: TCAN3413DR, LHRS_Passives:TCAN3413DR, F.Cu at (-7.64, 123.6)
- added IC6: TCAN3413DR, LHRS_Passives:TCAN3413DR, F.Cu at (-6.30, 74.5)
- added IC7: TPS552872RYQR, LHRS_ICs:TPS552892QWRYQRQ1, F.Cu at (-12.0, 115.0)
- added J15: Contactor Connector, LHRS_Connectors:Molex_Nano-Fit_105309-xx04_1x04_P2.50mm_Vertical, F.Cu at (-61.9, 105.9)
- added J16: Contactor Connector, LHRS_Connectors:Molex_Nano-Fit_105309-xx04_1x04_P2.50mm_Vertical, F.Cu at (-33.5, 78.6)
- added J17: Contactor Connector, LHRS_Connectors:Molex_Nano-Fit_105309-xx04_1x04_P2.50mm_Vertical, F.Cu at (-61.9, 78.6)
- added JP1: TRM, Connector_PinHeader_2.54mm:PinHeader_1x02_P2.54mm_Vertical, F.Cu at (-32.3, 130.1)
- added JP2: TRM, Connector_PinHeader_2.54mm:PinHeader_1x02_P2.54mm_Vertical, F.Cu at (-9.60, 129.2)
- added L1: 8.2u, LHRS_Passives:74439369082, F.Cu at (-27.8, 105.2)
- added L2: 4.7u, LHRS_Passives:74439369082, F.Cu at (-10.2, 105.2)
- added Q4: IRLML0030, Package_TO_SOT_SMD:SOT-23, F.Cu at (-43.4, 100.8)
- added Q5: IRLML0030, Package_TO_SOT_SMD:SOT-23, F.Cu at (-43.4, 105.3)
- added Q6: IRLML0030, Package_TO_SOT_SMD:SOT-23, F.Cu at (-15.0, 73.5)
- added Q7: IRLML0030, Package_TO_SOT_SMD:SOT-23, F.Cu at (-15.0, 77.9)
- added Q8: IRLML0030, Package_TO_SOT_SMD:SOT-23, F.Cu at (-43.4, 73.5)
- added Q9: IRLML0030, Package_TO_SOT_SMD:SOT-23, F.Cu at (-43.4, 77.9)
- added R137: 50k, Resistor_SMD:R_0603_1608Metric_Pad0.98x0.95mm_HandSolder, F.Cu at (25.1, 27.8)
- added R139: 1.455k, Resistor_SMD:R_0603_1608Metric_Pad0.98x0.95mm_HandSolder, F.Cu at (25.1, 30.3)
- added R140: 12.5m, Resistor_SMD:R_1210_3225Metric, F.Cu at (20.1, 32.9)
- added R141: 100k, Resistor_SMD:R_0603_1608Metric_Pad0.98x0.95mm_HandSolder, F.Cu at (25.1, 32.8)
- added R142: 11.1k, Resistor_SMD:R_0603_1608Metric_Pad0.98x0.95mm_HandSolder, F.Cu at (25.1, 35.3)
- added R20: 60, Resistor_SMD:R_0603_1608Metric_Pad0.98x0.95mm_HandSolder, F.Cu at (-36.7, 134.1)
- added R21: 60, Resistor_SMD:R_0603_1608Metric_Pad0.98x0.95mm_HandSolder, F.Cu at (-14.1, 126.6)
- added R22: 60, Resistor_SMD:R_0603_1608Metric_Pad0.98x0.95mm_HandSolder, F.Cu at (-14.1, 129.1)
- added R3: 30.1k, Resistor_SMD:R_0603_1608Metric_Pad0.98x0.95mm_HandSolder, F.Cu at (31.4, 17.8)
- added R4: 5k, Resistor_SMD:R_0603_1608Metric_Pad0.98x0.95mm_HandSolder, F.Cu at (31.4, 20.3)
- added R43: 66.67k, Resistor_SMD:R_0603_1608Metric_Pad0.98x0.95mm_HandSolder, F.Cu at (-56.7, 109.9)
- added R44: 0, Resistor_SMD:R_0603_1608Metric_Pad0.98x0.95mm_HandSolder, F.Cu at (-52.3, 99.8)
- added R45: 1k, Resistor_SMD:R_0603_1608Metric_Pad0.98x0.95mm_HandSolder, F.Cu at (-52.3, 102.3)
- added R46: 120k, Resistor_SMD:R_0603_1608Metric_Pad0.98x0.95mm_HandSolder, F.Cu at (-52.3, 104.9)
- added R47: 10k, Resistor_SMD:R_0603_1608Metric_Pad0.98x0.95mm_HandSolder, F.Cu at (-52.3, 107.4)
- added R48: 4.3k, Resistor_SMD:R_0603_1608Metric_Pad0.98x0.95mm_HandSolder, F.Cu at (-52.3, 109.9)
- added R49: 1, Resistor_SMD:R_0603_1608Metric_Pad0.98x0.95mm_HandSolder, F.Cu at (-48.0, 99.8)
- added R5: 1k, Resistor_SMD:R_0603_1608Metric_Pad0.98x0.95mm_HandSolder, F.Cu at (31.4, 22.8)
- added R50: 1k, Resistor_SMD:R_0603_1608Metric_Pad0.98x0.95mm_HandSolder, F.Cu at (-48.0, 102.3)
- added R51: 10k, Resistor_SMD:R_0603_1608Metric_Pad0.98x0.95mm_HandSolder, F.Cu at (-48.0, 104.9)
- added R52: 10k, Resistor_SMD:R_0603_1608Metric_Pad0.98x0.95mm_HandSolder, F.Cu at (-48.0, 107.4)
- added R6: 1k, Resistor_SMD:R_0603_1608Metric_Pad0.98x0.95mm_HandSolder, F.Cu at (31.4, 25.3)
- added R62: 66.67k, Resistor_SMD:R_0603_1608Metric_Pad0.98x0.95mm_HandSolder, F.Cu at (-28.3, 82.5)
- added R63: 0, Resistor_SMD:R_0603_1608Metric_Pad0.98x0.95mm_HandSolder, F.Cu at (-24.0, 72.5)
- added R64: 1k, Resistor_SMD:R_0603_1608Metric_Pad0.98x0.95mm_HandSolder, F.Cu at (-24.0, 75.0)
- added R66: 10k, Resistor_SMD:R_0603_1608Metric_Pad0.98x0.95mm_HandSolder, F.Cu at (-24.0, 77.5)
- added R67: 4.3k, Resistor_SMD:R_0603_1608Metric_Pad0.98x0.95mm_HandSolder, F.Cu at (-24.0, 80.0)
- added R68: 1, Resistor_SMD:R_0603_1608Metric_Pad0.98x0.95mm_HandSolder, F.Cu at (-24.0, 82.5)
- added R69: 1k, Resistor_SMD:R_0603_1608Metric_Pad0.98x0.95mm_HandSolder, F.Cu at (-19.6, 72.5)
- added R70: 10k, Resistor_SMD:R_0603_1608Metric_Pad0.98x0.95mm_HandSolder, F.Cu at (-19.6, 75.0)
- added R71: 10k, Resistor_SMD:R_0603_1608Metric_Pad0.98x0.95mm_HandSolder, F.Cu at (-19.6, 77.5)
- added R72: 66.67k, Resistor_SMD:R_0603_1608Metric_Pad0.98x0.95mm_HandSolder, F.Cu at (-56.7, 82.5)
- added R73: 0, Resistor_SMD:R_0603_1608Metric_Pad0.98x0.95mm_HandSolder, F.Cu at (-52.3, 72.5)
- added R74: 1k, Resistor_SMD:R_0603_1608Metric_Pad0.98x0.95mm_HandSolder, F.Cu at (-52.3, 75.0)
- added R75: 120k, Resistor_SMD:R_0603_1608Metric_Pad0.98x0.95mm_HandSolder, F.Cu at (-52.3, 77.5)
- added R76: 10k, Resistor_SMD:R_0603_1608Metric_Pad0.98x0.95mm_HandSolder, F.Cu at (-52.3, 80.0)
- added R77: 4.3k, Resistor_SMD:R_0603_1608Metric_Pad0.98x0.95mm_HandSolder, F.Cu at (-52.3, 82.5)
- added R78: 1, Resistor_SMD:R_0603_1608Metric_Pad0.98x0.95mm_HandSolder, F.Cu at (-48.0, 72.5)
- added R79: 1k, Resistor_SMD:R_0603_1608Metric_Pad0.98x0.95mm_HandSolder, F.Cu at (-48.0, 75.0)
- added R80: 10k, Resistor_SMD:R_0603_1608Metric_Pad0.98x0.95mm_HandSolder, F.Cu at (-48.0, 77.5)
- added R81: 10k, Resistor_SMD:R_0603_1608Metric_Pad0.98x0.95mm_HandSolder, F.Cu at (-48.0, 80.0)
- added R89: 100k, Resistor_SMD:R_0603_1608Metric, F.Cu at (-31.8, 115.5)
- added R90: 19.1k, Resistor_SMD:R_0603_1608Metric, F.Cu at (-31.8, 118.0)
- added TP10: Sense, TestPoint:TestPoint_Loop_D1.80mm_Drill1.0mm_Beaded, F.Cu at (-56.3, 91.4)
- added TP11: V_in_12V, TestPoint:TestPoint_Loop_D1.80mm_Drill1.0mm_Beaded, F.Cu at (-36.4, 101.1)
- added TP12: CB, TestPoint:TestPoint_Loop_D1.80mm_Drill1.0mm_Beaded, F.Cu at (-36.4, 106.2)
- added TP13: FB, TestPoint:TestPoint_Loop_D1.80mm_Drill1.0mm_Beaded, F.Cu at (-36.4, 111.2)
- added TP14: SW, TestPoint:TestPoint_Loop_D1.80mm_Drill1.0mm_Beaded, F.Cu at (-36.4, 116.3)
- added TP5: ctrl, TestPoint:TestPoint_Loop_D1.80mm_Drill1.0mm_Beaded, F.Cu at (-56.3, 113.7)
- added TP6: Sense, TestPoint:TestPoint_Loop_D1.80mm_Drill1.0mm_Beaded, F.Cu at (-56.3, 118.7)
- added TP7: ctrl, TestPoint:TestPoint_Loop_D1.80mm_Drill1.0mm_Beaded, F.Cu at (-28.0, 86.3)
- added TP8: Sense, TestPoint:TestPoint_Loop_D1.80mm_Drill1.0mm_Beaded, F.Cu at (-28.0, 91.4)
- added TP9: ctrl, TestPoint:TestPoint_Loop_D1.80mm_Drill1.0mm_Beaded, F.Cu at (-56.3, 86.3)
- added U12: LMR51635XDDCR, LHRS_ICs:DDC0006A-MFG, F.Cu at (-20.6, 113.8)
- added U18: CDSOT23-T24CAN, LHRS_ICs:CDSOT23-T24CAN, F.Cu at (-8.07, 80.2)
- added U2: CDSOT23-T24CAN, LHRS_ICs:CDSOT23-T24CAN, F.Cu at (-27.9, 123.7)
- added U3: CDSOT23-T24CAN, LHRS_ICs:CDSOT23-T24CAN, F.Cu at (-4.83, 129.3)
- added U5: DRV110APWR, LHRS_ICs:PW14_TEX, F.Cu at (-49.3, 114.5)
- added U7: DRV110APWR, LHRS_ICs:PW14_TEX, F.Cu at (-21.0, 87.2)
- added U8: DRV110APWR, LHRS_ICs:PW14_TEX, F.Cu at (-49.3, 87.2)
- TP1: renamed from TP3; footprint TestPoint:TestPoint_Loop_D2.50mm_Drill1.0mm -> TestPoint:TestPoint_Loop_D1.80mm_Drill1.0mm_Beaded
- TP20: footprint TestPoint:TestPoint_Pad_1.0x1.0mm -> TestPoint:TestPoint_Loop_D1.80mm_Drill1.0mm_Beaded
- TP3: renamed from TP1; footprint TestPoint:TestPoint_Loop_D2.50mm_Drill1.0mm -> TestPoint:TestPoint_Loop_D1.80mm_Drill1.0mm_Beaded
- TP4: renamed from TP2; footprint TestPoint:TestPoint_Loop_D2.50mm_Drill1.0mm -> TestPoint:TestPoint_Loop_D1.80mm_Drill1.0mm_Beaded
- renumbered C9 to C10, C10 to C11, C11 to C12, C12 to C13, C13 to C14, C14 to C15, C1 to C2, C23 to C24, C24 to C25, C25 to C26, C26 to C27, C2 to C3, C33 to C34, C3 to C4, C46 to C47, C47 to C48, C48 to C49, C4 to C5, C49 to C50, C50 to C51, C51 to C52, C52 to C53, C53 to C54, C58 to C59, C5 to C6, C59 to C60, C60 to C61, C61 to C62, C62 to C63, C63 to C64, C64 to C65, C65 to C66, C66 to C67, C67 to C68, C68 to C69, C6 to C7, C69 to C70, C70 to C71, C71 to C72, C72 to C73, C73 to C74, C74 to C75, C75 to C76, C76 to C77, C77 to C78, C78 to C79, C7 to C8, C79 to C80, C80 to C81, C81 to C82, C82 to C83, C83 to C84, C84 to C85, C85 to C86, C86 to C87, C87 to C88, C88 to C89, C8 to C9, C89 to C90, C90 to C91, C91 to C92, C92 to C93, C93 to C94, D2 to D4, D3 to D5, D4 to D6, R6 to R10, R96 to R100, R97 to R101, R98 to R102, R99 to R103, R100 to R104, R101 to R105, R102 to R106, R103 to R107, R104 to R108, R105 to R109, R7 to R11, R106 to R110, R107 to R111, R108 to R112, R109 to R113, R110 to R114, R111 to R115, R112 to R116, R113 to R117, R114 to R118, R115 to R119, R8 to R12, R116 to R120, R117 to R121, R118 to R122, R119 to R123, R120 to R124, R121 to R125, R122 to R126, R123 to R127, R124 to R128, R125 to R129, R9 to R13, R126 to R130, R127 to R131, R128 to R132, R129 to R133, R130 to R134, R131 to R135, R132 to R136, R10 to R14, R11 to R15, R12 to R16, R13 to R17, R14 to R18, R15 to R19, R19 to R23, R20 to R24, R21 to R25, R22 to R26, R23 to R27, R24 to R28, R25 to R29, R26 to R30, R27 to R31, R28 to R32, R29 to R33, R30 to R34, R31 to R35, R32 to R36, R33 to R37, R34 to R38, R35 to R39, R36 to R40, R37 to R41, R38 to R42, R49 to R53, R50 to R54, R51 to R55, R52 to R56, R53 to R57, R54 to R58, R55 to R59, R56 to R60, R57 to R61, R61 to R65, R3 to R7, R4 to R8, R78 to R82, R79 to R83, R80 to R84, R81 to R85, R82 to R86, R83 to R87, R84 to R88, R5 to R9, R87 to R91, R88 to R92, R89 to R93, R90 to R94, R91 to R95, R92 to R96, R93 to R97, R94 to R98, R95 to R99, TP4 to TP2, U8 to U10, U9 to U11, U11 to U13, U12 to U14, U13 to U15, U14 to U16, U15 to U17, U2 to U4, U4 to U6, U7 to U9
Connections:
- J18 pad SH: (no net) -> GND
- J4 pad 10: +12V -> /CAR_CAN_L
- J4 pad 11: /ESTOP_2- -> /CAR_CAN_H
- J4 pad 12: /ESTOP_1-/2+ -> GND
- J4 pad 2: GND -> /CAR_CAN_H
- J4 pad 3: /ELCON_LV+ -> /CAR_CAN_L
- J4 pad 4: GND -> /ELCON_LV+
- J4 pad 5: /CAR_CAN_H -> +12V
- J4 pad 6: /CAR_CAN_L -> /ESTOP_1-/2+
- J4 pad 7: /CAR_CAN_L -> /ESTOP_1-/2+
- J4 pad 8: /CAR_CAN_H -> /ESTOP_2-
- J4 pad 9: /ESTOP_1-/2+ -> GND
- R135 pad 2: Net-(C94-Pad2) -> Net-(C95-Pad1)
- R136 pad 1: Net-(C94-Pad2) -> Net-(C95-Pad1)
- R19 pad 2: Net-(C18-Pad2) -> Net-(C19-Pad1)
- R65 pad 2: Net-(U5-PEAK) -> Net-(U7-PEAK)
- U1 pad 1: /Peripherals/100PinMCU/PE2 -> /HV-_SENSE
- U1 pad 15: /Peripherals/100PinMCU/PC0 -> /ARRAY_SENSE
- U1 pad 16: /Peripherals/100PinMCU/PC1 -> /ARRAY_ECON
- U1 pad 17: /Peripherals/100PinMCU/PC2 -> /ARRAY_CTRL
- U1 pad 2: /Peripherals/100PinMCU/PE3 -> /HV-_ECON
- U1 pad 25: /Peripherals/100PinMCU/PA3 -> /BMS_NFAULT
- U1 pad 3: /Peripherals/100PinMCU/PE4 -> /HV-_CTRL
- U1 pad 56: /Peripherals/100PinMCU/PD9 -> /Peripherals/ESP_GPIO3
- U1 pad 57: /Peripherals/100PinMCU/PD10 -> /Peripherals/ESP_GPIO4
- U1 pad 58: /Peripherals/100PinMCU/PD11 -> /Peripherals/ESP_NRST
- U1 pad 84: /Peripherals/100PinMCU/PD2 -> /ESTOP_1_SENSE
- U1 pad 85: /Peripherals/100PinMCU/PD3 -> /ESTOP_2_SENSE
- U1 pad 86: /Peripherals/100PinMCU/PD4 -> /ESTOP_3_SENSE
- U1 pad 94: /Peripherals/100PinMCU/PB7 -> /FAN_ALERT
- U1 pad 96: /Peripherals/100PinMCU/PB9 -> /HV+_SENSE
- U1 pad 97: /Peripherals/100PinMCU/PE0 -> /HV+_ECON
- U1 pad 98: /Peripherals/100PinMCU/PE1 -> /HV+_CTRL
- U17 pad 6: /Power/Power_Mux_PD/PR1 -> /Power/Power_Mux_PD/PRI
- U6 pad 6: /Power/Power_Mux_PDU_ELCON/PR1 -> /Power/Power_Mux_PDU_ELCON/PRI
