File: hardware/PowerProtection.kicad_sch (KiCad schematic)
At the start: 18 parts, among them IC5 LM74502DDFR, Q13 PSMN012-100YS, Q14 PSMN012-100YS

Commit message: finished schematic except for 12v buck boost
Parts:
- renumbered D28 to D26, D29 to D27
Changed lines of the file:
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@@
 		(in_pos_files yes)
 		(dnp no)
-		(property "Reference" "D29"
+		(property "Reference" "D27"
 			(at 40.64 82.296 0)
 			(show_name no)
@@
 			(project "PS-BPSLeader"
 				(path "/d4a4ed4f-0983-4aef-b212-0e3284ab3963/69244dac-f10b-499c-a2b2-3cdf1370aa1f/809e2845-19f2-4000-97b2-9d58cc5520c6"
-					(reference "D29")
+					(reference "D27")
 					(unit 1)
 				)
@@
 		(in_pos_files yes)
 		(dnp no)
-		(property "Reference" "D28"
+		(property "Reference" "D26"
 			(at 22.606 49.276 0)
 			(show_name no)
@@
 			(project "PS-BPSLeader"
 				(path "/d4a4ed4f-0983-4aef-b212-0e3284ab3963/69244dac-f10b-499c-a2b2-3cdf1370aa1f/809e2845-19f2-4000-97b2-9d58cc5520c6"
-					(reference "D28")
-					(unit 1)
-				)
+					(reference "D26")
+					(unit 1)
+				)

Commit message: added 12V buck boost
Parts:
- renumbered C77 to C78, C78 to C79, C79 to C80, C80 to C81, C81 to C82, C82 to C83, C83 to C84, D26 to D28, D27 to D29, R115 to R119, R116 to R120, R117 to R121, R118 to R122, R119 to R123, R120 to R124
Changed lines of the file:
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@@
 		(in_pos_files yes)
 		(dnp no)
-		(property "Reference" "C83"
+		(property "Reference" "C84"
 			(at 125.984 89.154 90)
 			(show_name no)
@@
 			(project "PS-BPSLeader"
 				(path "/d4a4ed4f-0983-4aef-b212-0e3284ab3963/69244dac-f10b-499c-a2b2-3cdf1370aa1f/809e2845-19f2-4000-97b2-9d58cc5520c6"
-					(reference "C83")
+					(reference "C84")
 					(unit 1)
 				)
@@
 		(in_pos_files yes)
 		(dnp no)
-		(property "Reference" "D27"
+		(property "Reference" "D29"
 			(at 40.64 82.296 0)
 			(show_name no)
@@
 			(project "PS-BPSLeader"
 				(path "/d4a4ed4f-0983-4aef-b212-0e3284ab3963/69244dac-f10b-499c-a2b2-3cdf1370aa1f/809e2845-19f2-4000-97b2-9d58cc5520c6"
-					(reference "D27")
+					(reference "D29")
 					(unit 1)
 				)
@@
 		(dnp no)
 		(fields_autoplaced yes)
-		(property "Reference" "C79"
+		(property "Reference" "C80"
 			(at 57.785 80.0099 0)
 			(show_name no)
@@
 			(project "PS-BPSLeader"
 				(path "/d4a4ed4f-0983-4aef-b212-0e3284ab3963/69244dac-f10b-499c-a2b2-3cdf1370aa1f/809e2845-19f2-4000-97b2-9d58cc5520c6"
-					(reference "C79")
+					(reference "C80")
 					(unit 1)
 				)
@@
 		(in_pos_files yes)
 		(dnp no)
-		(property "Reference" "D26"
+		(property "Reference" "D28"
 			(at 22.606 49.276 0)
 			(show_name no)
@@
 			(project "PS-BPSLeader"
 				(path "/d4a4ed4f-0983-4aef-b212-0e3284ab3963/69244dac-f10b-499c-a2b2-3cdf1370aa1f/809e2845-19f2-4000-97b2-9d58cc5520c6"
-					(reference "D26")
+					(reference "D28")
 					(unit 1)
 				)
@@
 		(dnp no)
 		(fields_autoplaced yes)
-		(property "Reference" "R115"
+		(property "Reference" "R119"
 			(at 45.72 60.9599 0)
 			(show_name no)
@@
 			(project "PS-BPSLeader"
 				(path "/d4a4ed4f-0983-4aef-b212-0e3284ab3963/69244dac-f10b-499c-a2b2-3cdf1370aa1f/809e2845-19f2-4000-97b2-9d58cc5520c6"
-					(reference "R115")
+					(reference "R119")
 					(unit 1)
 				)
@@
 		(in_pos_files yes)
 		(dnp no)
-		(property "Reference" "R120"
+		(property "Reference" "R124"
 			(at 137.668 90.17 90)
 			(show_name no)
@@
 			(project "PS-BPSLeader"
 				(path "/d4a4ed4f-0983-4aef-b212-0e3284ab3963/69244dac-f10b-499c-a2b2-3cdf1370aa1f/809e2845-19f2-4000-97b2-9d58cc5520c6"
-					(reference "R120")
+					(reference "R124")
 					(unit 1)
 				)
@@
 		(in_pos_files yes)
 		(dnp no)
-		(property "Reference" "C77"
+		(property "Reference" "C78"
 			(at 38.1 49.5299 0)
 			(show_name no)
@@
 			(project "PS-BPSLeader"
 				(path "/d4a4ed4f-0983-4aef-b212-0e3284ab3963/69244dac-f10b-499c-a2b2-3cdf1370aa1f/809e2845-19f2-4000-97b2-9d58cc5520c6"
-					(reference "C77")
+					(reference "C78")
 					(unit 1)
 				)
@@
 		(in_pos_files yes)
 		(dnp no)
-		(property "Reference" "R116"
+		(property "Reference" "R120"
 			(at 67.31 54.61 90)
 			(show_name no)
@@
 			(project "PS-BPSLeader"
 				(path "/d4a4ed4f-0983-4aef-b212-0e3284ab3963/69244dac-f10b-499c-a2b2-3cdf1370aa1f/809e2845-19f2-4000-97b2-9d58cc5520c6"
-					(reference "R116")
+					(reference "R120")
 					(unit 1)
 				)
@@
 		(in_pos_files yes)
 		(dnp no)
-		(property "Reference" "C82"
+		(property "Reference" "C83"
 			(at 107.188 88.9 90)
 			(show_name no)
@@
 			(project "PS-BPSLeader"
 				(path "/d4a4ed4f-0983-4aef-b212-0e3284ab3963/69244dac-f10b-499c-a2b2-3cdf1370aa1f/809e2845-19f2-4000-97b2-9d58cc5520c6"
-					(reference "C82")
+					(reference "C83")
 					(unit 1)
 				)
@@
 		(in_pos_files yes)
 		(dnp no)
-		(property "Reference" "C80"
+		(property "Reference" "C81"
 			(at 54.864 62.23 0)
 			(show_name no)
@@
 			(project "PS-BPSLeader"
 				(path "/d4a4ed4f-0983-4aef-b212-0e3284ab3963/69244dac-f10b-499c-a2b2-3cdf1370aa1f/809e2845-19f2-4000-97b2-9d58cc5520c6"
-					(reference "C80")
+					(reference "C81")
 					(unit 1)
 				)
@@
 		(in_pos_files yes)
 		(dnp no)
-		(property "Reference" "C81"
+		(property "Reference" "C82"
 			(at 112.395 49.5299 0)
 			(show_name no)
@@
 			(project "PS-BPSLeader"
 				(path "/d4a4ed4f-0983-4aef-b212-0e3284ab3963/69244dac-f10b-499c-a2b2-3cdf1370aa1f/809e2845-19f2-4000-97b2-9d58cc5520c6"
-					(reference "C81")
+					(reference "C82")
 					(unit 1)
 				)
@@
 		(in_pos_files yes)
 		(dnp no)
-		(property "Reference" "R118"
+		(property "Reference" "R122"
 			(at 118.618 90.424 90)
 			(show_name no)
@@
 			(project "PS-BPSLeader"
 				(path "/d4a4ed4f-0983-4aef-b212-0e3284ab3963/69244dac-f10b-499c-a2b2-3cdf1370aa1f/809e2845-19f2-4000-97b2-9d58cc5520c6"
-					(reference "R118")
+					(reference "R122")
 					(unit 1)
 				)
@@
 		(in_pos_files yes)
 		(dnp no)
-		(property "Reference" "C78"
+		(property "Reference" "C79"
 			(at 31.75 82.5499 0)
 			(show_name no)
@@
 			(project "PS-BPSLeader"
 				(path "/d4a4ed4f-0983-4aef-b212-0e3284ab3963/69244dac-f10b-499c-a2b2-3cdf1370aa1f/809e2845-19f2-4000-97b2-9d58cc5520c6"
-					(reference "C78")
+					(reference "C79")
 					(unit 1)
 				)
@@
 		(in_pos_files yes)
 		(dnp no)
-		(property "Reference" "R117"
+		(property "Reference" "R121"
 			(at 118.11 78.74 90)
 			(show_name no)
@@
 			(project "PS-BPSLeader"
 				(path "/d4a4ed4f-0983-4aef-b212-0e3284ab3963/69244dac-f10b-499c-a2b2-3cdf1370aa1f/809e2845-19f2-4000-97b2-9d58cc5520c6"
-					(reference "R117")
+					(reference "R121")
 					(unit 1)
 				)
@@
 		(in_pos_files yes)
 		(dnp no)
-		(property "Reference" "R119"
+		(property "Reference" "R123"
 			(at 137.16 77.47 90)
 			(show_name no)
@@
 			(project "PS-BPSLeader"
 				(path "/d4a4ed4f-0983-4aef-b212-0e3284ab3963/69244dac-f10b-499c-a2b2-3cdf1370aa1f/809e2845-19f2-4000-97b2-9d58cc5520c6"
-					(reference "R119")
-					(unit 1)
-				)
+					(reference "R123")
+					(unit 1)
+				)
