File: hardware/Power_5VMux.kicad_sch (KiCad schematic)
At the start: 6 parts, among them U1 TPS2117DRLR

Commit message: finished schematic except for 12v buck boost
Parts:
- renumbered C1 to C84, C2 to C85, C3 to C86, C4 to C87, R1 to R121, U1 to U15
Changed lines of the file:
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@@
 		(in_pos_files yes)
 		(dnp no)
-		(property "Reference" "C4"
+		(property "Reference" "C87"
 			(at 91.8972 57.2516 0)
 			(show_name no)
@@
 			(project "PS-BPSLeader"
 				(path "/d4a4ed4f-0983-4aef-b212-0e3284ab3963/69244dac-f10b-499c-a2b2-3cdf1370aa1f/62b47865-4d17-4cd5-b20c-36169ba543a0"
-					(reference "C4")
+					(reference "C87")
 					(unit 1)
 				)
@@
 		(in_pos_files yes)
 		(dnp no)
-		(property "Reference" "C2"
+		(property "Reference" "C85"
 			(at 38.5572 44.5516 0)
 			(show_name no)
@@
 			(project "PS-BPSLeader"
 				(path "/d4a4ed4f-0983-4aef-b212-0e3284ab3963/69244dac-f10b-499c-a2b2-3cdf1370aa1f/62b47865-4d17-4cd5-b20c-36169ba543a0"
-					(reference "C2")
+					(reference "C85")
 					(unit 1)
 				)
@@
 		(in_pos_files yes)
 		(dnp no)
-		(property "Reference" "C1"
+		(property "Reference" "C84"
 			(at 24.5872 44.5516 0)
 			(show_name no)
@@
 			(project "PS-BPSLeader"
 				(path "/d4a4ed4f-0983-4aef-b212-0e3284ab3963/69244dac-f10b-499c-a2b2-3cdf1370aa1f/62b47865-4d17-4cd5-b20c-36169ba543a0"
-					(reference "C1")
+					(reference "C84")
 					(unit 1)
 				)
@@
 		(in_pos_files yes)
 		(dnp no)
-		(property "Reference" "C3"
+		(property "Reference" "C86"
 			(at 42.3672 67.4116 0)
 			(show_name no)
@@
 			(project "PS-BPSLeader"
 				(path "/d4a4ed4f-0983-4aef-b212-0e3284ab3963/69244dac-f10b-499c-a2b2-3cdf1370aa1f/62b47865-4d17-4cd5-b20c-36169ba543a0"
-					(reference "C3")
+					(reference "C86")
 					(unit 1)
 				)
@@
 		(dnp no)
 		(fields_autoplaced yes)
-		(property "Reference" "U1"
+		(property "Reference" "U15"
 			(at 60.96 44.45 0)
 			(show_name no)
@@
 			(project "PS-BPSLeader"
 				(path "/d4a4ed4f-0983-4aef-b212-0e3284ab3963/69244dac-f10b-499c-a2b2-3cdf1370aa1f/62b47865-4d17-4cd5-b20c-36169ba543a0"
-					(reference "U1")
+					(reference "U15")
 					(unit 1)
 				)
@@
 		(in_pos_files yes)
 		(dnp no)
-		(property "Reference" "R1"
+		(property "Reference" "R121"
 			(at 78.994 67.564 0)
 			(show_name no)
@@
 			(project "PS-BPSLeader"
 				(path "/d4a4ed4f-0983-4aef-b212-0e3284ab3963/69244dac-f10b-499c-a2b2-3cdf1370aa1f/62b47865-4d17-4cd5-b20c-36169ba543a0"
-					(reference "R1")
-					(unit 1)
-				)
+					(reference "R121")
+					(unit 1)
+				)

Commit message: added 12V buck boost
Parts:
- renumbered C84 to C85, C85 to C86, C86 to C87, C87 to C88, R121 to R125
Changed lines of the file:
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@@
 		(in_pos_files yes)
 		(dnp no)
-		(property "Reference" "C87"
+		(property "Reference" "C88"
 			(at 91.8972 57.2516 0)
 			(show_name no)
@@
 			(project "PS-BPSLeader"
 				(path "/d4a4ed4f-0983-4aef-b212-0e3284ab3963/69244dac-f10b-499c-a2b2-3cdf1370aa1f/62b47865-4d17-4cd5-b20c-36169ba543a0"
-					(reference "C87")
+					(reference "C88")
 					(unit 1)
 				)
@@
 		(in_pos_files yes)
 		(dnp no)
-		(property "Reference" "C85"
+		(property "Reference" "C86"
 			(at 38.5572 44.5516 0)
 			(show_name no)
@@
 			(project "PS-BPSLeader"
 				(path "/d4a4ed4f-0983-4aef-b212-0e3284ab3963/69244dac-f10b-499c-a2b2-3cdf1370aa1f/62b47865-4d17-4cd5-b20c-36169ba543a0"
-					(reference "C85")
+					(reference "C86")
 					(unit 1)
 				)
@@
 		(in_pos_files yes)
 		(dnp no)
-		(property "Reference" "C84"
+		(property "Reference" "C85"
 			(at 24.5872 44.5516 0)
 			(show_name no)
@@
 			(project "PS-BPSLeader"
 				(path "/d4a4ed4f-0983-4aef-b212-0e3284ab3963/69244dac-f10b-499c-a2b2-3cdf1370aa1f/62b47865-4d17-4cd5-b20c-36169ba543a0"
-					(reference "C84")
+					(reference "C85")
 					(unit 1)
 				)
@@
 		(in_pos_files yes)
 		(dnp no)
-		(property "Reference" "C86"
+		(property "Reference" "C87"
 			(at 42.3672 67.4116 0)
 			(show_name no)
@@
 			(project "PS-BPSLeader"
 				(path "/d4a4ed4f-0983-4aef-b212-0e3284ab3963/69244dac-f10b-499c-a2b2-3cdf1370aa1f/62b47865-4d17-4cd5-b20c-36169ba543a0"
-					(reference "C86")
+					(reference "C87")
 					(unit 1)
 				)
@@
 		(in_pos_files yes)
 		(dnp no)
-		(property "Reference" "R121"
+		(property "Reference" "R125"
 			(at 78.994 67.564 0)
 			(show_name no)
@@
 			(project "PS-BPSLeader"
 				(path "/d4a4ed4f-0983-4aef-b212-0e3284ab3963/69244dac-f10b-499c-a2b2-3cdf1370aa1f/62b47865-4d17-4cd5-b20c-36169ba543a0"
-					(reference "R121")
-					(unit 1)
-				)
+					(reference "R125")
+					(unit 1)
+				)
