File: hardware/Power_Mux_12V.kicad_sch (KiCad schematic)
At the start: 1 part

Commit message: new contactor design block, started power mux
Parts:
- removed R42: R_Small, symbol Device:R_Small
- added R?: 22.1k, symbol Device:R_Small
- added U?: TPS2121RUXR, LHRS_Power:IC_TPS2121RUXR, symbol lhrs_power:TPS2121RUXR
Connections:
- new net: R?.1, U?.10 (ILIM)
- new net: U?.1 (OUT), U?.1_1 (OUT), U?.8 (OUT), U?.8_1 (OUT)
- new net: U?.2 (IN2), U?.2_1 (IN2)
- new net: U?.7 (IN1), U?.7_1 (IN1)

Commit message: end of workday
Parts:
- added C?: 1u, symbol Device:C_Small
- added R?: 26.1k, symbol Device:R_Small
- added R? (x4): 5k, symbol Device:R_Small
- added R? (x3): 57.6k, symbol Device:R_Small
Connections:
- net GND: now reaches R?.2
- net GND: now also U?.12 (GND), U?.9 (ST), C?.2, R?.2, R?.2, R?.2, R?.2
- net 12V_MUX_OUT: now reaches U?.1 (OUT), U?.1_1 (OUT), U?.8 (OUT), U?.8_1 (OUT)
- net at U?.11 (SS): now also C?.1
- net Vin2: now reaches U?.2 (IN2), U?.2_1 (IN2)
- net Vin2: now also R?.1, R?.1
- net CP2: now reaches U?.3 (CP2)
- net CP2: now also R?.1, R?.2
- net OV2: now reaches U?.4 (OV2)
- net OV2: now also R?.1, R?.2
- net OV1: now reaches U?.5 (OV1)
- net OV1: now also R?.1, R?.2
- net PR1: now reaches U?.6 (PR1)
- net Vin1: now reaches U?.7 (IN1), U?.7_1 (IN1)
- net Vin1: now also R?.1, R?.1
- new net PRI: R?.1, R?.2
Other:
- note added: "12V -> OV = 13.2V -> R = 57.6k -> PRI= 10.2V -> R = 26.1k 14V -> OV = 15.4V -> R = 67.3k -> CP2= 14V -> R = 37.4k 20V -> OV = 22V -> R = 100k -> CP2= 20V -> R = 56.2k"
- note added: "Current Limit"
- note added: "Resistor Divider Settings"
- note added: "VREF=1.06V (overvoltage limit) VCP2=1.64V (seamless switchover) VPR1=1.64V (undervoltage swap)"

Commit message: finished schematic except for 12v buck boost
Parts:
- removed C?: 1u, symbol Device:C_Small
- removed R?: 26.1k, symbol Device:R_Small
- removed R? (x4): 5k, symbol Device:R_Small
- removed R? (x3): 57.6k, symbol Device:R_Small
- removed R?: 22.1k, symbol Device:R_Small
- removed U?: TPS2121RUXR, LHRS_Power:IC_TPS2121RUXR, symbol lhrs_power:TPS2121RUXR
- added C33: 1u, Capacitor_SMD:C_0603_1608Metric_Pad1.08x0.95mm_HandSolder, symbol Device:C_Small
- added R49, R51, R55: 57.6k, Resistor_SMD:R_0603_1608Metric_Pad0.98x0.95mm_HandSolder, symbol Device:R_Small
- added R50, R52, R54, R56: 5k, Resistor_SMD:R_0603_1608Metric_Pad0.98x0.95mm_HandSolder, symbol Device:R_Small
- added R53: 26.1k, Resistor_SMD:R_0603_1608Metric_Pad0.98x0.95mm_HandSolder, symbol Device:R_Small
- added R57: 22.1k, Resistor_SMD:R_0603_1608Metric_Pad0.98x0.95mm_HandSolder, symbol Device:R_Small
- added U6: TPS2121RUXR, LHRS_ICs:TPS2121RUXR, symbol lhrs_power:TPS2121RUXR
Connections:
- net 12V_MUX_OUT: now also U6.1 (OUT), U6.1_1 (OUT), U6.8 (OUT), U6.8_1 (OUT)
- net CP2: now also R55.2, R56.1, U6.3 (CP2)
- net GND: now also C33.2, R50.2, R52.2, R54.2, R56.2, R57.2, U6.12 (GND), U6.9 (ST)
- net OV1: now also R49.2, R50.1, U6.5 (OV1)
- net OV2: now also R51.2, R52.1, U6.4 (OV2)
- net PRI: now also R53.2, R54.1, U6.6 (PR1)
- net Vin1: now also R49.1, R53.1, U6.7 (IN1), U6.7_1 (IN1)
- net Vin2: now also R51.1, R55.1, U6.2 (IN2), U6.2_1 (IN2)
- new net: R57.1, U6.10 (ILIM)
- new net: C33.1, U6.11 (SS)

Commit message: added 12V buck boost
Parts:
- renumbered C33 to C34, R49 to R53, R50 to R54, R51 to R55, R52 to R56, R53 to R57, R54 to R58, R55 to R59, R56 to R60, R57 to R61
Changed lines of the file:
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@@
 		(dnp no)
 		(fields_autoplaced yes)
-		(property "Reference" "R57"
+		(property "Reference" "R61"
 			(at 113.665 94.6149 0)
 			(show_name no)
@@
 			(project "PS-BPSLeader"
 				(path "/d4a4ed4f-0983-4aef-b212-0e3284ab3963/69244dac-f10b-499c-a2b2-3cdf1370aa1f/1a445fba-997a-4276-b1d7-6bccd354442b"
-					(reference "R57")
+					(reference "R61")
 					(unit 1)
 				)
@@
 		(dnp no)
 		(fields_autoplaced yes)
-		(property "Reference" "C33"
+		(property "Reference" "C34"
 			(at 102.87 94.6212 0)
 			(show_name no)
@@
 			(project "PS-BPSLeader"
 				(path "/d4a4ed4f-0983-4aef-b212-0e3284ab3963/69244dac-f10b-499c-a2b2-3cdf1370aa1f/1a445fba-997a-4276-b1d7-6bccd354442b"
-					(reference "C33")
+					(reference "C34")
 					(unit 1)
 				)
@@
 		(dnp no)
 		(fields_autoplaced yes)
-		(property "Reference" "R50"
+		(property "Reference" "R54"
 			(at 29.21 56.5149 0)
 			(show_name no)
@@
 			(project "PS-BPSLeader"
 				(path "/d4a4ed4f-0983-4aef-b212-0e3284ab3963/69244dac-f10b-499c-a2b2-3cdf1370aa1f/1a445fba-997a-4276-b1d7-6bccd354442b"
-					(reference "R50")
+					(reference "R54")
 					(unit 1)
 				)
@@
 		(dnp no)
 		(fields_autoplaced yes)
-		(property "Reference" "R55"
+		(property "Reference" "R59"
 			(at 68.58 45.7199 0)
 			(show_name no)
@@
 			(project "PS-BPSLeader"
 				(path "/d4a4ed4f-0983-4aef-b212-0e3284ab3963/69244dac-f10b-499c-a2b2-3cdf1370aa1f/1a445fba-997a-4276-b1d7-6bccd354442b"
-					(reference "R55")
+					(reference "R59")
 					(unit 1)
 				)
@@
 		(dnp no)
 		(fields_autoplaced yes)
-		(property "Reference" "R49"
+		(property "Reference" "R53"
 			(at 29.21 45.7199 0)
 			(show_name no)
@@
 			(project "PS-BPSLeader"
 				(path "/d4a4ed4f-0983-4aef-b212-0e3284ab3963/69244dac-f10b-499c-a2b2-3cdf1370aa1f/1a445fba-997a-4276-b1d7-6bccd354442b"
-					(reference "R49")
+					(reference "R53")
 					(unit 1)
 				)
@@
 		(dnp no)
 		(fields_autoplaced yes)
-		(property "Reference" "R56"
+		(property "Reference" "R60"
 			(at 69.215 56.5149 0)
 			(show_name no)
@@
 			(project "PS-BPSLeader"
 				(path "/d4a4ed4f-0983-4aef-b212-0e3284ab3963/69244dac-f10b-499c-a2b2-3cdf1370aa1f/1a445fba-997a-4276-b1d7-6bccd354442b"
-					(reference "R56")
+					(reference "R60")
 					(unit 1)
 				)
@@
 		(dnp no)
 		(fields_autoplaced yes)
-		(property "Reference" "R53"
+		(property "Reference" "R57"
 			(at 55.88 45.7199 0)
 			(show_name no)
@@
 			(project "PS-BPSLeader"
 				(path "/d4a4ed4f-0983-4aef-b212-0e3284ab3963/69244dac-f10b-499c-a2b2-3cdf1370aa1f/1a445fba-997a-4276-b1d7-6bccd354442b"
-					(reference "R53")
+					(reference "R57")
 					(unit 1)
 				)
@@
 		(dnp no)
 		(fields_autoplaced yes)
-		(property "Reference" "R51"
+		(property "Reference" "R55"
 			(at 41.91 45.7199 0)
 			(show_name no)
@@
 			(project "PS-BPSLeader"
 				(path "/d4a4ed4f-0983-4aef-b212-0e3284ab3963/69244dac-f10b-499c-a2b2-3cdf1370aa1f/1a445fba-997a-4276-b1d7-6bccd354442b"
-					(reference "R51")
+					(reference "R55")
 					(unit 1)
 				)
@@
 		(dnp no)
 		(fields_autoplaced yes)
-		(property "Reference" "R54"
+		(property "Reference" "R58"
 			(at 55.88 56.5149 0)
 			(show_name no)
@@
 			(project "PS-BPSLeader"
 				(path "/d4a4ed4f-0983-4aef-b212-0e3284ab3963/69244dac-f10b-499c-a2b2-3cdf1370aa1f/1a445fba-997a-4276-b1d7-6bccd354442b"
-					(reference "R54")
+					(reference "R58")
 					(unit 1)
 				)
@@
 		(dnp no)
 		(fields_autoplaced yes)
-		(property "Reference" "R52"
+		(property "Reference" "R56"
 			(at 41.91 56.5149 0)
 			(show_name no)
@@
 			(project "PS-BPSLeader"
 				(path "/d4a4ed4f-0983-4aef-b212-0e3284ab3963/69244dac-f10b-499c-a2b2-3cdf1370aa1f/1a445fba-997a-4276-b1d7-6bccd354442b"
-					(reference "R52")
+					(reference "R56")
 					(unit 1)
 				)
