File: hardware/Power_Mux_12V.kicad_sch (KiCad schematic)
At the start: 11 parts, among them U6 TPS2121RUXR

Commit message: forgot to push last night
Parts:
- R55: value 57.6k -> 67.3k
- R59: value 57.6k -> 37.4k
Changed lines of the file:
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@@
 			)
 		)
-		(property "Value" "57.6k"
+		(property "Value" "37.4k"
 			(at 68.58 48.2599 0)
 			(show_name no)
@@
 			)
 		)
-		(property "Value" "57.6k"
+		(property "Value" "67.3k"
 			(at 41.91 48.2599 0)
 			(show_name no)
