File: hardware/SD_Card.kicad_sch (KiCad schematic)
At the start: 4 parts, among them J2 Micro_SD_Card_Det

Commit message: finished schematic except for 12v buck boost
Parts:
- CR1: footprint UTSVT_ICs:D5V0P4UR6SO-7 -> LHRS_ICs:D5V0P4UR6SO-7
- renumbered J2 to J18, R25 to R87, R22 to R88
Connections:
- net GND: now also J18.SH (SHIELD); no longer J18.11 (SHIELD)
Changed lines of the file:
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@@
 		(in_pos_files yes)
 		(dnp no)
-		(property "Reference" "J2"
+		(property "Reference" "J18"
 			(at 166.37 35.1282 0)
 			(show_name no)
@@
 		(pin "10"
 		)
-		(pin "11"
+		(pin "SH"
 		)
 		(pin "2"
@@
 			(project "PS-BPSLeader"
 				(path "/d4a4ed4f-0983-4aef-b212-0e3284ab3963/5da56964-fa04-4fec-bdfe-c6acfeda5c9a/252fc626-7591-4f51-9e25-7431ee334d05"
-					(reference "J2")
+					(reference "J18")
 					(unit 1)
 				)
@@
 		(in_pos_files yes)
 		(dnp no)
-		(property "Reference" "R22"
+		(property "Reference" "R88"
 			(at 134.366 58.674 90)
 			(show_name no)
@@
 			(project "PS-BPSLeader"
 				(path "/d4a4ed4f-0983-4aef-b212-0e3284ab3963/5da56964-fa04-4fec-bdfe-c6acfeda5c9a/252fc626-7591-4f51-9e25-7431ee334d05"
-					(reference "R22")
+					(reference "R88")
 					(unit 1)
 				)
@@
 			)
 		)
-		(property "Footprint" "UTSVT_ICs:D5V0P4UR6SO-7"
+		(property "Footprint" "LHRS_ICs:D5V0P4UR6SO-7"
 			(at 76.835 46.99 0)
 			(hide yes)
@@
 		(dnp no)
 		(fields_autoplaced yes)
-		(property "Reference" "R25"
+		(property "Reference" "R87"
 			(at 135.89 72.3899 0)
 			(show_name no)
@@
 			(project "PS-BPSLeader"
 				(path "/d4a4ed4f-0983-4aef-b212-0e3284ab3963/5da56964-fa04-4fec-bdfe-c6acfeda5c9a/252fc626-7591-4f51-9e25-7431ee334d05"
-					(reference "R25")
+					(reference "R87")
 					(unit 1)
 				)

Commit message: added 12V buck boost
Parts:
- renumbered R87 to R91, R88 to R92
Changed lines of the file:
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@@
 		(in_pos_files yes)
 		(dnp no)
-		(property "Reference" "R88"
+		(property "Reference" "R92"
 			(at 134.366 58.674 90)
 			(show_name no)
@@
 			(project "PS-BPSLeader"
 				(path "/d4a4ed4f-0983-4aef-b212-0e3284ab3963/5da56964-fa04-4fec-bdfe-c6acfeda5c9a/252fc626-7591-4f51-9e25-7431ee334d05"
-					(reference "R88")
+					(reference "R92")
 					(unit 1)
 				)
@@
 		(dnp no)
 		(fields_autoplaced yes)
-		(property "Reference" "R87"
+		(property "Reference" "R91"
 			(at 135.89 72.3899 0)
 			(show_name no)
@@
 			(project "PS-BPSLeader"
 				(path "/d4a4ed4f-0983-4aef-b212-0e3284ab3963/5da56964-fa04-4fec-bdfe-c6acfeda5c9a/252fc626-7591-4f51-9e25-7431ee334d05"
-					(reference "R87")
+					(reference "R91")
 					(unit 1)
 				)
