File: hardware/Power_Mux_PD.kicad_sch (KiCad schematic)
At the start: 11 parts

Commit message: finished schematic except for 12v buck boost
Parts:
- C90: renamed from C?; footprint (none) -> Capacitor_SMD:C_0603_1608Metric_Pad1.08x0.95mm_HandSolder
- R122, R123, R124, R125, R126, R127, R128, R129, R130: renamed from R?; footprint (none) -> Resistor_SMD:R_0603_1608Metric_Pad0.98x0.95mm_HandSolder
- U17: renamed from U?; footprint LHRS_Power:IC_TPS2121RUXR -> LHRS_ICs:TPS2121RUXR
Connections:
- net PR1 is gone; now on net PRI: U17.6 (PR1)
Changed lines of the file:
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@@
 	(wire
 		(pts
+			(xy 149.86 67.31) (xy 149.86 69.85)
+		)
+		(stroke
+			(width 0)
+			(type default)
+		)
+	)
+	(wire
+		(pts
 			(xy 112.395 77.47) (xy 117.475 77.47)
 		)
@@
 	(wire
 		(pts
+			(xy 142.875 67.31) (xy 149.86 67.31)
+		)
+		(stroke
+			(width 0)
+			(type default)
+		)
+	)
+	(wire
+		(pts
 			(xy 53.34 52.705) (xy 53.34 55.245)
 		)
@@
 		)
 	)
-	(label "PR1"
+	(label "PRI"
 		(at 112.395 67.31 0)
 		(effects
@@
 	(hierarchical_label "GND"
 		(shape input)
-		(at 142.875 67.31 270)
+		(at 149.86 69.85 270)
 		(effects
 			(font
@@
 		(dnp no)
 		(fields_autoplaced yes)
-		(property "Reference" "R?"
+		(property "Reference" "R126"
 			(at 55.88 45.7199 0)
 			(show_name no)
@@
 			)
 		)
-		(property "Footprint" ""
+		(property "Footprint" "Resistor_SMD:R_0603_1608Metric_Pad0.98x0.95mm_HandSolder"
 			(at 53.34 46.99 0)
 			(hide yes)
@@
 			(project "PS-BPSLeader"
 				(path "/d4a4ed4f-0983-4aef-b212-0e3284ab3963/69244dac-f10b-499c-a2b2-3cdf1370aa1f/0f3e3992-4755-4e76-a363-7a4e463e2a3d"
-					(reference "R?")
+					(reference "R126")
 					(unit 1)
 				)
@@
 		(dnp no)
 		(fields_autoplaced yes)
-		(property "Reference" "R?"
+		(property "Reference" "R125"
 			(at 41.91 56.5149 0)
 			(show_name no)
@@
 			)
 		)
-		(property "Footprint" ""
+		(property "Footprint" "Resistor_SMD:R_0603_1608Metric_Pad0.98x0.95mm_HandSolder"
 			(at 39.37 57.785 0)
 			(hide yes)
@@
 			(project "PS-BPSLeader"
 				(path "/d4a4ed4f-0983-4aef-b212-0e3284ab3963/69244dac-f10b-499c-a2b2-3cdf1370aa1f/0f3e3992-4755-4e76-a363-7a4e463e2a3d"
-					(reference "R?")
+					(reference "R125")
 					(unit 1)
 				)
@@
 		(dnp no)
 		(fields_autoplaced yes)
-		(property "Reference" "R?"
+		(property "Reference" "R123"
 			(at 29.21 56.5149 0)
 			(show_name no)
@@
 			)
 		)
-		(property "Footprint" ""
+		(property "Footprint" "Resistor_SMD:R_0603_1608Metric_Pad0.98x0.95mm_HandSolder"
 			(at 26.67 57.785 0)
 			(hide yes)
@@
 			(project "PS-BPSLeader"
 				(path "/d4a4ed4f-0983-4aef-b212-0e3284ab3963/69244dac-f10b-499c-a2b2-3cdf1370aa1f/0f3e3992-4755-4e76-a363-7a4e463e2a3d"
-					(reference "R?")
+					(reference "R123")
 					(unit 1)
 				)
@@
 		(dnp no)
 		(fields_autoplaced yes)
-		(property "Reference" "R?"
+		(property "Reference" "R122"
 			(at 29.21 45.7199 0)
 			(show_name no)
@@
 			)
 		)
-		(property "Footprint" ""
+		(property "Footprint" "Resistor_SMD:R_0603_1608Metric_Pad0.98x0.95mm_HandSolder"
 			(at 26.67 46.99 0)
 			(hide yes)
@@
 			(project "PS-BPSLeader"
 				(path "/d4a4ed4f-0983-4aef-b212-0e3284ab3963/69244dac-f10b-499c-a2b2-3cdf1370aa1f/0f3e3992-4755-4e76-a363-7a4e463e2a3d"
-					(reference "R?")
+					(reference "R122")
 					(unit 1)
 				)
@@
 		(dnp no)
 		(fields_autoplaced yes)
-		(property "Reference" "R?"
+		(property "Reference" "R124"
 			(at 41.91 45.7199 0)
 			(show_name no)
@@
 			)
 		)
-		(property "Footprint" ""
+		(property "Footprint" "Resistor_SMD:R_0603_1608Metric_Pad0.98x0.95mm_HandSolder"
 			(at 39.37 46.99 0)
 			(hide yes)
@@
 			(project "PS-BPSLeader"
 				(path "/d4a4ed4f-0983-4aef-b212-0e3284ab3963/69244dac-f10b-499c-a2b2-3cdf1370aa1f/0f3e3992-4755-4e76-a363-7a4e463e2a3d"
-					(reference "R?")
+					(reference "R124")
 					(unit 1)
 				)
@@
 		(dnp no)
 		(fields_autoplaced yes)
-		(property "Reference" "R?"
+		(property "Reference" "R130"
 			(at 113.665 94.6149 0)
 			(show_name no)
@@
 			)
 		)
-		(property "Footprint" ""
+		(property "Footprint" "Resistor_SMD:R_0603_1608Metric_Pad0.98x0.95mm_HandSolder"
 			(at 111.76 95.885 0)
 			(hide yes)
@@
 			(project "PS-BPSLeader"
 				(path "/d4a4ed4f-0983-4aef-b212-0e3284ab3963/69244dac-f10b-499c-a2b2-3cdf1370aa1f/0f3e3992-4755-4e76-a363-7a4e463e2a3d"
-					(reference "R?")
+					(reference "R130")
 					(unit 1)
 				)
@@
 		(dnp no)
 		(fields_autoplaced yes)
-		(property "Reference" "U?"
+		(property "Reference" "U17"
 			(at 130.175 54.61 0)
 			(show_name no)
@@
 			)
 		)
-		(property "Footprint" "LHRS_Power:IC_TPS2121RUXR"
+		(property "Footprint" "LHRS_ICs:TPS2121RUXR"
 			(at 130.175 80.01 0)
 			(hide yes)
@@
 			(project "PS-BPSLeader"
 				(path "/d4a4ed4f-0983-4aef-b212-0e3284ab3963/69244dac-f10b-499c-a2b2-3cdf1370aa1f/0f3e3992-4755-4e76-a363-7a4e463e2a3d"
-					(reference "U?")
+					(reference "U17")
 					(unit 1)
 				)
@@
 		(dnp no)
 		(fields_autoplaced yes)
-		(property "Reference" "R?"
+		(property "Reference" "R128"
 			(at 68.58 45.7199 0)
 			(show_name no)
@@
 			)
 		)
-		(property "Footprint" ""
+		(property "Footprint" "Resistor_SMD:R_0603_1608Metric_Pad0.98x0.95mm_HandSolder"
 			(at 66.675 46.99 0)
 			(hide yes)
@@
 			(project "PS-BPSLeader"
 				(path "/d4a4ed4f-0983-4aef-b212-0e3284ab3963/69244dac-f10b-499c-a2b2-3cdf1370aa1f/0f3e3992-4755-4e76-a363-7a4e463e2a3d"
-					(reference "R?")
+					(reference "R128")
 					(unit 1)
 				)
@@
 		(dnp no)
 		(fields_autoplaced yes)
-		(property "Reference" "C?"
+		(property "Reference" "C90"
 			(at 102.87 94.6212 0)
 			(show_name no)
@@
 			)
 		)
-		(property "Footprint" ""
+		(property "Footprint" "Capacitor_SMD:C_0603_1608Metric_Pad1.08x0.95mm_HandSolder"
 			(at 105.41 95.885 0)
 			(hide yes)
@@
 			(project "PS-BPSLeader"
 				(path "/d4a4ed4f-0983-4aef-b212-0e3284ab3963/69244dac-f10b-499c-a2b2-3cdf1370aa1f/0f3e3992-4755-4e76-a363-7a4e463e2a3d"
-					(reference "C?")
+					(reference "C90")
 					(unit 1)
 				)
@@
 		(dnp no)
 		(fields_autoplaced yes)
-		(property "Reference" "R?"
+		(property "Reference" "R127"
 			(at 55.88 56.5149 0)
 			(show_name no)
@@
 			)
 		)
-		(property "Footprint" ""
+		(property "Footprint" "Resistor_SMD:R_0603_1608Metric_Pad0.98x0.95mm_HandSolder"
 			(at 53.34 57.785 0)
 			(hide yes)
@@
 			(project "PS-BPSLeader"
 				(path "/d4a4ed4f-0983-4aef-b212-0e3284ab3963/69244dac-f10b-499c-a2b2-3cdf1370aa1f/0f3e3992-4755-4e76-a363-7a4e463e2a3d"
-					(reference "R?")
+					(reference "R127")
 					(unit 1)
 				)
@@
 		(dnp no)
 		(fields_autoplaced yes)
-		(property "Reference" "R?"
+		(property "Reference" "R129"
 			(at 69.215 56.5149 0)
 			(show_name no)
@@
 			)
 		)
-		(property "Footprint" ""
+		(property "Footprint" "Resistor_SMD:R_0603_1608Metric_Pad0.98x0.95mm_HandSolder"
 			(at 66.675 57.785 0)
 			(hide yes)
@@
 			(project "PS-BPSLeader"
 				(path "/d4a4ed4f-0983-4aef-b212-0e3284ab3963/69244dac-f10b-499c-a2b2-3cdf1370aa1f/0f3e3992-4755-4e76-a363-7a4e463e2a3d"
-					(reference "R?")
+					(reference "R129")
 					(unit 1)
 				)

Commit message: added 12V buck boost
Parts:
- renumbered C90 to C91, R122 to R126, R123 to R127, R124 to R128, R125 to R129, R126 to R130, R127 to R131, R128 to R132, R129 to R133, R130 to R134
Changed lines of the file:
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@@
 		(dnp no)
 		(fields_autoplaced yes)
-		(property "Reference" "R126"
+		(property "Reference" "R130"
 			(at 55.88 45.7199 0)
 			(show_name no)
@@
 			(project "PS-BPSLeader"
 				(path "/d4a4ed4f-0983-4aef-b212-0e3284ab3963/69244dac-f10b-499c-a2b2-3cdf1370aa1f/0f3e3992-4755-4e76-a363-7a4e463e2a3d"
-					(reference "R126")
+					(reference "R130")
 					(unit 1)
 				)
@@
 		(dnp no)
 		(fields_autoplaced yes)
-		(property "Reference" "R125"
+		(property "Reference" "R129"
 			(at 41.91 56.5149 0)
 			(show_name no)
@@
 			(project "PS-BPSLeader"
 				(path "/d4a4ed4f-0983-4aef-b212-0e3284ab3963/69244dac-f10b-499c-a2b2-3cdf1370aa1f/0f3e3992-4755-4e76-a363-7a4e463e2a3d"
-					(reference "R125")
+					(reference "R129")
 					(unit 1)
 				)
@@
 		(dnp no)
 		(fields_autoplaced yes)
-		(property "Reference" "R123"
+		(property "Reference" "R127"
 			(at 29.21 56.5149 0)
 			(show_name no)
@@
 			(project "PS-BPSLeader"
 				(path "/d4a4ed4f-0983-4aef-b212-0e3284ab3963/69244dac-f10b-499c-a2b2-3cdf1370aa1f/0f3e3992-4755-4e76-a363-7a4e463e2a3d"
-					(reference "R123")
+					(reference "R127")
 					(unit 1)
 				)
@@
 		(dnp no)
 		(fields_autoplaced yes)
-		(property "Reference" "R122"
+		(property "Reference" "R126"
 			(at 29.21 45.7199 0)
 			(show_name no)
@@
 			(project "PS-BPSLeader"
 				(path "/d4a4ed4f-0983-4aef-b212-0e3284ab3963/69244dac-f10b-499c-a2b2-3cdf1370aa1f/0f3e3992-4755-4e76-a363-7a4e463e2a3d"
-					(reference "R122")
+					(reference "R126")
 					(unit 1)
 				)
@@
 		(dnp no)
 		(fields_autoplaced yes)
-		(property "Reference" "R124"
+		(property "Reference" "R128"
 			(at 41.91 45.7199 0)
 			(show_name no)
@@
 			(project "PS-BPSLeader"
 				(path "/d4a4ed4f-0983-4aef-b212-0e3284ab3963/69244dac-f10b-499c-a2b2-3cdf1370aa1f/0f3e3992-4755-4e76-a363-7a4e463e2a3d"
-					(reference "R124")
+					(reference "R128")
 					(unit 1)
 				)
@@
 		(dnp no)
 		(fields_autoplaced yes)
-		(property "Reference" "R130"
+		(property "Reference" "R134"
 			(at 113.665 94.6149 0)
 			(show_name no)
@@
 			(project "PS-BPSLeader"
 				(path "/d4a4ed4f-0983-4aef-b212-0e3284ab3963/69244dac-f10b-499c-a2b2-3cdf1370aa1f/0f3e3992-4755-4e76-a363-7a4e463e2a3d"
-					(reference "R130")
+					(reference "R134")
 					(unit 1)
 				)
@@
 		(dnp no)
 		(fields_autoplaced yes)
-		(property "Reference" "R128"
+		(property "Reference" "R132"
 			(at 68.58 45.7199 0)
 			(show_name no)
@@
 			(project "PS-BPSLeader"
 				(path "/d4a4ed4f-0983-4aef-b212-0e3284ab3963/69244dac-f10b-499c-a2b2-3cdf1370aa1f/0f3e3992-4755-4e76-a363-7a4e463e2a3d"
-					(reference "R128")
+					(reference "R132")
 					(unit 1)
 				)
@@
 		(dnp no)
 		(fields_autoplaced yes)
-		(property "Reference" "C90"
+		(property "Reference" "C91"
 			(at 102.87 94.6212 0)
 			(show_name no)
@@
 			(project "PS-BPSLeader"
 				(path "/d4a4ed4f-0983-4aef-b212-0e3284ab3963/69244dac-f10b-499c-a2b2-3cdf1370aa1f/0f3e3992-4755-4e76-a363-7a4e463e2a3d"
-					(reference "C90")
+					(reference "C91")
 					(unit 1)
 				)
@@
 		(dnp no)
 		(fields_autoplaced yes)
-		(property "Reference" "R127"
+		(property "Reference" "R131"
 			(at 55.88 56.5149 0)
 			(show_name no)
@@
 			(project "PS-BPSLeader"
 				(path "/d4a4ed4f-0983-4aef-b212-0e3284ab3963/69244dac-f10b-499c-a2b2-3cdf1370aa1f/0f3e3992-4755-4e76-a363-7a4e463e2a3d"
-					(reference "R127")
+					(reference "R131")
 					(unit 1)
 				)
@@
 		(dnp no)
 		(fields_autoplaced yes)
-		(property "Reference" "R129"
+		(property "Reference" "R133"
 			(at 69.215 56.5149 0)
 			(show_name no)
@@
 			(project "PS-BPSLeader"
 				(path "/d4a4ed4f-0983-4aef-b212-0e3284ab3963/69244dac-f10b-499c-a2b2-3cdf1370aa1f/0f3e3992-4755-4e76-a363-7a4e463e2a3d"
-					(reference "R129")
+					(reference "R133")
 					(unit 1)
 				)

Commit message: forgot to push last night
Parts:
- R128: value 57.6k -> 100k
Changed lines of the file:
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@@
 			)
 		)
-		(property "Value" "57.6k"
+		(property "Value" "100k"
 			(at 41.91 48.2599 0)
 			(show_name no)
