File: hardware/ESTOP.kicad_sch (KiCad schematic)
At the start: 0 parts

Commit message: added more stuff wip
Parts:
- added ESTOP1, ESTOP2, ESTOP3: LED, LED_SMD:LED_0603_1608Metric, symbol Device:LED
- added E_JP1, E_JP2, E_JP3: Jumper_2_Open, Connector_PinHeader_2.54mm:PinHeader_1x02_P2.54mm_Vertical, symbol Jumper:Jumper_2_Open
- added J10: Conn_01x02, UTSVT_Connectors:Molex_Nano-Fit_105309-xx02_1x02_P2.50mm_Vertical, symbol Connector_Generic:Conn_01x02
- added Q5, Q7, Q8: SQ2315CES-T1_GE3, CustomKiCad-Library:SOT95P237X112-3N, symbol CustomSymbols:SQ2315CES-T1_GE3
- added R34, R35, R95: 33k, Resistor_SMD:R_0603_1608Metric, symbol Device:R_US
- added R63, R72, R73, R91, R93, R94: 10k, Resistor_SMD:R_0603_1608Metric, symbol Device:R_US
- added R69, R70, R71: 470, Resistor_SMD:R_0603_1608Metric, symbol Device:R_US
Connections:
- new net: Q7.3 (D), R69.1, R72.1
- new net: ESTOP2.2 (A), R69.2
- new net: ESTOP1.2 (A), R71.2
- new net: Q5.1 (G), R34.1, R94.2
- new net: Q8.1 (G), R35.1, R91.2
- new net: Q8.3 (D), R71.1, R73.1
- new net: Q5.3 (D), R63.1, R70.1
- new net: Q7.1 (G), R93.2, R95.1
- new net: ESTOP3.2 (A), R70.2
- new net +24V: E_JP1.1 (A)
- new net +3.3V: Q5.2 (S), Q7.2 (S), Q8.2 (S)
- new net ESTOP_1-/2+: E_JP1.2 (B), E_JP2.1 (A), R35.2
- new net ESTOP_1_SENSE: R73.2
- new net ESTOP_2-: E_JP2.2 (B), E_JP3.1 (A), J10.1 (Pin_1), R95.2
- new net ESTOP_2_SENSE: R72.2
- new net ESTOP_3_SENSE: R63.2
- new net ESTOP_OUT: E_JP3.2 (B), J10.2 (Pin_2), R34.2
- new net GND: ESTOP1.1 (K), ESTOP2.1 (K), ESTOP3.1 (K), R91.1, R93.1, R94.1
Other:
- note added: "Estop Driver"
- note added: "Vgs = 10k/(33k+10k)*24V = 5.58V"

Commit message: power updates
Parts:
- R34, R35, R63, R69, R70, R71, R72, R73, R91, R93, R94, R95: symbol Device:R_US -> Device:R
Changed lines of the file:
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@@
 	)
 	(symbol
-		(lib_id "Device:R_US")
+		(lib_id "Device:R")
 		(at 60.96 91.44 270)
 		(unit 1)
@@
 		)
 		(property "Footprint" "Resistor_SMD:R_0603_1608Metric"
-			(at 60.706 92.456 90)
-			(effects
-				(font
-					(size 1.27 1.27)
-				)
-				(hide yes)
-			)
-		)
-		(property "Datasheet" "https://www.vishay.com/docs/20035/dcrcwe3.pdf"
+			(at 60.96 89.662 90)
+			(effects
+				(font
+					(size 1.27 1.27)
+				)
+				(hide yes)
+			)
+		)
+		(property "Datasheet" "~"
 			(at 60.96 91.44 0)
 			(effects
@@
 			)
 		)
-		(property "Description" "Resistor, US symbol"
+		(property "Description" "Resistor"
 			(at 60.96 91.44 0)
 			(effects
@@
 	)
 	(symbol
-		(lib_id "Device:R_US")
+		(lib_id "Device:R")
 		(at 59.69 86.36 270)
 		(mirror x)
@@
 		)
 		(property "Footprint" "Resistor_SMD:R_0603_1608Metric"
-			(at 59.436 85.344 90)
-			(effects
-				(font
-					(size 1.27 1.27)
-				)
-				(hide yes)
-			)
-		)
-		(property "Datasheet" "https://www.vishay.com/docs/20035/dcrcwe3.pdf"
+			(at 59.69 88.138 90)
+			(effects
+				(font
+					(size 1.27 1.27)
+				)
+				(hide yes)
+			)
+		)
+		(property "Datasheet" "~"
 			(at 59.69 86.36 0)
 			(effects
@@
 			)
 		)
-		(property "Description" "Resistor, US symbol"
+		(property "Description" "Resistor"
 			(at 59.69 86.36 0)
 			(effects
@@
 	)
 	(symbol
-		(lib_id "Device:R_US")
+		(lib_id "Device:R")
 		(at 82.55 111.76 0)
 		(mirror x)
@@
 		)
 		(property "Footprint" "Resistor_SMD:R_0603_1608Metric"
-			(at 83.566 111.506 90)
-			(effects
-				(font
-					(size 1.27 1.27)
-				)
-				(hide yes)
-			)
-		)
-		(property "Datasheet" "https://www.vishay.com/docs/20035/dcrcwe3.pdf"
+			(at 80.772 111.76 90)
+			(effects
+				(font
+					(size 1.27 1.27)
+				)
+				(hide yes)
+			)
+		)
+		(property "Datasheet" "~"
 			(at 82.55 111.76 0)
 			(effects
@@
 			)
 		)
-		(property "Description" "Resistor, US symbol"
+		(property "Description" "Resistor"
 			(at 82.55 111.76 0)
 			(effects
@@
 	)
 	(symbol
-		(lib_id "Device:R_US")
+		(lib_id "Device:R")
 		(at 58.42 115.57 270)
 		(mirror x)
@@
 		)
 		(property "Footprint" "Resistor_SMD:R_0603_1608Metric"
-			(at 58.166 114.554 90)
-			(effects
-				(font
-					(size 1.27 1.27)
-				)
-				(hide yes)
-			)
-		)
-		(property "Datasheet" "https://www.vishay.com/docs/20035/dcrcwe3.pdf"
+			(at 58.42 117.348 90)
+			(effects
+				(font
+					(size 1.27 1.27)
+				)
+				(hide yes)
+			)
+		)
+		(property "Datasheet" "~"
 			(at 58.42 115.57 0)
 			(effects
@@
 			)
 		)
-		(property "Description" "Resistor, US symbol"
+		(property "Description" "Resistor"
 			(at 58.42 115.57 0)
 			(effects
@@
 	)
 	(symbol
-		(lib_id "Device:R_US")
+		(lib_id "Device:R")
 		(at 82.55 82.55 0)
 		(mirror x)
@@
 		)
 		(property "Footprint" "Resistor_SMD:R_0603_1608Metric"
-			(at 83.566 82.296 90)
-			(effects
-				(font
-					(size 1.27 1.27)
-				)
-				(hide yes)
-			)
-		)
-		(property "Datasheet" "https://www.vishay.com/docs/20035/dcrcwe3.pdf"
+			(at 80.772 82.55 90)
+			(effects
+				(font
+					(size 1.27 1.27)
+				)
+				(hide yes)
+			)
+		)
+		(property "Datasheet" "~"
 			(at 82.55 82.55 0)
 			(effects
@@
 			)
 		)
-		(property "Description" "Resistor, US symbol"
+		(property "Description" "Resistor"
 			(at 82.55 82.55 0)
 			(effects
@@
 	)
 	(symbol
-		(lib_id "Device:R_US")
+		(lib_id "Device:R")
 		(at 88.9 76.2 90)
 		(mirror x)
@@
 		)
 		(property "Footprint" "Resistor_SMD:R_0603_1608Metric"
-			(at 89.154 77.216 90)
-			(effects
-				(font
-					(size 1.27 1.27)
-				)
-				(hide yes)
-			)
-		)
-		(property "Datasheet" "https://www.vishay.com/docs/20035/dcrcwe3.pdf"
+			(at 88.9 74.422 90)
+			(effects
+				(font
+					(size 1.27 1.27)
+				)
+				(hide yes)
+			)
+		)
+		(property "Datasheet" "~"
 			(at 88.9 76.2 0)
 			(effects
@@
 			)
 		)
-		(property "Description" "Resistor, US symbol"
+		(property "Description" "Resistor"
 			(at 88.9 76.2 0)
 			(effects
@@
 	)
 	(symbol
-		(lib_id "Device:R_US")
+		(lib_id "Device:R")
 		(at 59.69 54.61 270)
 		(mirror x)
@@
 		)
 		(property "Footprint" "Resistor_SMD:R_0603_1608Metric"
-			(at 59.436 53.594 90)
-			(effects
-				(font
-					(size 1.27 1.27)
-				)
-				(hide yes)
-			)
-		)
-		(property "Datasheet" "https://www.vishay.com/docs/20035/dcrcwe3.pdf"
+			(at 59.69 56.388 90)
+			(effects
+				(font
+					(size 1.27 1.27)
+				)
+				(hide yes)
+			)
+		)
+		(property "Datasheet" "~"
 			(at 59.69 54.61 0)
 			(effects
@@
 			)
 		)
-		(property "Description" "Resistor, US symbol"
+		(property "Description" "Resistor"
 			(at 59.69 54.61 0)
 			(effects
@@
 	)
 	(symbol
-		(lib_id "Device:R_US")
+		(lib_id "Device:R")
 		(at 62.23 59.69 270)
 		(unit 1)
@@
 		)
 		(property "Footprint" "Resistor_SMD:R_0603_1608Metric"
-			(at 61.976 60.706 90)
-			(effects
-				(font
-					(size 1.27 1.27)
-				)
-				(hide yes)
-			)
-		)
-		(property "Datasheet" "https://www.vishay.com/docs/20035/dcrcwe3.pdf"
+			(at 62.23 57.912 90)
+			(effects
+				(font
+					(size 1.27 1.27)
+				)
+				(hide yes)
+			)
+		)
+		(property "Datasheet" "~"
 			(at 62.23 59.69 0)
 			(effects
@@
 			)
 		)
-		(property "Description" "Resistor, US symbol"
+		(property "Description" "Resistor"
 			(at 62.23 59.69 0)
 			(effects
@@
 	)
 	(symbol
-		(lib_id "Device:R_US")
+		(lib_id "Device:R")
 		(at 60.96 120.65 270)
 		(unit 1)
@@
 		)
 		(property "Footprint" "Resistor_SMD:R_0603_1608Metric"
-			(at 60.706 121.666 90)
-			(effects
-				(font
-					(size 1.27 1.27)
-				)
-				(hide yes)
-			)
-		)
-		(property "Datasheet" "https://www.vishay.com/docs/20035/dcrcwe3.pdf"
+			(at 60.96 118.872 90)
+			(effects
+				(font
+					(size 1.27 1.27)
+				)
+				(hide yes)
+			)
+		)
+		(property "Datasheet" "~"
 			(at 60.96 120.65 0)
 			(effects
@@
 			)
 		)
-		(property "Description" "Resistor, US symbol"
+		(property "Description" "Resistor"
 			(at 60.96 120.65 0)
 			(effects
@@
 	)
 	(symbol
-		(lib_id "Device:R_US")
+		(lib_id "Device:R")
 		(at 82.55 50.8 0)
 		(mirror x)
@@
 		)
 		(property "Footprint" "Resistor_SMD:R_0603_1608Metric"
-			(at 83.566 50.546 90)
-			(effects
-				(font
-					(size 1.27 1.27)
-				)
-				(hide yes)
-			)
-		)
-		(property "Datasheet" "https://www.vishay.com/docs/20035/dcrcwe3.pdf"
+			(at 80.772 50.8 90)
+			(effects
+				(font
+					(size 1.27 1.27)
+				)
+				(hide yes)
+			)
+		)
+		(property "Datasheet" "~"
 			(at 82.55 50.8 0)
 			(effects
@@
 			)
 		)
-		(property "Description" "Resistor, US symbol"
+		(property "Description" "Resistor"
 			(at 82.55 50.8 0)
 			(effects
@@
 	)
 	(symbol
-		(lib_id "Device:R_US")
+		(lib_id "Device:R")
 		(at 88.9 44.45 90)
 		(mirror x)
@@
 		)
 		(property "Footprint" "Resistor_SMD:R_0603_1608Metric"
-			(at 89.154 45.466 90)
-			(effects
-				(font
-					(size 1.27 1.27)
-				)
-				(hide yes)
-			)
-		)
-		(property "Datasheet" "https://www.vishay.com/docs/20035/dcrcwe3.pdf"
+			(at 88.9 42.672 90)
+			(effects
+				(font
+					(size 1.27 1.27)
+				)
+				(hide yes)
+			)
+		)
+		(property "Datasheet" "~"
 			(at 88.9 44.45 0)
 			(effects
@@
 			)
 		)
-		(property "Description" "Resistor, US symbol"
+		(property "Description" "Resistor"
 			(at 88.9 44.45 0)
 			(effects
@@
 	)
 	(symbol
-		(lib_id "Device:R_US")
+		(lib_id "Device:R")
 		(at 88.9 105.41 90)
 		(mirror x)
@@
 		)
 		(property "Footprint" "Resistor_SMD:R_0603_1608Metric"
-			(at 89.154 106.426 90)
-			(effects
-				(font
-					(size 1.27 1.27)
-				)
-				(hide yes)
-			)
-		)
-		(property "Datasheet" "https://www.vishay.com/docs/20035/dcrcwe3.pdf"
+			(at 88.9 103.632 90)
+			(effects
+				(font
+					(size 1.27 1.27)
+				)
+				(hide yes)
+			)
+		)
+		(property "Datasheet" "~"
 			(at 88.9 105.41 0)
 			(effects
@@
 			)
 		)
-		(property "Description" "Resistor, US symbol"
+		(property "Description" "Resistor"
 			(at 88.9 105.41 0)
 			(effects

Commit message: end of workday
Connections:
- net +24V renamed +12V
Changed lines of the file:
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@@
 			)
 		)
-		(property "Value" "+24V"
+		(property "Value" "+12V"
 			(at 110.49 24.13 0)
 			(show_name no)

Commit message: finished schematic except for 12v buck boost
Parts:
- ESTOP1: renamed from ESTOP2; footprint LED_SMD:LED_0603_1608Metric -> LED_SMD:LED_0603_1608Metric_Pad1.05x0.95mm_HandSolder
- ESTOP2: renamed from ESTOP3; footprint LED_SMD:LED_0603_1608Metric -> LED_SMD:LED_0603_1608Metric_Pad1.05x0.95mm_HandSolder
- ESTOP3: renamed from ESTOP1; footprint LED_SMD:LED_0603_1608Metric -> LED_SMD:LED_0603_1608Metric_Pad1.05x0.95mm_HandSolder
- J14: renamed from J10; footprint UTSVT_Connectors:Molex_Nano-Fit_105309-xx02_1x02_P2.50mm_Vertical -> LHRS_Connectors:Molex_Nano-Fit_105309-xx02_1x02_P2.50mm_Vertical
- Q1: renamed from Q7; footprint CustomKiCad-Library:SOT95P237X112-3N -> Package_TO_SOT_SMD:TSOT-23-6_HandSoldering
- Q2: renamed from Q5; footprint CustomKiCad-Library:SOT95P237X112-3N -> Package_TO_SOT_SMD:TSOT-23-6_HandSoldering
- Q3: renamed from Q8; footprint CustomKiCad-Library:SOT95P237X112-3N -> Package_TO_SOT_SMD:TSOT-23-6_HandSoldering
- R27: renamed from R63; footprint Resistor_SMD:R_0603_1608Metric -> Resistor_SMD:R_0603_1608Metric_Pad0.98x0.95mm_HandSolder
- R28: renamed from R73; footprint Resistor_SMD:R_0603_1608Metric -> Resistor_SMD:R_0603_1608Metric_Pad0.98x0.95mm_HandSolder
- R29: renamed from R72; footprint Resistor_SMD:R_0603_1608Metric -> Resistor_SMD:R_0603_1608Metric_Pad0.98x0.95mm_HandSolder
- R30: renamed from R69; footprint Resistor_SMD:R_0603_1608Metric -> Resistor_SMD:R_0603_1608Metric_Pad0.98x0.95mm_HandSolder
- R31: renamed from R70; footprint Resistor_SMD:R_0603_1608Metric -> Resistor_SMD:R_0603_1608Metric_Pad0.98x0.95mm_HandSolder
- R32: renamed from R71; footprint Resistor_SMD:R_0603_1608Metric -> Resistor_SMD:R_0603_1608Metric_Pad0.98x0.95mm_HandSolder
- R33: renamed from R91; footprint Resistor_SMD:R_0603_1608Metric -> Resistor_SMD:R_0603_1608Metric_Pad0.98x0.95mm_HandSolder
- R34: renamed from R93; footprint Resistor_SMD:R_0603_1608Metric -> Resistor_SMD:R_0603_1608Metric_Pad0.98x0.95mm_HandSolder
- R35: renamed from R94; footprint Resistor_SMD:R_0603_1608Metric -> Resistor_SMD:R_0603_1608Metric_Pad0.98x0.95mm_HandSolder
- R36: renamed from R35; footprint Resistor_SMD:R_0603_1608Metric -> Resistor_SMD:R_0603_1608Metric_Pad0.98x0.95mm_HandSolder
- R37: renamed from R95; footprint Resistor_SMD:R_0603_1608Metric -> Resistor_SMD:R_0603_1608Metric_Pad0.98x0.95mm_HandSolder
- R38: renamed from R34; footprint Resistor_SMD:R_0603_1608Metric -> Resistor_SMD:R_0603_1608Metric_Pad0.98x0.95mm_HandSolder

Commit message: added 12V buck boost
Parts:
- renumbered R27 to R31, R28 to R32, R29 to R33, R30 to R34, R31 to R35, R32 to R36, R33 to R37, R34 to R38, R35 to R39, R36 to R40, R37 to R41, R38 to R42
Changed lines of the file:
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@@
 		(in_pos_files yes)
 		(dnp no)
-		(property "Reference" "R30"
+		(property "Reference" "R34"
 			(at 60.96 96.52 90)
 			(show_name no)
@@
 			(project "PS-BPSLeader"
 				(path "/d4a4ed4f-0983-4aef-b212-0e3284ab3963/ff3d6d8a-5585-4a16-aaa1-d2e71ebe7413"
-					(reference "R30")
+					(reference "R34")
 					(unit 1)
 				)
@@
 		(in_pos_files yes)
 		(dnp no)
-		(property "Reference" "R29"
+		(property "Reference" "R33"
 			(at 61.976 83.82 90)
 			(show_name no)
@@
 			(project "PS-BPSLeader"
 				(path "/d4a4ed4f-0983-4aef-b212-0e3284ab3963/ff3d6d8a-5585-4a16-aaa1-d2e71ebe7413"
-					(reference "R29")
+					(reference "R33")
 					(unit 1)
 				)
@@
 		(in_pos_files yes)
 		(dnp no)
-		(property "Reference" "R35"
+		(property "Reference" "R39"
 			(at 80.772 110.744 0)
 			(show_name no)
@@
 			(project "PS-BPSLeader"
 				(path "/d4a4ed4f-0983-4aef-b212-0e3284ab3963/ff3d6d8a-5585-4a16-aaa1-d2e71ebe7413"
-					(reference "R35")
+					(reference "R39")
 					(unit 1)
 				)
@@
 		(in_pos_files yes)
 		(dnp no)
-		(property "Reference" "R27"
+		(property "Reference" "R31"
 			(at 60.706 113.03 90)
 			(show_name no)
@@
 			(project "PS-BPSLeader"
 				(path "/d4a4ed4f-0983-4aef-b212-0e3284ab3963/ff3d6d8a-5585-4a16-aaa1-d2e71ebe7413"
-					(reference "R27")
+					(reference "R31")
 					(unit 1)
 				)
@@
 		(in_pos_files yes)
 		(dnp no)
-		(property "Reference" "R34"
+		(property "Reference" "R38"
 			(at 80.772 81.534 0)
 			(show_name no)
@@
 			(project "PS-BPSLeader"
 				(path "/d4a4ed4f-0983-4aef-b212-0e3284ab3963/ff3d6d8a-5585-4a16-aaa1-d2e71ebe7413"
-					(reference "R34")
+					(reference "R38")
 					(unit 1)
 				)
@@
 		(in_pos_files yes)
 		(dnp no)
-		(property "Reference" "R37"
+		(property "Reference" "R41"
 			(at 88.646 74.168 90)
 			(show_name no)
@@
 			(project "PS-BPSLeader"
 				(path "/d4a4ed4f-0983-4aef-b212-0e3284ab3963/ff3d6d8a-5585-4a16-aaa1-d2e71ebe7413"
-					(reference "R37")
+					(reference "R41")
 					(unit 1)
 				)
@@
 		(in_pos_files yes)
 		(dnp no)
-		(property "Reference" "R28"
+		(property "Reference" "R32"
 			(at 61.976 52.07 90)
 			(show_name no)
@@
 			(project "PS-BPSLeader"
 				(path "/d4a4ed4f-0983-4aef-b212-0e3284ab3963/ff3d6d8a-5585-4a16-aaa1-d2e71ebe7413"
-					(reference "R28")
+					(reference "R32")
 					(unit 1)
 				)
@@
 		(in_pos_files yes)
 		(dnp no)
-		(property "Reference" "R32"
+		(property "Reference" "R36"
 			(at 62.23 64.77 90)
 			(show_name no)
@@
 			(project "PS-BPSLeader"
 				(path "/d4a4ed4f-0983-4aef-b212-0e3284ab3963/ff3d6d8a-5585-4a16-aaa1-d2e71ebe7413"
-					(reference "R32")
+					(reference "R36")
 					(unit 1)
 				)
@@
 		(in_pos_files yes)
 		(dnp no)
-		(property "Reference" "R31"
+		(property "Reference" "R35"
 			(at 60.96 125.73 90)
 			(show_name no)
@@
 			(project "PS-BPSLeader"
 				(path "/d4a4ed4f-0983-4aef-b212-0e3284ab3963/ff3d6d8a-5585-4a16-aaa1-d2e71ebe7413"
-					(reference "R31")
+					(reference "R35")
 					(unit 1)
 				)
@@
 		(in_pos_files yes)
 		(dnp no)
-		(property "Reference" "R33"
+		(property "Reference" "R37"
 			(at 80.772 49.784 0)
 			(show_name no)
@@
 			(project "PS-BPSLeader"
 				(path "/d4a4ed4f-0983-4aef-b212-0e3284ab3963/ff3d6d8a-5585-4a16-aaa1-d2e71ebe7413"
-					(reference "R33")
+					(reference "R37")
 					(unit 1)
 				)
@@
 		(in_pos_files yes)
 		(dnp no)
-		(property "Reference" "R36"
+		(property "Reference" "R40"
 			(at 88.646 42.418 90)
 			(show_name no)
@@
 			(project "PS-BPSLeader"
 				(path "/d4a4ed4f-0983-4aef-b212-0e3284ab3963/ff3d6d8a-5585-4a16-aaa1-d2e71ebe7413"
-					(reference "R36")
+					(reference "R40")
 					(unit 1)
 				)
@@
 		(in_pos_files yes)
 		(dnp no)
-		(property "Reference" "R38"
+		(property "Reference" "R42"
 			(at 88.646 103.378 90)
 			(show_name no)
@@
 			(project "PS-BPSLeader"
 				(path "/d4a4ed4f-0983-4aef-b212-0e3284ab3963/ff3d6d8a-5585-4a16-aaa1-d2e71ebe7413"
-					(reference "R38")
+					(reference "R42")
 					(unit 1)
 				)

Commit message: forgot to push last night
Parts:
- Q1, Q2, Q3: footprint Package_TO_SOT_SMD:TSOT-23-6_HandSoldering -> Package_TO_SOT_SMD:SOT-23
Changed lines of the file:
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@@
 			)
 		)
-		(property "Footprint" "Package_TO_SOT_SMD:TSOT-23-6_HandSoldering"
+		(property "Footprint" "Package_TO_SOT_SMD:SOT-23"
 			(at 66.04 -54.28 0)
 			(hide yes)
@@
 			)
 		)
-		(property "Footprint" "Package_TO_SOT_SMD:TSOT-23-6_HandSoldering"
+		(property "Footprint" "Package_TO_SOT_SMD:SOT-23"
 			(at 64.77 -22.53 0)
 			(hide yes)
@@
 			)
 		)
-		(property "Footprint" "Package_TO_SOT_SMD:TSOT-23-6_HandSoldering"
+		(property "Footprint" "Package_TO_SOT_SMD:SOT-23"
 			(at 64.77 6.68 0)
 			(hide yes)

Commit message: kms drc crashed and didn't save layout
Parts:
- R34, R35, R36: value 470 -> 1k
Changed lines of the file:
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@@
 			)
 		)
-		(property "Value" "470"
+		(property "Value" "1k"
 			(at 60.96 93.98 90)
 			(show_name no)
@@
 			)
 		)
-		(property "Value" "470"
+		(property "Value" "1k"
 			(at 62.23 62.23 90)
 			(show_name no)
@@
 			)
 		)
-		(property "Value" "470"
+		(property "Value" "1k"
 			(at 60.96 123.19 90)
 			(show_name no)
