File: hardware/ESTOP.kicad_sch (KiCad schematic)
At the start: 22 parts, among them J14 Conn_01x02, Q1 SQ2315CES-T1_GE3, Q2 SQ2315CES-T1_GE3, Q3 SQ2315CES-T1_GE3

Commit message: push gerbers and stuff
Parts:
- E_JP1, E_JP2, E_JP3: now left out of the parts list
Changed lines of the file:
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@@
 		(body_style 1)
 		(exclude_from_sim no)
-		(in_bom yes)
+		(in_bom no)
 		(on_board yes)
 		(in_pos_files yes)
@@
 		(body_style 1)
 		(exclude_from_sim no)
-		(in_bom yes)
+		(in_bom no)
 		(on_board yes)
 		(in_pos_files yes)
@@
 		(body_style 1)
 		(exclude_from_sim no)
-		(in_bom yes)
+		(in_bom no)
 		(on_board yes)
 		(in_pos_files yes)
