File: hardware/ESP32.kicad_sch (KiCad schematic)
At the start: 21 parts, among them J1 USB_C_Receptacle_USB2.0_16P, SW1 BOOT Switch, SW2 RESET Button, U1 ESP32-C6-MINI-1

Commit message: finished schematic except for 12v buck boost
Parts:
- C23: renamed from C1; footprint Capacitor_SMD:C_0805_2012Metric -> Capacitor_SMD:C_0805_2012Metric_Pad1.18x1.45mm_HandSolder
- C24: renamed from C2; footprint Capacitor_SMD:C_0805_2012Metric -> Capacitor_SMD:C_0805_2012Metric_Pad1.18x1.45mm_HandSolder
- C25: renamed from C3; footprint Capacitor_SMD:C_0603_1608Metric -> Capacitor_SMD:C_0603_1608Metric_Pad1.08x0.95mm_HandSolder
- C26: renamed from C4; footprint Capacitor_SMD:C_0603_1608Metric -> Capacitor_SMD:C_0603_1608Metric_Pad1.08x0.95mm_HandSolder
- D7: renamed from D3; footprint Diode_SMD:D_0603_1608Metric -> LED_SMD:LED_0603_1608Metric_Pad1.05x0.95mm_HandSolder
- D8: renamed from D4; footprint Diode_SMD:D_0603_1608Metric -> LED_SMD:LED_0603_1608Metric_Pad1.05x0.95mm_HandSolder
- D9: renamed from D5; footprint Diode_SMD:D_0603_1608Metric -> LED_SMD:LED_0603_1608Metric_Pad1.05x0.95mm_HandSolder
- J13: renamed from J1; footprint UTSVT_Connectors:USB_C_Receptacle_GCT_USB4105-xx-A_16P_TopMnt_Horizontal -> LHRS_Connectors:USB_C_Receptacle_GCT_USB4105-xx-A_16P_TopMnt_Horizontal
- R19: renamed from R10; footprint Resistor_SMD:R_0603_1608Metric -> Resistor_SMD:R_0603_1608Metric_Pad0.98x0.95mm_HandSolder
- R20: renamed from R11; footprint Resistor_SMD:R_0603_1608Metric -> Resistor_SMD:R_0603_1608Metric_Pad0.98x0.95mm_HandSolder
- R21: renamed from R12; footprint Resistor_SMD:R_0603_1608Metric -> Resistor_SMD:R_0603_1608Metric_Pad0.98x0.95mm_HandSolder
- R22: renamed from R13; footprint Resistor_SMD:R_0603_1608Metric -> Resistor_SMD:R_0603_1608Metric_Pad0.98x0.95mm_HandSolder
- R23: renamed from R14; footprint Resistor_SMD:R_0603_1608Metric -> Resistor_SMD:R_0603_1608Metric_Pad0.98x0.95mm_HandSolder
- R24: renamed from R15; footprint Resistor_SMD:R_0603_1608Metric -> Resistor_SMD:R_0603_1608Metric_Pad0.98x0.95mm_HandSolder
- R25: renamed from R16; footprint Resistor_SMD:R_0603_1608Metric -> Resistor_SMD:R_0603_1608Metric_Pad0.98x0.95mm_HandSolder
- R26: renamed from R17; footprint Resistor_SMD:R_0603_1608Metric -> Resistor_SMD:R_0603_1608Metric_Pad0.98x0.95mm_HandSolder
- SW2: renamed from SW1; footprint UTSVT_Special:BootSW -> LHRS_Special:BootSW
- SW3: renamed from SW2; footprint UTSVT_Special:TL3365AF180QG -> LHRS_Special:TL3365AF180QG
- U4: renamed from U1; footprint UTSVT_Special:ESP32-C6-MINI-1 -> LHRS_Special:ESP32-C6-MINI-1
- renumbered D1 to D5, D2 to D6

Commit message: added 12V buck boost
Parts:
- renumbered C23 to C24, C24 to C25, C25 to C26, C26 to C27, D8 to D10, D9 to D11, D5 to D7, D6 to D8, D7 to D9, R19 to R23, R20 to R24, R21 to R25, R22 to R26, R23 to R27, R24 to R28, R25 to R29, R26 to R30
Changed lines of the file:
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@@
 		(dnp no)
 		(fields_autoplaced yes)
-		(property "Reference" "R25"
+		(property "Reference" "R29"
 			(at 200.66 29.21 90)
 			(show_name no)
@@
 			(project "PS-BPSLeader"
 				(path "/d4a4ed4f-0983-4aef-b212-0e3284ab3963/5da56964-fa04-4fec-bdfe-c6acfeda5c9a/37240678-40e7-4b21-a99e-c284d3b12e6a"
-					(reference "R25")
+					(reference "R29")
 					(unit 1)
 				)
@@
 		(in_pos_files yes)
 		(dnp no)
-		(property "Reference" "C23"
+		(property "Reference" "C24"
 			(at 74.168 78.486 0)
 			(show_name no)
@@
 			(project "PS-BPSLeader"
 				(path "/d4a4ed4f-0983-4aef-b212-0e3284ab3963/5da56964-fa04-4fec-bdfe-c6acfeda5c9a/37240678-40e7-4b21-a99e-c284d3b12e6a"
-					(reference "C23")
+					(reference "C24")
 					(unit 1)
 				)
@@
 		(in_pos_files yes)
 		(dnp no)
-		(property "Reference" "C25"
+		(property "Reference" "C26"
 			(at 145.034 72.644 0)
 			(show_name no)
@@
 			(project "PS-BPSLeader"
 				(path "/d4a4ed4f-0983-4aef-b212-0e3284ab3963/5da56964-fa04-4fec-bdfe-c6acfeda5c9a/37240678-40e7-4b21-a99e-c284d3b12e6a"
-					(reference "C25")
+					(reference "C26")
 					(unit 1)
 				)
@@
 		(dnp no)
 		(fields_autoplaced yes)
-		(property "Reference" "D6"
+		(property "Reference" "D8"
 			(at 74.93 135.89 90)
 			(show_name no)
@@
 			(project "PS-BPSLeader"
 				(path "/d4a4ed4f-0983-4aef-b212-0e3284ab3963/5da56964-fa04-4fec-bdfe-c6acfeda5c9a/37240678-40e7-4b21-a99e-c284d3b12e6a"
-					(reference "D6")
+					(reference "D8")
 					(unit 1)
 				)
@@
 		(in_pos_files yes)
 		(dnp no)
-		(property "Reference" "R26"
+		(property "Reference" "R30"
 			(at 200.66 42.418 90)
 			(show_name no)
@@
 			(project "PS-BPSLeader"
 				(path "/d4a4ed4f-0983-4aef-b212-0e3284ab3963/5da56964-fa04-4fec-bdfe-c6acfeda5c9a/37240678-40e7-4b21-a99e-c284d3b12e6a"
-					(reference "R26")
+					(reference "R30")
 					(unit 1)
 				)
@@
 		(in_pos_files yes)
 		(dnp no)
-		(property "Reference" "C24"
+		(property "Reference" "C25"
 			(at 135.636 72.644 0)
 			(show_name no)
@@
 			(project "PS-BPSLeader"
 				(path "/d4a4ed4f-0983-4aef-b212-0e3284ab3963/5da56964-fa04-4fec-bdfe-c6acfeda5c9a/37240678-40e7-4b21-a99e-c284d3b12e6a"
-					(reference "C24")
+					(reference "C25")
 					(unit 1)
 				)
@@
 		(in_pos_files yes)
 		(dnp no)
-		(property "Reference" "D9"
+		(property "Reference" "D11"
 			(at 211.074 42.164 0)
 			(show_name no)
@@
 			(project "PS-BPSLeader"
 				(path "/d4a4ed4f-0983-4aef-b212-0e3284ab3963/5da56964-fa04-4fec-bdfe-c6acfeda5c9a/37240678-40e7-4b21-a99e-c284d3b12e6a"
-					(reference "D9")
+					(reference "D11")
 					(unit 1)
 				)
@@
 		(in_pos_files yes)
 		(dnp no)
-		(property "Reference" "R23"
+		(property "Reference" "R27"
 			(at 197.104 101.854 90)
 			(show_name no)
@@
 			(project "PS-BPSLeader"
 				(path "/d4a4ed4f-0983-4aef-b212-0e3284ab3963/5da56964-fa04-4fec-bdfe-c6acfeda5c9a/37240678-40e7-4b21-a99e-c284d3b12e6a"
-					(reference "R23")
+					(reference "R27")
 					(unit 1)
 				)
@@
 		(dnp no)
 		(fields_autoplaced yes)
-		(property "Reference" "R21"
+		(property "Reference" "R25"
 			(at 107.95 29.21 90)
 			(show_name no)
@@
 			(project "PS-BPSLeader"
 				(path "/d4a4ed4f-0983-4aef-b212-0e3284ab3963/5da56964-fa04-4fec-bdfe-c6acfeda5c9a/37240678-40e7-4b21-a99e-c284d3b12e6a"
-					(reference "R21")
+					(reference "R25")
 					(unit 1)
 				)
@@
 		(in_pos_files yes)
 		(dnp no)
-		(property "Reference" "R20"
+		(property "Reference" "R24"
 			(at 50.038 81.28 90)
 			(show_name no)
@@
 			(project "PS-BPSLeader"
 				(path "/d4a4ed4f-0983-4aef-b212-0e3284ab3963/5da56964-fa04-4fec-bdfe-c6acfeda5c9a/37240678-40e7-4b21-a99e-c284d3b12e6a"
-					(reference "R20")
+					(reference "R24")
 					(unit 1)
 				)
@@
 		(in_pos_files yes)
 		(dnp no)
-		(property "Reference" "R22"
+		(property "Reference" "R26"
 			(at 151.384 25.654 0)
 			(show_name no)
@@
 			(project "PS-BPSLeader"
 				(path "/d4a4ed4f-0983-4aef-b212-0e3284ab3963/5da56964-fa04-4fec-bdfe-c6acfeda5c9a/37240678-40e7-4b21-a99e-c284d3b12e6a"
-					(reference "R22")
+					(reference "R26")
 					(unit 1)
 				)
@@
 		(in_pos_files yes)
 		(dnp no)
-		(property "Reference" "D5"
+		(property "Reference" "D7"
 			(at 61.722 66.04 0)
 			(show_name no)
@@
 			(project "PS-BPSLeader"
 				(path "/d4a4ed4f-0983-4aef-b212-0e3284ab3963/5da56964-fa04-4fec-bdfe-c6acfeda5c9a/37240678-40e7-4b21-a99e-c284d3b12e6a"
-					(reference "D5")
+					(reference "D7")
 					(unit 1)
 				)
@@
 		(in_pos_files yes)
 		(dnp no)
-		(property "Reference" "C26"
+		(property "Reference" "C27"
 			(at 153.924 35.814 0)
 			(show_name no)
@@
 			(project "PS-BPSLeader"
 				(path "/d4a4ed4f-0983-4aef-b212-0e3284ab3963/5da56964-fa04-4fec-bdfe-c6acfeda5c9a/37240678-40e7-4b21-a99e-c284d3b12e6a"
-					(reference "C26")
+					(reference "C27")
 					(unit 1)
 				)
@@
 		(in_pos_files yes)
 		(dnp no)
-		(property "Reference" "R19"
+		(property "Reference" "R23"
 			(at 50.292 76.2 90)
 			(show_name no)
@@
 			(project "PS-BPSLeader"
 				(path "/d4a4ed4f-0983-4aef-b212-0e3284ab3963/5da56964-fa04-4fec-bdfe-c6acfeda5c9a/37240678-40e7-4b21-a99e-c284d3b12e6a"
-					(reference "R19")
+					(reference "R23")
 					(unit 1)
 				)
@@
 		(in_pos_files yes)
 		(dnp no)
-		(property "Reference" "D8"
+		(property "Reference" "D10"
 			(at 210.82 27.94 0)
 			(show_name no)
@@
 			(project "PS-BPSLeader"
 				(path "/d4a4ed4f-0983-4aef-b212-0e3284ab3963/5da56964-fa04-4fec-bdfe-c6acfeda5c9a/37240678-40e7-4b21-a99e-c284d3b12e6a"
-					(reference "D8")
+					(reference "D10")
 					(unit 1)
 				)
@@
 		(dnp no)
 		(fields_autoplaced yes)
-		(property "Reference" "R24"
+		(property "Reference" "R28"
 			(at 200.66 19.05 90)
 			(show_name no)
@@
 			(project "PS-BPSLeader"
 				(path "/d4a4ed4f-0983-4aef-b212-0e3284ab3963/5da56964-fa04-4fec-bdfe-c6acfeda5c9a/37240678-40e7-4b21-a99e-c284d3b12e6a"
-					(reference "R24")
+					(reference "R28")
 					(unit 1)
 				)
@@
 		(in_pos_files yes)
 		(dnp no)
-		(property "Reference" "D7"
+		(property "Reference" "D9"
 			(at 210.82 17.78 0)
 			(show_name no)
@@
 			(project "PS-BPSLeader"
 				(path "/d4a4ed4f-0983-4aef-b212-0e3284ab3963/5da56964-fa04-4fec-bdfe-c6acfeda5c9a/37240678-40e7-4b21-a99e-c284d3b12e6a"
-					(reference "D7")
+					(reference "D9")
 					(unit 1)
 				)

Commit message: papercut -linkin park
Connections:
- net ESP_GPIO1: now also U4.12 (GPIO0/ADC1_CH0/XTAL_32K_P); no longer U4.19 (GPIO14)
- net ESP_GPIO2: now also U4.13 (GPIO1/ADC1_CH1/XTAL_32K_N); no longer U4.20 (GPIO15)
- net ESP_GPIO3: now also U4.15 (MTCK/GPIO6/ADC1_CH6); no longer U4.24 (GPIO18)
- net ESP_GPIO4: now also U4.16 (MTDO/GPIO7); no longer U4.25 (GPIO19)
Changed lines of the file:
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@@
+	)
+	(no_connect
+		(at 196.85 111.76)
+	)
+	(no_connect
+		(at 196.85 116.84)
 	)
 	(no_connect
@@
 	)
 	(no_connect
-		(at 128.27 111.76)
-	)
-	(no_connect
 		(at 46.99 100.33)
 	)
@@
 	)
 	(no_connect
+		(at 196.85 119.38)
+	)
+	(no_connect
 		(at 128.27 99.06)
-	)
-	(no_connect
-		(at 128.27 93.98)
-	)
-	(no_connect
-		(at 128.27 114.3)
 	)
 	(no_connect
@@
 	)
 	(no_connect
-		(at 128.27 91.44)
+		(at 196.85 114.3)
 	)
 	(wire
@@
 			)
 			(justify right bottom)
+		)
+	)
+	(hierarchical_label "ESP_GPIO3"
+		(shape bidirectional)
+		(at 128.27 111.76 180)
+		(effects
+			(font
+				(size 1.27 1.27)
+			)
+			(justify right)
 		)
 	)
@@
 		)
 	)
-	(hierarchical_label "ESP_GPIO1"
-		(shape bidirectional)
-		(at 196.85 111.76 0)
-		(effects
-			(font
-				(size 1.27 1.27)
-			)
-			(justify left)
-		)
-	)
 	(hierarchical_label "ESP_GPIO2"
 		(shape bidirectional)
-		(at 196.85 114.3 0)
-		(effects
-			(font
-				(size 1.27 1.27)
-			)
-			(justify left)
+		(at 128.27 93.98 180)
+		(effects
+			(font
+				(size 1.27 1.27)
+			)
+			(justify right)
 		)
 	)
@@
 		)
 	)
-	(hierarchical_label "ESP_GPIO3"
+	(hierarchical_label "ESP_GPIO1"
 		(shape bidirectional)
-		(at 196.85 116.84 0)
-		(effects
-			(font
-				(size 1.27 1.27)
-			)
-			(justify left)
+		(at 128.27 91.44 180)
+		(effects
+			(font
+				(size 1.27 1.27)
+			)
+			(justify right)
 		)
 	)
@@
 		)
 	)
+	(hierarchical_label "ESP_GPIO4"
+		(shape bidirectional)
+		(at 128.27 114.3 180)
+		(effects
+			(font
+				(size 1.27 1.27)
+			)
+			(justify right)
+		)
+	)
 	(hierarchical_label "GND"
 		(shape input)
@@
 		)
 	)
-	(hierarchical_label "ESP_GPIO4"
-		(shape bidirectional)
-		(at 196.85 119.38 0)
-		(effects
-			(font
-				(size 1.27 1.27)
-			)
-			(justify left)
-		)
-	)
