File: hardware/ESP32_LDO.kicad_sch (KiCad schematic)
At the start: 5 parts, among them U1 MCP1826S

Commit message: finished schematic except for 12v buck boost
Parts:
- renumbered C1 to C48, C2 to C49, D1 to D21, U1 to U10
Changed lines of the file:
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@@
 		(dnp no)
 		(fields_autoplaced yes)
-		(property "Reference" "C2"
+		(property "Reference" "C49"
 			(at 168.275 68.5735 0)
 			(show_name no)
@@
 			(project "PS-BPSLeader"
 				(path "/d4a4ed4f-0983-4aef-b212-0e3284ab3963/5da56964-fa04-4fec-bdfe-c6acfeda5c9a/92d40a22-22a8-4e19-ae2b-d2176aa2e41e"
-					(reference "C2")
+					(reference "C49")
 					(unit 1)
 				)
@@
 		(dnp no)
 		(fields_autoplaced yes)
-		(property "Reference" "U1"
+		(property "Reference" "U10"
 			(at 152.4 56.515 0)
 			(show_name no)
@@
 			(project "PS-BPSLeader"
 				(path "/d4a4ed4f-0983-4aef-b212-0e3284ab3963/5da56964-fa04-4fec-bdfe-c6acfeda5c9a/92d40a22-22a8-4e19-ae2b-d2176aa2e41e"
-					(reference "U1")
+					(reference "U10")
 					(unit 1)
 				)
@@
 		(dnp no)
 		(fields_autoplaced yes)
-		(property "Reference" "D1"
+		(property "Reference" "D21"
 			(at 133.604 57.15 0)
 			(show_name no)
@@
 			(project "PS-BPSLeader"
 				(path "/d4a4ed4f-0983-4aef-b212-0e3284ab3963/5da56964-fa04-4fec-bdfe-c6acfeda5c9a/92d40a22-22a8-4e19-ae2b-d2176aa2e41e"
-					(reference "D1")
+					(reference "D21")
 					(unit 1)
 				)
@@
 		(dnp no)
 		(fields_autoplaced yes)
-		(property "Reference" "C1"
+		(property "Reference" "C48"
 			(at 142.875 68.5735 0)
 			(show_name no)
@@
 			(project "PS-BPSLeader"
 				(path "/d4a4ed4f-0983-4aef-b212-0e3284ab3963/5da56964-fa04-4fec-bdfe-c6acfeda5c9a/92d40a22-22a8-4e19-ae2b-d2176aa2e41e"
-					(reference "C1")
-					(unit 1)
-				)
+					(reference "C48")
+					(unit 1)
+				)

Commit message: added 12V buck boost
Parts:
- renumbered C48 to C49, C49 to C50, D21 to D23
Changed lines of the file:
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@@
 		(dnp no)
 		(fields_autoplaced yes)
-		(property "Reference" "C49"
+		(property "Reference" "C50"
 			(at 168.275 68.5735 0)
 			(show_name no)
@@
 			(project "PS-BPSLeader"
 				(path "/d4a4ed4f-0983-4aef-b212-0e3284ab3963/5da56964-fa04-4fec-bdfe-c6acfeda5c9a/92d40a22-22a8-4e19-ae2b-d2176aa2e41e"
-					(reference "C49")
+					(reference "C50")
 					(unit 1)
 				)
@@
 		(dnp no)
 		(fields_autoplaced yes)
-		(property "Reference" "D21"
+		(property "Reference" "D23"
 			(at 133.604 57.15 0)
 			(show_name no)
@@
 			(project "PS-BPSLeader"
 				(path "/d4a4ed4f-0983-4aef-b212-0e3284ab3963/5da56964-fa04-4fec-bdfe-c6acfeda5c9a/92d40a22-22a8-4e19-ae2b-d2176aa2e41e"
-					(reference "D21")
+					(reference "D23")
 					(unit 1)
 				)
@@
 		(dnp no)
 		(fields_autoplaced yes)
-		(property "Reference" "C48"
+		(property "Reference" "C49"
 			(at 142.875 68.5735 0)
 			(show_name no)
@@
 			(project "PS-BPSLeader"
 				(path "/d4a4ed4f-0983-4aef-b212-0e3284ab3963/5da56964-fa04-4fec-bdfe-c6acfeda5c9a/92d40a22-22a8-4e19-ae2b-d2176aa2e41e"
-					(reference "C48")
-					(unit 1)
-				)
+					(reference "C49")
+					(unit 1)
+				)

Commit message: push gerbers and stuff
Parts:
- TP_3.3V1: now not fitted
Changed lines of the file:
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@@
 		(on_board yes)
 		(in_pos_files yes)
-		(dnp no)
+		(dnp yes)
 		(property "Reference" "TP_3.3V1"
 			(at 166.624 54.356 90)
