File: hardware/HV_Plus_Contactor.kicad_sch (KiCad schematic)
At the start: 25 parts, among them J16 Contactor Connector, Q6 IRLML0030, Q7 IRLML0030, U7 DRV110APWR

Commit message: added 12V buck boost
Parts:
- TP7, TP8: footprint TestPoint:TestPoint_THTPad_D3.0mm_Drill1.5mm -> TestPoint:TestPoint_Loop_D1.80mm_Drill1.0mm_Beaded
- renumbered C34 to C35, C35 to C36, C36 to C37, C37 to C38, C38 to C39, C39 to C40, D13 to D15, D14 to D16, D15 to D17, R58 to R62, R59 to R63, R60 to R64, R61 to R65, R62 to R66, R63 to R67, R64 to R68, R65 to R69, R66 to R70, R67 to R71
Changed lines of the file:
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@@
 		(dnp no)
 		(fields_autoplaced yes)
-		(property "Reference" "R58"
+		(property "Reference" "R62"
 			(at 47.625 93.3449 0)
 			(show_name no)
@@
 			(project "PS-BPSLeader"
 				(path "/d4a4ed4f-0983-4aef-b212-0e3284ab3963/d0687915-3890-41dc-9a8f-e7ee1bda9492"
-					(reference "R58")
+					(reference "R62")
 					(unit 1)
 				)
@@
 		(dnp no)
 		(fields_autoplaced yes)
-		(property "Reference" "R63"
+		(property "Reference" "R67"
 			(at 130.175 48.895 90)
 			(show_name no)
@@
 			(project "PS-BPSLeader"
 				(path "/d4a4ed4f-0983-4aef-b212-0e3284ab3963/d0687915-3890-41dc-9a8f-e7ee1bda9492"
-					(reference "R63")
+					(reference "R67")
 					(unit 1)
 				)
@@
 		(dnp no)
 		(fields_autoplaced yes)
-		(property "Reference" "C36"
+		(property "Reference" "C37"
 			(at 59.055 69.2149 0)
 			(show_name no)
@@
 			(project "PS-BPSLeader"
 				(path "/d4a4ed4f-0983-4aef-b212-0e3284ab3963/d0687915-3890-41dc-9a8f-e7ee1bda9492"
-					(reference "C36")
+					(reference "C37")
 					(unit 1)
 				)
@@
 		(dnp no)
 		(fields_autoplaced yes)
-		(property "Reference" "C35"
+		(property "Reference" "C36"
 			(at 55.245 97.1612 0)
 			(show_name no)
@@
 			(project "PS-BPSLeader"
 				(path "/d4a4ed4f-0983-4aef-b212-0e3284ab3963/d0687915-3890-41dc-9a8f-e7ee1bda9492"
-					(reference "C35")
+					(reference "C36")
 					(unit 1)
 				)
@@
 		(dnp no)
 		(fields_autoplaced yes)
-		(property "Reference" "C34"
+		(property "Reference" "C35"
 			(at 43.815 50.1649 0)
 			(show_name no)
@@
 			(project "PS-BPSLeader"
 				(path "/d4a4ed4f-0983-4aef-b212-0e3284ab3963/d0687915-3890-41dc-9a8f-e7ee1bda9492"
-					(reference "C34")
+					(reference "C35")
 					(unit 1)
 				)
@@
 		(dnp no)
 		(fields_autoplaced yes)
-		(property "Reference" "R59"
+		(property "Reference" "R63"
 			(at 62.865 98.4249 0)
 			(show_name no)
@@
 			(project "PS-BPSLeader"
 				(path "/d4a4ed4f-0983-4aef-b212-0e3284ab3963/d0687915-3890-41dc-9a8f-e7ee1bda9492"
-					(reference "R59")
+					(reference "R63")
 					(unit 1)
 				)
@@
 			)
 		)
-		(property "Footprint" "TestPoint:TestPoint_THTPad_D3.0mm_Drill1.5mm"
+		(property "Footprint" "TestPoint:TestPoint_Loop_D1.80mm_Drill1.0mm_Beaded"
 			(at 181.61 51.435 0)
 			(hide yes)
@@
 		(dnp no)
 		(fields_autoplaced yes)
-		(property "Reference" "R66"
+		(property "Reference" "R70"
 			(at 198.12 56.5149 0)
 			(show_name no)
@@
 			(project "PS-BPSLeader"
 				(path "/d4a4ed4f-0983-4aef-b212-0e3284ab3963/d0687915-3890-41dc-9a8f-e7ee1bda9492"
-					(reference "R66")
+					(reference "R70")
 					(unit 1)
 				)
@@
 		(dnp no)
 		(fields_autoplaced yes)
-		(property "Reference" "D14"
+		(property "Reference" "D16"
 			(at 126.365 61.9124 90)
 			(show_name no)
@@
 			(project "PS-BPSLeader"
 				(path "/d4a4ed4f-0983-4aef-b212-0e3284ab3963/d0687915-3890-41dc-9a8f-e7ee1bda9492"
-					(reference "D14")
+					(reference "D16")
 					(unit 1)
 				)
@@
 		(dnp no)
 		(fields_autoplaced yes)
-		(property "Reference" "R61"
+		(property "Reference" "R65"
 			(at 70.485 100.9649 0)
 			(show_name no)
@@
 			(project "PS-BPSLeader"
 				(path "/d4a4ed4f-0983-4aef-b212-0e3284ab3963/d0687915-3890-41dc-9a8f-e7ee1bda9492"
-					(reference "R61")
+					(reference "R65")
 					(unit 1)
 				)
@@
 		(dnp no)
 		(fields_autoplaced yes)
-		(property "Reference" "R62"
+		(property "Reference" "R66"
 			(at 123.19 78.74 90)
 			(show_name no)
@@
 			(project "PS-BPSLeader"
 				(path "/d4a4ed4f-0983-4aef-b212-0e3284ab3963/d0687915-3890-41dc-9a8f-e7ee1bda9492"
-					(reference "R62")
+					(reference "R66")
 					(unit 1)
 				)
@@
 		(dnp no)
 		(fields_autoplaced yes)
-		(property "Reference" "C37"
+		(property "Reference" "C38"
 			(at 154.305 95.8912 0)
 			(show_name no)
@@
 			(project "PS-BPSLeader"
 				(path "/d4a4ed4f-0983-4aef-b212-0e3284ab3963/d0687915-3890-41dc-9a8f-e7ee1bda9492"
-					(reference "C37")
+					(reference "C38")
 					(unit 1)
 				)
@@
 		(dnp no)
 		(fields_autoplaced yes)
-		(property "Reference" "R60"
+		(property "Reference" "R64"
 			(at 66.675 53.9749 0)
 			(show_name no)
@@
 			(project "PS-BPSLeader"
 				(path "/d4a4ed4f-0983-4aef-b212-0e3284ab3963/d0687915-3890-41dc-9a8f-e7ee1bda9492"
-					(reference "R60")
+					(reference "R64")
 					(unit 1)
 				)
@@
 		(dnp no)
 		(fields_autoplaced yes)
-		(property "Reference" "R65"
+		(property "Reference" "R69"
 			(at 143.51 84.455 90)
 			(show_name no)
@@
 			(project "PS-BPSLeader"
 				(path "/d4a4ed4f-0983-4aef-b212-0e3284ab3963/d0687915-3890-41dc-9a8f-e7ee1bda9492"
-					(reference "R65")
+					(reference "R69")
 					(unit 1)
 				)
@@
 		(in_pos_files yes)
 		(dnp no)
-		(property "Reference" "C39"
+		(property "Reference" "C40"
 			(at 214.63 52.7051 0)
 			(show_name no)
@@
 			(project "PS-BPSLeader"
 				(path "/d4a4ed4f-0983-4aef-b212-0e3284ab3963/d0687915-3890-41dc-9a8f-e7ee1bda9492"
-					(reference "C39")
+					(reference "C40")
 					(unit 1)
 				)
@@
 		(dnp no)
 		(fields_autoplaced yes)
-		(property "Reference" "R64"
+		(property "Reference" "R68"
 			(at 140.335 95.2499 0)
 			(show_name no)
@@
 			(project "PS-BPSLeader"
 				(path "/d4a4ed4f-0983-4aef-b212-0e3284ab3963/d0687915-3890-41dc-9a8f-e7ee1bda9492"
-					(reference "R64")
+					(reference "R68")
 					(unit 1)
 				)
@@
 		(in_pos_files yes)
 		(dnp no)
-		(property "Reference" "D13"
+		(property "Reference" "D15"
 			(at 45.085 67.945 90)
 			(show_name no)
@@
 			(project "PS-BPSLeader"
 				(path "/d4a4ed4f-0983-4aef-b212-0e3284ab3963/d0687915-3890-41dc-9a8f-e7ee1bda9492"
-					(reference "D13")
+					(reference "D15")
 					(unit 1)
 				)
@@
 			)
 		)
-		(property "Footprint" "TestPoint:TestPoint_THTPad_D3.0mm_Drill1.5mm"
+		(property "Footprint" "TestPoint:TestPoint_Loop_D1.80mm_Drill1.0mm_Beaded"
 			(at 106.045 76.835 0)
 			(hide yes)
@@
 		(dnp no)
 		(fields_autoplaced yes)
-		(property "Reference" "R67"
+		(property "Reference" "R71"
 			(at 220.98 38.735 90)
 			(show_name no)
@@
 			(project "PS-BPSLeader"
 				(path "/d4a4ed4f-0983-4aef-b212-0e3284ab3963/d0687915-3890-41dc-9a8f-e7ee1bda9492"
-					(reference "R67")
+					(reference "R71")
 					(unit 1)
 				)
@@
 		(in_pos_files yes)
 		(dnp no)
-		(property "Reference" "D15"
+		(property "Reference" "D17"
 			(at 140.335 59.055 90)
 			(show_name no)
@@
 			(project "PS-BPSLeader"
 				(path "/d4a4ed4f-0983-4aef-b212-0e3284ab3963/d0687915-3890-41dc-9a8f-e7ee1bda9492"
-					(reference "D15")
+					(reference "D17")
 					(unit 1)
 				)
@@
 		(dnp no)
 		(fields_autoplaced yes)
-		(property "Reference" "C38"
+		(property "Reference" "C39"
 			(at 183.515 56.5149 0)
 			(show_name no)
@@
 			(project "PS-BPSLeader"
 				(path "/d4a4ed4f-0983-4aef-b212-0e3284ab3963/d0687915-3890-41dc-9a8f-e7ee1bda9492"
-					(reference "C38")
-					(unit 1)
-				)
+					(reference "C39")
+					(unit 1)
+				)

Commit message: push gerbers and stuff
Parts:
- TP7: now not fitted
Changed lines of the file:
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@@
 		(on_board yes)
 		(in_pos_files yes)
-		(dnp no)
+		(dnp yes)
 		(property "Reference" "TP7"
 			(at 112.395 69.215 0)
