File: hardware/Power_USB_PD.kicad_sch (KiCad schematic)
At the start: 38 parts, among them IC1 CYPD3177-24LQXQ, Q1 SI7997DP-T1-GE3, Q2 SI7997DP-T1-GE3, Q3 IRLML0030

Commit message: finished schematic except for 12v buck boost
Parts:
- renumbered C1 to C58, C2 to C59, C3 to C60, C4 to C61, C5 to C62, C6 to C63, C7 to C64, C8 to C65, C9 to C66, D4 to D22, D5 to D23, D6 to D24, D7 to D25, IC1 to IC3, Q1 to Q10, Q2 to Q11, Q3 to Q12, R18 to R100, R19 to R101, R20 to R102, R21 to R103, R7 to R89, R8 to R90, R9 to R91, R10 to R92, R11 to R93, R12 to R94, R13 to R95, R14 to R96, R15 to R97, R16 to R98, R17 to R99

Commit message: added 12V buck boost
Parts:
- TP20: footprint TestPoint:TestPoint_Pad_1.0x1.0mm -> TestPoint:TestPoint_Loop_D1.80mm_Drill1.0mm_Beaded
- renumbered C58 to C59, C59 to C60, C60 to C61, C61 to C62, C62 to C63, C63 to C64, C64 to C65, C65 to C66, C66 to C67, D22 to D24, D23 to D25, D24 to D26, D25 to D27, R96 to R100, R97 to R101, R98 to R102, R99 to R103, R100 to R104, R101 to R105, R102 to R106, R103 to R107, R89 to R93, R90 to R94, R91 to R95, R92 to R96, R93 to R97, R94 to R98, R95 to R99

Commit message: forgot to push last night
Parts:
- R107: value 1k -> 10k
- TP15, TP16, TP17, TP18, TP19: footprint Connector_PinHeader_2.54mm:PinHeader_1x01_P2.54mm_Vertical -> TestPoint:TestPoint_Loop_D1.80mm_Drill1.0mm_Beaded
Changed lines of the file:
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@@
 			)
 		)
-		(property "Value" "1k"
+		(property "Value" "10k"
 			(at 255.27 86.36 0)
 			(show_name no)
@@
 			)
 		)
-		(property "Footprint" "Connector_PinHeader_2.54mm:PinHeader_1x01_P2.54mm_Vertical"
+		(property "Footprint" "TestPoint:TestPoint_Loop_D1.80mm_Drill1.0mm_Beaded"
 			(at 143.51 171.45 0)
 			(hide yes)
@@
 			)
 		)
-		(property "Footprint" "Connector_PinHeader_2.54mm:PinHeader_1x01_P2.54mm_Vertical"
+		(property "Footprint" "TestPoint:TestPoint_Loop_D1.80mm_Drill1.0mm_Beaded"
 			(at 143.51 138.43 0)
 			(hide yes)
@@
 			)
 		)
-		(property "Footprint" "Connector_PinHeader_2.54mm:PinHeader_1x01_P2.54mm_Vertical"
+		(property "Footprint" "TestPoint:TestPoint_Loop_D1.80mm_Drill1.0mm_Beaded"
 			(at 49.53 46.99 0)
 			(hide yes)
@@
 			)
 		)
-		(property "Footprint" "Connector_PinHeader_2.54mm:PinHeader_1x01_P2.54mm_Vertical"
+		(property "Footprint" "TestPoint:TestPoint_Loop_D1.80mm_Drill1.0mm_Beaded"
 			(at 163.83 53.34 0)
 			(hide yes)
@@
 			)
 		)
-		(property "Footprint" "Connector_PinHeader_2.54mm:PinHeader_1x01_P2.54mm_Vertical"
+		(property "Footprint" "TestPoint:TestPoint_Loop_D1.80mm_Drill1.0mm_Beaded"
 			(at 151.13 43.18 0)
 			(hide yes)

Commit message: push gerbers and stuff
Parts:
- TP16, TP17, TP18, TP19: now not fitted
Changed lines of the file:
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@@
 		(on_board yes)
 		(in_pos_files yes)
-		(dnp no)
+		(dnp yes)
 		(property "Reference" "TP17"
 			(at 135.89 169.4181 0)
@@
 		(on_board yes)
 		(in_pos_files yes)
-		(dnp no)
+		(dnp yes)
 		(property "Reference" "TP16"
 			(at 135.89 136.3981 0)
@@
 		(on_board yes)
 		(in_pos_files yes)
-		(dnp no)
+		(dnp yes)
 		(property "Reference" "TP19"
 			(at 165.8619 45.72 0)
@@
 		(on_board yes)
 		(in_pos_files yes)
-		(dnp no)
+		(dnp yes)
 		(property "Reference" "TP18"
 			(at 149.0981 50.8 0)
